File: hardware/power.sch (KiCad schematic (older format))
At the start: 14 parts

Commit message: update for power symbol,
Parts:
- added JP?: WS2812_EN, Jumper:SolderJumper-2_P1.3mm_Open_RoundedPad1.0x1.5mm, symbol my_solder_jumper:SolderJumper_2_Open_round
- added JP?: STM32_EN, Jumper:SolderJumper-2_P1.3mm_Open_RoundedPad1.0x1.5mm, symbol my_solder_jumper:SolderJumper_2_Open_round
- added JP?: OLED_EN, Jumper:SolderJumper-2_P1.3mm_Open_RoundedPad1.0x1.5mm, symbol my_solder_jumper:SolderJumper_2_Open_round
- added JP?: BUZZER_EN, Jumper:SolderJumper-2_P1.3mm_Open_RoundedPad1.0x1.5mm, symbol my_solder_jumper:SolderJumper_2_Open_round
Connections:
- net +5V: now also JP?.2 (B), JP?.2 (B), JP?.2 (B), JP?.2 (B)
- new net Vbuzzer: JP?.1 (A)
- new net Voled: JP?.1 (A)
- new net Vstm32: JP?.1 (A)
- new net Vws2812: JP?.1 (A)
Other:
- moved on the sheet: C?, D?, R?, TP?, U?
