File: hardware/power.sch (KiCad schematic (older format))
At the start: 22 parts, among them U2 AMS1117-3.3

Commit message: update route,
Parts:
- U2: footprint Package_TO_SOT_SMD:SOT-223-3_TabPin2 -> footprint-lib:AMS1117_SOT-223
Changed lines of the file:
@@
 EESchema Schematic File Version 4
-LIBS:stm32_aux_keyboard-cache
 EELAYER 29 0
 EELAYER END
 $Descr A4 11693 8268
 encoding utf-8
-Sheet 3 13
+Sheet 1 1
 Title ""
 Date ""
@@
 AR Path="/5CF345FD/5CF4706E" Ref="#PWR?"  Part="1"
 AR Path="/5CF34646/5CF4706E" Ref="#PWR011"  Part="1"
+AR Path="/5CF4706E" Ref="#PWR011"  Part="1"
 F 0 "#PWR011" H 6550 2850 50  0001 C CNN
 F 1 "+5V" H 6600 3200 50  0000 C CNN
@@
 AR Path="/5CF345FD/5D0DF879" Ref="R?"  Part="1"
 AR Path="/5CF34646/5D0DF879" Ref="R5"  Part="1"
+AR Path="/5D0DF879" Ref="R5"  Part="1"
 F 0 "R5" H 6609 3596 50  0000 L CNN
 F 1 "R511,0603" H 6609 3505 50  0000 L CNN
@@
 AR Path="/5CF345FD/5D0DF873" Ref="R?"  Part="1"
 AR Path="/5CF34646/5D0DF873" Ref="R6"  Part="1"
+AR Path="/5D0DF873" Ref="R6"  Part="1"
 F 0 "R6" H 7259 3596 50  0000 L CNN
 F 1 "R511,0603" H 7259 3505 50  0000 L CNN
@@
 AR Path="/5CF345FD/5D0DF86D" Ref="#PWR?"  Part="1"
 AR Path="/5CF34646/5D0DF86D" Ref="#PWR012"  Part="1"
+AR Path="/5D0DF86D" Ref="#PWR012"  Part="1"
 F 0 "#PWR012" H 7200 2850 50  0001 C CNN
 F 1 "+3V3" H 7250 3200 50  0000 C CNN
@@
 AR Path="/5CF345FD/5D0DF85E" Ref="#PWR?"  Part="1"
 AR Path="/5CF34646/5D0DF85E" Ref="#PWR019"  Part="1"
+AR Path="/5D0DF85E" Ref="#PWR019"  Part="1"
 F 0 "#PWR019" H 7200 3500 50  0001 C CNN
 F 1 "GND" H 7205 3577 50  0000 C CNN
@@
 AR Path="/5CF345FD/5D0DF858" Ref="D?"  Part="1"
 AR Path="/5CF34646/5D0DF858" Ref="D2"  Part="1"
+AR Path="/5D0DF858" Ref="D2"  Part="1"
 F 0 "D2" V 7246 3182 50  0000 R CNN
 F 1 "LED_ORANGE" V 7155 3182 50  0000 R CNN
@@
 AR Path="/5CF345FD/5D0DF84F" Ref="#PWR?"  Part="1"
 AR Path="/5CF34646/5D0DF84F" Ref="#PWR018"  Part="1"
+AR Path="/5D0DF84F" Ref="#PWR018"  Part="1"
 F 0 "#PWR018" H 6550 3500 50  0001 C CNN
 F 1 "GND" H 6555 3577 50  0000 C CNN
@@
 AR Path="/5CF345FD/5D0DF849" Ref="D?"  Part="1"
 AR Path="/5CF34646/5D0DF849" Ref="D1"  Part="1"
+AR Path="/5D0DF849" Ref="D1"  Part="1"
 F 0 "D1" V 6596 3182 50  0000 R CNN
 F 1 "LED_GREEN" V 6505 3182 50  0000 R CNN
@@
 AR Path="/5CF345FD/5D0D3B5F" Ref="C?"  Part="1"
 AR Path="/5CF34646/5D0D3B5F" Ref="C3"  Part="1"
+AR Path="/5D0D3B5F" Ref="C3"  Part="1"
 F 0 "C3" H 5488 3496 50  0000 L CNN
 F 1 "CP100uf,16V" H 5488 3405 50  0000 L CNN
@@
 AR Path="/5CF345FD/5D0D3B59" Ref="C?"  Part="1"
 AR Path="/5CF34646/5D0D3B59" Ref="C2"  Part="1"
+AR Path="/5D0D3B59" Ref="C2"  Part="1"
 F 0 "C2" H 4538 3496 50  0000 L CNN
 F 1 "CP100uf,16V" H 4538 3405 50  0000 L CNN
@@
 AR Path="/5CF345FD/5D0D3B53" Ref="#PWR?"  Part="1"
 AR Path="/5CF34646/5D0D3B53" Ref="#PWR09"  Part="1"
+AR Path="/5D0D3B53" Ref="#PWR09"  Part="1"
 F 0 "#PWR09" H 4300 2850 50  0001 C CNN
 F 1 "+5V" H 4350 3200 50  0000 C CNN
@@
 AR Path="/5CF345FD/5D0D3B4D" Ref="#PWR?"  Part="1"
 AR Path="/5CF34646/5D0D3B4D" Ref="#PWR010"  Part="1"
+AR Path="/5D0D3B4D" Ref="#PWR010"  Part="1"
 F 0 "#PWR010" H 5900 2850 50  0001 C CNN
 F 1 "+3V3" H 5950 3200 50  0000 C CNN
@@
 AR Path="/5CF345FD/5D0D3B3E" Ref="#PWR?"  Part="1"
 AR Path="/5CF34646/5D0D3B3E" Ref="#PWR017"  Part="1"
+AR Path="/5D0D3B3E" Ref="#PWR017"  Part="1"
 F 0 "#PWR017" H 5600 3500 50  0001 C CNN
 F 1 "GND" H 5605 3577 50  0000 C CNN
@@
 AR Path="/5CF345FD/5D0D3B32" Ref="#PWR?"  Part="1"
 AR Path="/5CF34646/5D0D3B32" Ref="#PWR016"  Part="1"
+AR Path="/5D0D3B32" Ref="#PWR016"  Part="1"
 F 0 "#PWR016" H 4950 3500 50  0001 C CNN
 F 1 "GND" H 4955 3577 50  0000 C CNN
@@
 AR Path="/5CF345FD/5D0D3B2B" Ref="#PWR?"  Part="1"
 AR Path="/5CF34646/5D0D3B2B" Ref="#PWR015"  Part="1"
+AR Path="/5D0D3B2B" Ref="#PWR015"  Part="1"
 F 0 "#PWR015" H 4450 3500 50  0001 C CNN
 F 1 "GND" H 4455 3577 50  0000 C CNN
@@
 AR Path="/5CF345FD/5D0D3B20" Ref="C?"  Part="1"
 AR Path="/5CF34646/5D0D3B20" Ref="C4"  Part="1"
+AR Path="/5D0D3B20" Ref="C4"  Part="1"
 F 0 "C4" H 5892 3496 50  0000 L CNN
 F 1 "C105" H 5892 3405 50  0000 L CNN
@@
 AR Path="/5CF345FD/5D0D3B1A" Ref="U?"  Part="1"
 AR Path="/5CF34646/5D0D3B1A" Ref="U2"  Part="1"
+AR Path="/5D0D3B1A" Ref="U2"  Part="1"
 F 0 "U2" H 4950 3442 50  0000 C CNN
 F 1 "AMS1117-3.3" H 4950 3351 50  0000 C CNN
-F 2 "Package_TO_SOT_SMD:SOT-223-3_TabPin2" H 4950 3400 50  0001 C CNN
+F 2 "footprint-lib:AMS1117_SOT-223" H 4950 3400 50  0001 C CNN
 F 3 "http://www.advanced-monolithic.com/pdf/ds1117.pdf" H 5050 2950 50  0001 C CNN
 	1    4950 3200
@@
 AR Path="/5CF35582/5D10DD1D" Ref="JP?"  Part="1"
 AR Path="/5CF34646/5D10DD1D" Ref="JP4"  Part="1"
+AR Path="/5D10DD1D" Ref="JP4"  Part="1"
 F 0 "JP4" H 9900 4075 50  0000 C CNN
 F 1 "BUZZER_EN" H 9900 4166 50  0000 C CNN
@@
 AR Path="/5CF35582/5D10AC55" Ref="JP?"  Part="1"
 AR Path="/5CF34646/5D10AC55" Ref="JP3"  Part="1"
+AR Path="/5D10AC55" Ref="JP3"  Part="1"
 F 0 "JP3" H 9900 3725 50  0000 C CNN
 F 1 "OLED_EN" H 9900 3816 50  0000 C CNN
@@
 AR Path="/5CF35582/5D0FA2FF" Ref="JP?"  Part="1"
 AR Path="/5CF34646/5D0FA2FF" Ref="JP2"  Part="1"
+AR Path="/5D0FA2FF" Ref="JP2"  Part="1"
 F 0 "JP2" H 9900 3375 50  0000 C CNN
 F 1 "STM32_EN" H 9900 3466 50  0000 C CNN
@@
 AR Path="/5CF35582/5D0F1DEA" Ref="#PWR?"  Part="1"
 AR Path="/5CF34646/5D0F1DEA" Ref="#PWR06"  Part="1"
+AR Path="/5D0F1DEA" Ref="#PWR06"  Part="1"
 F 0 "#PWR06" H 10450 2650 50  0001 C CNN
 F 1 "Vws2812" V 10455 2928 50  0000 L CNN
@@
 AR Path="/5CF35582/5D0F1DE3" Ref="JP?"  Part="1"
 AR Path="/5CF34646/5D0F1DE3" Ref="JP1"  Part="1"
+AR Path="/5D0F1DE3" Ref="JP1"  Part="1"
 F 0 "JP1" H 9900 2575 50  0000 C CNN
 F 1 "WS2812_EN" H 9900 2666 50  0000 C CNN
@@
 AR Path="/5CF35582/5D0F1DDD" Ref="#PWR?"  Part="1"
 AR Path="/5CF34646/5D0F1DDD" Ref="#PWR05"  Part="1"
+AR Path="/5D0F1DDD" Ref="#PWR05"  Part="1"
 F 0 "#PWR05" H 9100 2400 50  0001 C CNN
 F 1 "+5V" H 9150 2750 50  0000 C CNN

Commit message: update footprint,
Parts:
- D1, D2: footprint LED_SMD:LED_0805_2012Metric_Pad1.15x1.40mm_HandSolder -> footprint-lib:LED_0603_1608Metric
Changed lines of the file:
@@
 F 0 "D2" V 7246 3182 50  0000 R CNN
 F 1 "LED_ORANGE" V 7155 3182 50  0000 R CNN
-F 2 "LED_SMD:LED_0805_2012Metric_Pad1.15x1.40mm_HandSolder" V 7200 3250 50  0001 C CNN
+F 2 "footprint-lib:LED_0603_1608Metric" V 7200 3250 50  0001 C CNN
 F 3 "~" V 7200 3250 50  0001 C CNN
 	1    7200 3250
@@
 F 0 "D1" V 6596 3182 50  0000 R CNN
 F 1 "LED_GREEN" V 6505 3182 50  0000 R CNN
-F 2 "LED_SMD:LED_0805_2012Metric_Pad1.15x1.40mm_HandSolder" V 6550 3250 50  0001 C CNN
+F 2 "footprint-lib:LED_0603_1608Metric" V 6550 3250 50  0001 C CNN
 F 3 "~" V 6550 3250 50  0001 C CNN
 	1    6550 3250
