File: hardware/keyboard_key.sch (KiCad schematic (older format))
At the start: 24 parts, among them SW10 KEY33, SW11 KEY41, SW12 KEY42, SW13 KEY43, SW2 KEY11, SW3 KEY12, SW4 KEY13, SW5 KEY21, SW6 KEY22, SW7 KEY23, SW8 KEY31, SW9 KEY32

Commit message: update,
Parts:
- renumbered D4 to D27, D5 to D28, D6 to D29, D7 to D30, D8 to D31, D9 to D32, D10 to D33, D11 to D34, D12 to D35, D13 to D36, D14 to D37, D15 to D38, SW6 to SW10, SW7 to SW11, SW8 to SW12, SW9 to SW13, SW10 to SW14, SW11 to SW15, SW12 to SW16, SW13 to SW17, SW2 to SW6, SW3 to SW7, SW4 to SW8, SW5 to SW9
Changed lines of the file:
@@
 $EndDescr
 $Comp
-L taobao-button:cherry_mx_no_led SW2
+L taobao-button:cherry_mx_no_led SW6
 U 1 1 5CF38962
 P 3050 850
-F 0 "SW2" H 3050 1135 50  0000 C CNN
+F 0 "SW6" H 3050 1135 50  0000 C CNN
 F 1 "KEY11" H 3050 1044 50  0000 C CNN
 F 2 "footprints-lib:cherry_mx_without_led_100H" H 3050 1050 50  0001 C CNN
@@
 $EndComp
 $Comp
-L taobao-d:D_1N4148_T4 D4
+L taobao-d:D_1N4148_T4 D27
 U 1 1 5CF3D741
 P 2750 1050
-F 0 "D4" V 2796 982 50  0000 R CNN
+F 0 "D27" V 2796 982 50  0000 R CNN
 F 1 "D_1N4148_T4" V 2705 982 50  0000 R CNN
 F 2 "Diode_SMD:D_SOD-123" V 2750 1050 50  0001 C CNN
@@
 	2750 850  2850 850
 $Comp
-L taobao-button:cherry_mx_no_led SW5
+L taobao-button:cherry_mx_no_led SW9
 U 1 1 5CF3E618
 P 3050 1650
-F 0 "SW5" H 3050 1935 50  0000 C CNN
+F 0 "SW9" H 3050 1935 50  0000 C CNN
 F 1 "KEY21" H 3050 1844 50  0000 C CNN
 F 2 "footprints-lib:cherry_mx_without_led_100H" H 3050 1850 50  0001 C CNN
@@
 $EndComp
 $Comp
-L taobao-d:D_1N4148_T4 D7
+L taobao-d:D_1N4148_T4 D30
 U 1 1 5CF3E622
 P 2750 1850
-F 0 "D7" V 2796 1782 50  0000 R CNN
+F 0 "D30" V 2796 1782 50  0000 R CNN
 F 1 "D_1N4148_T4" V 2705 1782 50  0000 R CNN
 F 2 "Diode_SMD:D_SOD-123" V 2750 1850 50  0001 C CNN
@@
 	2750 1650 2850 1650
 $Comp
-L taobao-button:cherry_mx_no_led SW8
+L taobao-button:cherry_mx_no_led SW12
 U 1 1 5CF3EEEC
 P 3050 2450
-F 0 "SW8" H 3050 2735 50  0000 C CNN
+F 0 "SW12" H 3050 2735 50  0000 C CNN
 F 1 "KEY31" H 3050 2644 50  0000 C CNN
 F 2 "footprints-lib:cherry_mx_without_led_100H" H 3050 2650 50  0001 C CNN
@@
 $EndComp
 $Comp
-L taobao-d:D_1N4148_T4 D10
+L taobao-d:D_1N4148_T4 D33
 U 1 1 5CF3EEF6
 P 2750 2650
-F 0 "D10" V 2796 2582 50  0000 R CNN
+F 0 "D33" V 2796 2582 50  0000 R CNN
 F 1 "D_1N4148_T4" V 2705 2582 50  0000 R CNN
 F 2 "Diode_SMD:D_SOD-123" V 2750 2650 50  0001 C CNN
@@
 	2750 2450 2850 2450
 $Comp
-L taobao-button:cherry_mx_no_led SW11
+L taobao-button:cherry_mx_no_led SW15
 U 1 1 5CF3EF02
 P 3050 3250
-F 0 "SW11" H 3050 3535 50  0000 C CNN
+F 0 "SW15" H 3050 3535 50  0000 C CNN
 F 1 "KEY41" H 3050 3444 50  0000 C CNN
 F 2 "footprints-lib:cherry_mx_without_led_100H" H 3050 3450 50  0001 C CNN
@@
 $EndComp
 $Comp
-L taobao-d:D_1N4148_T4 D13
+L taobao-d:D_1N4148_T4 D36
 U 1 1 5CF3EF0C
 P 2750 3450
-F 0 "D13" V 2796 3382 50  0000 R CNN
+F 0 "D36" V 2796 3382 50  0000 R CNN
 F 1 "D_1N4148_T4" V 2705 3382 50  0000 R CNN
 F 2 "Diode_SMD:D_SOD-123" V 2750 3450 50  0001 C CNN
@@
 	2750 3250 2850 3250
 $Comp
-L taobao-button:cherry_mx_no_led SW3
+L taobao-button:cherry_mx_no_led SW7
 U 1 1 5CF44234
 P 4150 850
-F 0 "SW3" H 4150 1135 50  0000 C CNN
+F 0 "SW7" H 4150 1135 50  0000 C CNN
 F 1 "KEY12" H 4150 1044 50  0000 C CNN
 F 2 "footprints-lib:cherry_mx_without_led_100H" H 4150 1050 50  0001 C CNN
@@
 $EndComp
 $Comp
-L taobao-d:D_1N4148_T4 D5
+L taobao-d:D_1N4148_T4 D28
 U 1 1 5CF4423E
 P 3850 1050
-F 0 "D5" V 3896 982 50  0000 R CNN
+F 0 "D28" V 3896 982 50  0000 R CNN
 F 1 "D_1N4148_T4" V 3805 982 50  0000 R CNN
 F 2 "Diode_SMD:D_SOD-123" V 3850 1050 50  0001 C CNN
@@
 	3850 850  3950 850
 $Comp
-L taobao-button:cherry_mx_no_led SW6
+L taobao-button:cherry_mx_no_led SW10
 U 1 1 5CF4424A
 P 4150 1650
-F 0 "SW6" H 4150 1935 50  0000 C CNN
+F 0 "SW10" H 4150 1935 50  0000 C CNN
 F 1 "KEY22" H 4150 1844 50  0000 C CNN
 F 2 "footprints-lib:cherry_mx_without_led_100H" H 4150 1850 50  0001 C CNN
@@
 $EndComp
 $Comp
-L taobao-d:D_1N4148_T4 D8
+L taobao-d:D_1N4148_T4 D31
 U 1 1 5CF44254
 P 3850 1850
-F 0 "D8" V 3896 1782 50  0000 R CNN
+F 0 "D31" V 3896 1782 50  0000 R CNN
 F 1 "D_1N4148_T4" V 3805 1782 50  0000 R CNN
 F 2 "Diode_SMD:D_SOD-123" V 3850 1850 50  0001 C CNN
@@
 	3850 1650 3950 1650
 $Comp
-L taobao-button:cherry_mx_no_led SW9
+L taobao-button:cherry_mx_no_led SW13
 U 1 1 5CF44260
 P 4150 2450
-F 0 "SW9" H 4150 2735 50  0000 C CNN
+F 0 "SW13" H 4150 2735 50  0000 C CNN
 F 1 "KEY32" H 4150 2644 50  0000 C CNN
 F 2 "footprints-lib:cherry_mx_without_led_100H" H 4150 2650 50  0001 C CNN
@@
 $EndComp
 $Comp
-L taobao-d:D_1N4148_T4 D11
+L taobao-d:D_1N4148_T4 D34
 U 1 1 5CF4426A
 P 3850 2650
-F 0 "D11" V 3896 2582 50  0000 R CNN
+F 0 "D34" V 3896 2582 50  0000 R CNN
 F 1 "D_1N4148_T4" V 3805 2582 50  0000 R CNN
 F 2 "Diode_SMD:D_SOD-123" V 3850 2650 50  0001 C CNN
@@
 	3850 2450 3950 2450
 $Comp
-L taobao-button:cherry_mx_no_led SW12
+L taobao-button:cherry_mx_no_led SW16
 U 1 1 5CF44276
 P 4150 3250
-F 0 "SW12" H 4150 3535 50  0000 C CNN
+F 0 "SW16" H 4150 3535 50  0000 C CNN
 F 1 "KEY42" H 4150 3444 50  0000 C CNN
 F 2 "footprints-lib:cherry_mx_without_led_100H" H 4150 3450 50  0001 C CNN
@@
 $EndComp
 $Comp
-L taobao-d:D_1N4148_T4 D14
+L taobao-d:D_1N4148_T4 D37
 U 1 1 5CF44280
 P 3850 3450
-F 0 "D14" V 3896 3382 50  0000 R CNN
+F 0 "D37" V 3896 3382 50  0000 R CNN
 F 1 "D_1N4148_T4" V 3805 3382 50  0000 R CNN
 F 2 "Diode_SMD:D_SOD-123" V 3850 3450 50  0001 C CNN
@@
 	3850 3250 3950 3250
 $Comp
-L taobao-button:cherry_mx_no_led SW4
+L taobao-button:cherry_mx_no_led SW8
 U 1 1 5CF46C3C
 P 5150 850
-F 0 "SW4" H 5150 1135 50  0000 C CNN
+F 0 "SW8" H 5150 1135 50  0000 C CNN
 F 1 "KEY13" H 5150 1044 50  0000 C CNN
 F 2 "footprints-lib:cherry_mx_without_led_100H" H 5150 1050 50  0001 C CNN
@@
 $EndComp
 $Comp
-L taobao-d:D_1N4148_T4 D6
+L taobao-d:D_1N4148_T4 D29
 U 1 1 5CF46C46
 P 4850 1050
-F 0 "D6" V 4896 982 50  0000 R CNN
+F 0 "D29" V 4896 982 50  0000 R CNN
 F 1 "D_1N4148_T4" V 4805 982 50  0000 R CNN
 F 2 "Diode_SMD:D_SOD-123" V 4850 1050 50  0001 C CNN
@@
 	4850 850  4950 850
 $Comp
-L taobao-button:cherry_mx_no_led SW7
+L taobao-button:cherry_mx_no_led SW11
 U 1 1 5CF46C52
 P 5150 1650
-F 0 "SW7" H 5150 1935 50  0000 C CNN
+F 0 "SW11" H 5150 1935 50  0000 C CNN
 F 1 "KEY23" H 5150 1844 50  0000 C CNN
 F 2 "footprints-lib:cherry_mx_without_led_100H" H 5150 1850 50  0001 C CNN
@@
 $EndComp
 $Comp
-L taobao-d:D_1N4148_T4 D9
+L taobao-d:D_1N4148_T4 D32
 U 1 1 5CF46C5C
 P 4850 1850
-F 0 "D9" V 4896 1782 50  0000 R CNN
+F 0 "D32" V 4896 1782 50  0000 R CNN
 F 1 "D_1N4148_T4" V 4805 1782 50  0000 R CNN
 F 2 "Diode_SMD:D_SOD-123" V 4850 1850 50  0001 C CNN
@@
 	4850 1650 4950 1650
 $Comp
-L taobao-button:cherry_mx_no_led SW10
+L taobao-button:cherry_mx_no_led SW14
 U 1 1 5CF46C68
 P 5150 2450
-F 0 "SW10" H 5150 2735 50  0000 C CNN
+F 0 "SW14" H 5150 2735 50  0000 C CNN
 F 1 "KEY33" H 5150 2644 50  0000 C CNN
 F 2 "footprints-lib:cherry_mx_without_led_100H" H 5150 2650 50  0001 C CNN
@@
 $EndComp
 $Comp
-L taobao-d:D_1N4148_T4 D12
+L taobao-d:D_1N4148_T4 D35
 U 1 1 5CF46C72
 P 4850 2650
-F 0 "D12" V 4896 2582 50  0000 R CNN
+F 0 "D35" V 4896 2582 50  0000 R CNN
 F 1 "D_1N4148_T4" V 4805 2582 50  0000 R CNN
 F 2 "Diode_SMD:D_SOD-123" V 4850 2650 50  0001 C CNN
@@
 	4850 2450 4950 2450
 $Comp
-L taobao-button:cherry_mx_no_led SW13
+L taobao-button:cherry_mx_no_led SW17
 U 1 1 5CF46C7E
 P 5150 3250
-F 0 "SW13" H 5150 3535 50  0000 C CNN
+F 0 "SW17" H 5150 3535 50  0000 C CNN
 F 1 "KEY43" H 5150 3444 50  0000 C CNN
 F 2 "footprints-lib:cherry_mx_without_led_100H" H 5150 3450 50  0001 C CNN
@@
 $EndComp
 $Comp
-L taobao-d:D_1N4148_T4 D15
+L taobao-d:D_1N4148_T4 D38
 U 1 1 5CF46C88
 P 4850 3450
-F 0 "D15" V 4896 3382 50  0000 R CNN
+F 0 "D38" V 4896 3382 50  0000 R CNN
 F 1 "D_1N4148_T4" V 4805 3382 50  0000 R CNN
 F 2 "Diode_SMD:D_SOD-123" V 4850 3450 50  0001 C CNN

Commit message: update footprint,
Parts:
- SW10, SW11, SW12, SW13, SW14, SW15, SW16, SW17, SW6, SW7, SW8, SW9: footprint footprints-lib:cherry_mx_without_led_100H -> footprint-lib:cherry_mx_without_led_100H
Changed lines of the file:
@@
 F 0 "SW6" H 3050 1135 50  0000 C CNN
 F 1 "KEY11" H 3050 1044 50  0000 C CNN
-F 2 "footprints-lib:cherry_mx_without_led_100H" H 3050 1050 50  0001 C CNN
+F 2 "footprint-lib:cherry_mx_without_led_100H" H 3050 1050 50  0001 C CNN
 F 3 "~" H 3050 1050 50  0001 C CNN
 	1    3050 850
@@
 F 0 "SW9" H 3050 1935 50  0000 C CNN
 F 1 "KEY21" H 3050 1844 50  0000 C CNN
-F 2 "footprints-lib:cherry_mx_without_led_100H" H 3050 1850 50  0001 C CNN
+F 2 "footprint-lib:cherry_mx_without_led_100H" H 3050 1850 50  0001 C CNN
 F 3 "~" H 3050 1850 50  0001 C CNN
 	1    3050 1650
@@
 F 0 "SW12" H 3050 2735 50  0000 C CNN
 F 1 "KEY31" H 3050 2644 50  0000 C CNN
-F 2 "footprints-lib:cherry_mx_without_led_100H" H 3050 2650 50  0001 C CNN
+F 2 "footprint-lib:cherry_mx_without_led_100H" H 3050 2650 50  0001 C CNN
 F 3 "~" H 3050 2650 50  0001 C CNN
 	1    3050 2450
@@
 F 0 "SW15" H 3050 3535 50  0000 C CNN
 F 1 "KEY41" H 3050 3444 50  0000 C CNN
-F 2 "footprints-lib:cherry_mx_without_led_100H" H 3050 3450 50  0001 C CNN
+F 2 "footprint-lib:cherry_mx_without_led_100H" H 3050 3450 50  0001 C CNN
 F 3 "~" H 3050 3450 50  0001 C CNN
 	1    3050 3250
@@
 F 0 "SW7" H 4150 1135 50  0000 C CNN
 F 1 "KEY12" H 4150 1044 50  0000 C CNN
-F 2 "footprints-lib:cherry_mx_without_led_100H" H 4150 1050 50  0001 C CNN
+F 2 "footprint-lib:cherry_mx_without_led_100H" H 4150 1050 50  0001 C CNN
 F 3 "~" H 4150 1050 50  0001 C CNN
 	1    4150 850
@@
 F 0 "SW10" H 4150 1935 50  0000 C CNN
 F 1 "KEY22" H 4150 1844 50  0000 C CNN
-F 2 "footprints-lib:cherry_mx_without_led_100H" H 4150 1850 50  0001 C CNN
+F 2 "footprint-lib:cherry_mx_without_led_100H" H 4150 1850 50  0001 C CNN
 F 3 "~" H 4150 1850 50  0001 C CNN
 	1    4150 1650
@@
 F 0 "SW13" H 4150 2735 50  0000 C CNN
 F 1 "KEY32" H 4150 2644 50  0000 C CNN
-F 2 "footprints-lib:cherry_mx_without_led_100H" H 4150 2650 50  0001 C CNN
+F 2 "footprint-lib:cherry_mx_without_led_100H" H 4150 2650 50  0001 C CNN
 F 3 "~" H 4150 2650 50  0001 C CNN
 	1    4150 2450
@@
 F 0 "SW16" H 4150 3535 50  0000 C CNN
 F 1 "KEY42" H 4150 3444 50  0000 C CNN
-F 2 "footprints-lib:cherry_mx_without_led_100H" H 4150 3450 50  0001 C CNN
+F 2 "footprint-lib:cherry_mx_without_led_100H" H 4150 3450 50  0001 C CNN
 F 3 "~" H 4150 3450 50  0001 C CNN
 	1    4150 3250
@@
 F 0 "SW8" H 5150 1135 50  0000 C CNN
 F 1 "KEY13" H 5150 1044 50  0000 C CNN
-F 2 "footprints-lib:cherry_mx_without_led_100H" H 5150 1050 50  0001 C CNN
+F 2 "footprint-lib:cherry_mx_without_led_100H" H 5150 1050 50  0001 C CNN
 F 3 "~" H 5150 1050 50  0001 C CNN
 	1    5150 850
@@
 F 0 "SW11" H 5150 1935 50  0000 C CNN
 F 1 "KEY23" H 5150 1844 50  0000 C CNN
-F 2 "footprints-lib:cherry_mx_without_led_100H" H 5150 1850 50  0001 C CNN
+F 2 "footprint-lib:cherry_mx_without_led_100H" H 5150 1850 50  0001 C CNN
 F 3 "~" H 5150 1850 50  0001 C CNN
 	1    5150 1650
@@
 F 0 "SW14" H 5150 2735 50  0000 C CNN
 F 1 "KEY33" H 5150 2644 50  0000 C CNN
-F 2 "footprints-lib:cherry_mx_without_led_100H" H 5150 2650 50  0001 C CNN
+F 2 "footprint-lib:cherry_mx_without_led_100H" H 5150 2650 50  0001 C CNN
 F 3 "~" H 5150 2650 50  0001 C CNN
 	1    5150 2450
@@
 F 0 "SW17" H 5150 3535 50  0000 C CNN
 F 1 "KEY43" H 5150 3444 50  0000 C CNN
-F 2 "footprints-lib:cherry_mx_without_led_100H" H 5150 3450 50  0001 C CNN
+F 2 "footprint-lib:cherry_mx_without_led_100H" H 5150 3450 50  0001 C CNN
 F 3 "~" H 5150 3450 50  0001 C CNN
 	1    5150 3250

Commit message: update route,
Parts:
- removed D36, D37, D38: D_1N4148_T4, Diode_SMD:D_SOD-123, symbol taobao-d:D_1N4148_T4
- removed SW15: KEY41, footprint-lib:cherry_mx_without_led_100H, symbol taobao-button:cherry_mx_no_led
- removed SW16: KEY42, footprint-lib:cherry_mx_without_led_100H, symbol taobao-button:cherry_mx_no_led
- removed SW17: KEY43, footprint-lib:cherry_mx_without_led_100H, symbol taobao-button:cherry_mx_no_led
Changed lines of the file:
@@
 $Descr User 8500 5500
 encoding utf-8
-Sheet 11 13
+Sheet 1 13
 Title ""
 Date ""
@@
 	2750 2450 2850 2450
 $Comp
-L taobao-button:cherry_mx_no_led SW15
-U 1 1 5CF3EF02
-P 3050 3250
-F 0 "SW15" H 3050 3535 50  0000 C CNN
-F 1 "KEY41" H 3050 3444 50  0000 C CNN
-F 2 "footprint-lib:cherry_mx_without_led_100H" H 3050 3450 50  0001 C CNN
-F 3 "~" H 3050 3450 50  0001 C CNN
-	1    3050 3250
-	1    0    0    -1
-$EndComp
-$Comp
-L taobao-d:D_1N4148_T4 D36
-U 1 1 5CF3EF0C
-P 2750 3450
-F 0 "D36" V 2796 3382 50  0000 R CNN
-F 1 "D_1N4148_T4" V 2705 3382 50  0000 R CNN
-F 2 "Diode_SMD:D_SOD-123" V 2750 3450 50  0001 C CNN
-F 3 "~" V 2750 3450 50  0001 C CNN
-	1    2750 3450
-	0    -1   -1   0
-$EndComp
-Wire Wire Line
-	2750 3350 2750 3250
-Wire Wire Line
-	2750 3250 2850 3250
-$Comp
 L taobao-button:cherry_mx_no_led SW7
 U 1 1 5CF44234
@@
 	3850 2450 3950 2450
 $Comp
-L taobao-button:cherry_mx_no_led SW16
-U 1 1 5CF44276
-P 4150 3250
-F 0 "SW16" H 4150 3535 50  0000 C CNN
-F 1 "KEY42" H 4150 3444 50  0000 C CNN
-F 2 "footprint-lib:cherry_mx_without_led_100H" H 4150 3450 50  0001 C CNN
-F 3 "~" H 4150 3450 50  0001 C CNN
-	1    4150 3250
-	1    0    0    -1
-$EndComp
-$Comp
-L taobao-d:D_1N4148_T4 D37
-U 1 1 5CF44280
-P 3850 3450
-F 0 "D37" V 3896 3382 50  0000 R CNN
-F 1 "D_1N4148_T4" V 3805 3382 50  0000 R CNN
-F 2 "Diode_SMD:D_SOD-123" V 3850 3450 50  0001 C CNN
-F 3 "~" V 3850 3450 50  0001 C CNN
-	1    3850 3450
-	0    -1   -1   0
-$EndComp
-Wire Wire Line
-	3850 3350 3850 3250
-Wire Wire Line
-	3850 3250 3950 3250
-$Comp
 L taobao-button:cherry_mx_no_led SW8
 U 1 1 5CF46C3C
@@
 Wire Wire Line
 	4850 2450 4950 2450
-$Comp
-L taobao-button:cherry_mx_no_led SW17
-U 1 1 5CF46C7E
-P 5150 3250
-F 0 "SW17" H 5150 3535 50  0000 C CNN
-F 1 "KEY43" H 5150 3444 50  0000 C CNN
-F 2 "footprint-lib:cherry_mx_without_led_100H" H 5150 3450 50  0001 C CNN
-F 3 "~" H 5150 3450 50  0001 C CNN
-	1    5150 3250
-	1    0    0    -1
-$EndComp
-$Comp
-L taobao-d:D_1N4148_T4 D38
-U 1 1 5CF46C88
-P 4850 3450
-F 0 "D38" V 4896 3382 50  0000 R CNN
-F 1 "D_1N4148_T4" V 4805 3382 50  0000 R CNN
-F 2 "Diode_SMD:D_SOD-123" V 4850 3450 50  0001 C CNN
-F 3 "~" V 4850 3450 50  0001 C CNN
-	1    4850 3450
-	0    -1   -1   0
-$EndComp
-Wire Wire Line
-	4850 3350 4850 3250
-Wire Wire Line
-	4850 3250 4950 3250
 Text Label 1000 750  0    50   ~ 0
 ROW1
@@
 Text Label 2000 2850 0    50   ~ 0
 ROW3
-Text Label 2000 3700 0    50   ~ 0
-ROW4
-Wire Wire Line
-	2000 3700 2750 3700
-Wire Wire Line
-	2750 3700 2750 3550
-Wire Wire Line
-	2750 3700 3850 3700
-Wire Wire Line
-	3850 3700 3850 3550
-Connection ~ 2750 3700
-Wire Wire Line
-	3850 3700 4850 3700
-Wire Wire Line
-	4850 3700 4850 3550
-Connection ~ 3850 3700
 Wire Wire Line
 	2000 2850 2750 2850
@@
 Connection ~ 3400 1650
 Wire Wire Line
-	3400 3250 3250 3250
-Wire Wire Line
 	3400 1650 3400 2450
-Connection ~ 3400 2450
-Wire Wire Line
-	3400 2450 3400 3250
 Wire Wire Line
 	4450 1650 4350 1650
@@
 Connection ~ 4450 1650
 Wire Wire Line
-	4450 3250 4350 3250
-Wire Wire Line
 	4450 1650 4450 2450
-Connection ~ 4450 2450
-Wire Wire Line
-	4450 2450 4450 3250
 Wire Wire Line
 	5450 1650 5350 1650
@@
 Connection ~ 5450 1650
 Wire Wire Line
-	5450 3250 5350 3250
-Wire Wire Line
 	5450 1650 5450 2450
-Connection ~ 5450 2450
-Wire Wire Line
-	5450 2450 5450 3250
 $EndSCHEMATC
