File: hardware/oled.sch (KiCad schematic (older format))
At the start: 3 parts, among them U2 SSD1306-OLED-I2C

Commit message: update,
Parts:
- added J?: I2C_HEADER,2.54, Connector_PinHeader_2.54mm:PinHeader_1x02_P2.54mm_Vertical, symbol taobao-components:I2C_HEADER,2.54
Connections:
- net SCL: now also J?.SCL
- net SDA: now also J?.SDA
Changed lines of the file:
@@
 $Descr User 8500 5500
 encoding utf-8
-Sheet 3 13
+Sheet 2 13
 Title ""
 Date ""
@@
 Wire Wire Line
 	2450 1700 2450 1950
+$Comp
+L taobao-components:I2C_HEADER,2.54 J?
+U 1 1 5D459F93
+P 900 1250
+F 0 "J?" H 872 1182 50  0000 R CNN
+F 1 "I2C_HEADER,2.54" H 872 1273 50  0000 R CNN
+F 2 "Connector_PinHeader_2.54mm:PinHeader_1x02_P2.54mm_Vertical" H 900 850 50  0001 C CNN
+F 3 "" H 900 1200 50  0001 C CNN
+	1    900  1250
+	1    0    0    1
+$EndComp
+Text Label 1600 1300 2    50   ~ 0
+SDA
+Text Label 1600 1200 2    50   ~ 0
+SCL
+Wire Wire Line
+	1100 1200 1600 1200
+Wire Wire Line
+	1600 1300 1100 1300
 $EndSCHEMATC

Commit message: update,
Parts:
- added C?: CP10uf,16V, Capacitor_SMD:CP_Elec_4x5.3, symbol taobao-cp:CP10uf,16V
- gave numbers to parts that had none: 1
Connections:
- net GND: now also C?.2
- net Voled: now also C?.1
Changed lines of the file:
@@
 	2450 1700 2450 1950
 $Comp
-L taobao-components:I2C_HEADER,2.54 J?
+L taobao-components:I2C_HEADER,2.54 J8
 U 1 1 5D459F93
 P 900 1250
-F 0 "J?" H 872 1182 50  0000 R CNN
+F 0 "J8" H 872 1182 50  0000 R CNN
 F 1 "I2C_HEADER,2.54" H 872 1273 50  0000 R CNN
 F 2 "Connector_PinHeader_2.54mm:PinHeader_1x02_P2.54mm_Vertical" H 900 850 50  0001 C CNN
@@
 Wire Wire Line
 	1600 1300 1100 1300
+$Comp
+L my_power:Voled #PWR?
+U 1 1 5D6199EC
+P 2300 1200
+F 0 "#PWR?" H 2300 1050 50  0001 C CNN
+F 1 "Voled" H 2305 1373 50  0000 C CNN
+F 2 "" H 2300 1200 50  0001 C CNN
+F 3 "" H 2300 1200 50  0001 C CNN
+	1    2300 1200
+	0    -1   -1   0
+$EndComp
+$Comp
+L taobao-cp:CP10uf,16V C?
+U 1 1 5D619F23
+P 2500 1200
+F 0 "C?" V 2725 1200 50  0000 C CNN
+F 1 "CP10uf,16V" V 2634 1200 50  0000 C CNN
+F 2 "Capacitor_SMD:CP_Elec_4x5.3" H 2500 1200 50  0001 C CNN
+F 3 "~" H 2500 1200 50  0001 C CNN
+	1    2500 1200
+	0    -1   -1   0
+$EndComp
+$Comp
+L power:GND #PWR?
+U 1 1 5D61A2A1
+P 2700 1200
+F 0 "#PWR?" H 2700 950 50  0001 C CNN
+F 1 "GND" H 2705 1027 50  0000 C CNN
+F 2 "" H 2700 1200 50  0001 C CNN
+F 3 "" H 2700 1200 50  0001 C CNN
+	1    2700 1200
+	0    -1   -1   0
+$EndComp
+Wire Wire Line
+	2600 1200 2700 1200
+Wire Wire Line
+	2300 1200 2400 1200
 $EndSCHEMATC

Commit message: update,
Parts:
- gave numbers to parts that had none: 1
Changed lines of the file:
@@
 	1600 1300 1100 1300
 $Comp
-L my_power:Voled #PWR?
+L my_power:Voled #PWR0167
 U 1 1 5D6199EC
 P 2300 1200
-F 0 "#PWR?" H 2300 1050 50  0001 C CNN
+F 0 "#PWR0167" H 2300 1050 50  0001 C CNN
 F 1 "Voled" H 2305 1373 50  0000 C CNN
 F 2 "" H 2300 1200 50  0001 C CNN
@@
 $EndComp
 $Comp
-L taobao-cp:CP10uf,16V C?
+L taobao-cp:CP10uf,16V C57
 U 1 1 5D619F23
 P 2500 1200
-F 0 "C?" V 2725 1200 50  0000 C CNN
+F 0 "C57" V 2725 1200 50  0000 C CNN
 F 1 "CP10uf,16V" V 2634 1200 50  0000 C CNN
 F 2 "Capacitor_SMD:CP_Elec_4x5.3" H 2500 1200 50  0001 C CNN
@@
 $EndComp
 $Comp
-L power:GND #PWR?
+L power:GND #PWR0168
 U 1 1 5D61A2A1
 P 2700 1200
-F 0 "#PWR?" H 2700 950 50  0001 C CNN
+F 0 "#PWR0168" H 2700 950 50  0001 C CNN
 F 1 "GND" H 2705 1027 50  0000 C CNN
 F 2 "" H 2700 1200 50  0001 C CNN

Commit message: update,
Parts:
- renumbered C57 to C1, J8 to J1, R11 to R1, R12 to R2, U2 to U1
Changed lines of the file:
@@
 $EndBitmap
 $Comp
-L taobao-board:SSD1306-OLED-I2C U2
+L taobao-board:SSD1306-OLED-I2C U1
 U 1 1 5D09D217
 P 2050 2250
-F 0 "U2" H 2167 2765 50  0000 C CNN
+F 0 "U1" H 2167 2765 50  0000 C CNN
 F 1 "SSD1306-OLED-I2C" H 2167 2674 50  0000 C CNN
 F 2 "" H 2050 2100 50  0001 C CNN
@@
 $EndComp
 $Comp
-L power:GND #PWR019
+L power:GND #PWR04
 U 1 1 5D09E684
 P 2400 2500
-F 0 "#PWR019" H 2400 2250 50  0001 C CNN
+F 0 "#PWR04" H 2400 2250 50  0001 C CNN
 F 1 "GND" H 2405 2327 50  0000 C CNN
 F 2 "" H 2400 2500 50  0001 C CNN
@@
 $EndComp
 $Comp
-L taobao-r:R472,0603 R11
+L taobao-r:R472,0603 R1
 U 1 1 5D09E950
 P 2750 2100
-F 0 "R11" V 2554 2100 50  0000 C CNN
+F 0 "R1" V 2554 2100 50  0000 C CNN
 F 1 "R472,0603" V 2645 2100 50  0000 C CNN
 F 2 "Resistor_SMD:R_0603_1608Metric_Pad1.05x0.95mm_HandSolder" H 2750 2100 50  0001 C CNN
@@
 $EndComp
 $Comp
-L taobao-r:R472,0603 R12
+L taobao-r:R472,0603 R2
 U 1 1 5D09EC8C
 P 2850 2100
-F 0 "R12" V 2654 2100 50  0000 C CNN
+F 0 "R2" V 2654 2100 50  0000 C CNN
 F 1 "R472,0603" V 2745 2100 50  0000 C CNN
 F 2 "Resistor_SMD:R_0603_1608Metric_Pad1.05x0.95mm_HandSolder" H 2850 2100 50  0001 C CNN
@@
 	2850 2400 3250 2400
 $Comp
-L my_power:Voled #PWR018
+L my_power:Voled #PWR03
 U 1 1 5D0FFF44
 P 2450 1700
-F 0 "#PWR018" H 2450 1550 50  0001 C CNN
+F 0 "#PWR03" H 2450 1550 50  0001 C CNN
 F 1 "Voled" H 2455 1873 50  0000 C CNN
 F 2 "" H 2450 1700 50  0001 C CNN
@@
 	2450 1700 2450 1950
 $Comp
-L taobao-components:I2C_HEADER,2.54 J8
+L taobao-components:I2C_HEADER,2.54 J1
 U 1 1 5D459F93
 P 900 1250
-F 0 "J8" H 872 1182 50  0000 R CNN
+F 0 "J1" H 872 1182 50  0000 R CNN
 F 1 "I2C_HEADER,2.54" H 872 1273 50  0000 R CNN
 F 2 "Connector_PinHeader_2.54mm:PinHeader_1x02_P2.54mm_Vertical" H 900 850 50  0001 C CNN
@@
 	1600 1300 1100 1300
 $Comp
-L my_power:Voled #PWR0167
+L my_power:Voled #PWR01
 U 1 1 5D6199EC
 P 2300 1200
-F 0 "#PWR0167" H 2300 1050 50  0001 C CNN
+F 0 "#PWR01" H 2300 1050 50  0001 C CNN
 F 1 "Voled" H 2305 1373 50  0000 C CNN
 F 2 "" H 2300 1200 50  0001 C CNN
@@
 $EndComp
 $Comp
-L taobao-cp:CP10uf,16V C57
+L taobao-cp:CP10uf,16V C1
 U 1 1 5D619F23
 P 2500 1200
-F 0 "C57" V 2725 1200 50  0000 C CNN
+F 0 "C1" V 2725 1200 50  0000 C CNN
 F 1 "CP10uf,16V" V 2634 1200 50  0000 C CNN
 F 2 "Capacitor_SMD:CP_Elec_4x5.3" H 2500 1200 50  0001 C CNN
@@
 $EndComp
 $Comp
-L power:GND #PWR0168
+L power:GND #PWR02
 U 1 1 5D61A2A1
 P 2700 1200
-F 0 "#PWR0168" H 2700 950 50  0001 C CNN
+F 0 "#PWR02" H 2700 950 50  0001 C CNN
 F 1 "GND" H 2705 1027 50  0000 C CNN
 F 2 "" H 2700 1200 50  0001 C CNN
