File: hardware/oled.sch (KiCad schematic (older format))
At the start: 5 parts, among them J1 I2C_HEADER,2.54, U1 SSD1306-OLED-I2C

Commit message: update footprint,
Parts:
- J1: footprint Connector_PinHeader_2.54mm:PinHeader_1x02_P2.54mm_Vertical -> footprint-lib:I2C_DEBUG,2.54
- U1: footprint (none) -> footprint-lib:SSD1306_OLED-0.91-128x32_4pin
Changed lines of the file:
@@
 F 0 "U1" H 2167 2765 50  0000 C CNN
 F 1 "SSD1306-OLED-I2C" H 2167 2674 50  0000 C CNN
-F 2 "" H 2050 2100 50  0001 C CNN
+F 2 "footprint-lib:SSD1306_OLED-0.91-128x32_4pin" H 2050 2100 50  0001 C CNN
 F 3 "" H 2050 2100 50  0001 C CNN
 	1    2050 2250
@@
 F 0 "J1" H 872 1182 50  0000 R CNN
 F 1 "I2C_HEADER,2.54" H 872 1273 50  0000 R CNN
-F 2 "Connector_PinHeader_2.54mm:PinHeader_1x02_P2.54mm_Vertical" H 900 850 50  0001 C CNN
+F 2 "footprint-lib:I2C_DEBUG,2.54" H 900 850 50  0001 C CNN
 F 3 "" H 900 1200 50  0001 C CNN
 	1    900  1250
