File: hardware/rot_enc.sch (KiCad schematic (older format))
At the start: 8 parts

Commit message: update for cherry key,wd
Parts:
- SW?: value EC11_VERTICAL -> ROT1
Changed lines of the file:
@@
 AR Path="/5CFF7883/5D0A34E5" Ref="SW?"  Part="1"
 F 0 "SW?" H 3900 2300 50  0000 C CNN
-F 1 "EC11_VERTICAL" H 3900 2400 50  0000 C CNN
+F 1 "ROT1" H 3900 2400 50  0000 C CNN
 F 2 "footprint-lib:RotaryEncoder_Alps_EC11E_Vertical_H20mm" H 3900 2350 50  0001 C CNN
 F 3 "https://item.taobao.com/item.htm?spm=a1z09.2.0.0.61152e8dxnonTp&id=532637189592&_u=rot8j1n8a4b" H 3900 2960 50  0001 C CNN

Commit message: update,
Parts:
- removed C? (x2): C104,0603, Capacitor_SMD:C_0603_1608Metric_Pad1.05x0.95mm_HandSolder, symbol taobao-c:C104,0603
- removed R? (x2): R273,0603, Resistor_SMD:R_0603_1608Metric_Pad1.05x0.95mm_HandSolder, symbol taobao-r:R273,0603
- added C23, C24: C104,0603, Capacitor_SMD:C_0603_1608Metric_Pad1.05x0.95mm_HandSolder, symbol taobao-c:C104,0603
- added R18, R19: R273,0603, Resistor_SMD:R_0603_1608Metric_Pad1.05x0.95mm_HandSolder, symbol taobao-r:R273,0603
- gave numbers to parts that had none: 4
Connections:
- net B: now also C23.1, R18.2
- net GND: now also C23.2, C24.2
- net SW_OUT: now also C24.1, R19.2
- net at SW14.A: now also R18.1
- net at SW14.D: now also R19.1
Changed lines of the file:
@@
 $EndDescr
 $Comp
-L taobao-components:EC11_VERTICAL SW?
+L taobao-components:EC11_VERTICAL SW14
 U 1 1 5D0A34E5
 P 3900 2700
-AR Path="/5CF34744/5D0A34E5" Ref="SW?"  Part="1"
+AR Path="/5CF34744/5D0A34E5" Ref="SW14"  Part="1"
 AR Path="/5CFF7883/5D0A34E5" Ref="SW?"  Part="1"
-F 0 "SW?" H 3900 2300 50  0000 C CNN
+F 0 "SW14" H 3900 2300 50  0000 C CNN
 F 1 "ROT1" H 3900 2400 50  0000 C CNN
 F 2 "footprint-lib:RotaryEncoder_Alps_EC11E_Vertical_H20mm" H 3900 2350 50  0001 C CNN
@@
 $EndBitmap
 $Comp
-L taobao-r:R273,0603 R?
+L taobao-r:R273,0603 R17
 U 1 1 5CED60AF
 P 3150 2300
-AR Path="/5CF34744/5CED60AF" Ref="R?"  Part="1"
+AR Path="/5CF34744/5CED60AF" Ref="R17"  Part="1"
 AR Path="/5CFF7883/5CED60AF" Ref="R?"  Part="1"
-F 0 "R?" V 2900 2300 50  0000 C CNN
+F 0 "R17" V 2900 2300 50  0000 C CNN
 F 1 "R273,0603" V 3000 2300 50  0000 C CNN
 F 2 "Resistor_SMD:R_0603_1608Metric_Pad1.05x0.95mm_HandSolder" H 3150 2300 50  0001 C CNN
@@
 $EndComp
 $Comp
-L taobao-r:R273,0603 R?
-U 1 1 5CED6622
+L taobao-r:R273,0603 R18
+U 1 1 5D32A3BC
 P 3150 2800
-AR Path="/5CF34744/5CED6622" Ref="R?"  Part="1"
-AR Path="/5CFF7883/5CED6622" Ref="R?"  Part="1"
-F 0 "R?" V 2900 2800 50  0000 C CNN
+AR Path="/5CF34744/5D32A3BC" Ref="R18"  Part="1"
+AR Path="/5CFF7883/5D32A3BC" Ref="R?"  Part="1"
+F 0 "R18" V 2900 2800 50  0000 C CNN
 F 1 "R273,0603" V 3000 2800 50  0000 C CNN
 F 2 "Resistor_SMD:R_0603_1608Metric_Pad1.05x0.95mm_HandSolder" H 3150 2800 50  0001 C CNN
@@
 $EndComp
 $Comp
-L taobao-r:R273,0603 R?
-U 1 1 5CED67EF
+L taobao-r:R273,0603 R19
+U 1 1 5D32A3BD
 P 3150 3250
-AR Path="/5CF34744/5CED67EF" Ref="R?"  Part="1"
-AR Path="/5CFF7883/5CED67EF" Ref="R?"  Part="1"
-F 0 "R?" V 2900 3250 50  0000 C CNN
+AR Path="/5CF34744/5D32A3BD" Ref="R19"  Part="1"
+AR Path="/5CFF7883/5D32A3BD" Ref="R?"  Part="1"
+F 0 "R19" V 2900 3250 50  0000 C CNN
 F 1 "R273,0603" V 3000 3250 50  0000 C CNN
 F 2 "Resistor_SMD:R_0603_1608Metric_Pad1.05x0.95mm_HandSolder" H 3150 3250 50  0001 C CNN
@@
 $EndComp
 $Comp
-L taobao-c:C104,0603 C?
-U 1 1 5CED6CD1
+L taobao-c:C104,0603 C24
+U 1 1 5D32A3BE
 P 2800 3450
-AR Path="/5CF34744/5CED6CD1" Ref="C?"  Part="1"
-AR Path="/5CFF7883/5CED6CD1" Ref="C?"  Part="1"
-F 0 "C?" H 2900 3500 50  0000 L CNN
+AR Path="/5CF34744/5D32A3BE" Ref="C24"  Part="1"
+AR Path="/5CFF7883/5D32A3BE" Ref="C?"  Part="1"
+F 0 "C24" H 2900 3500 50  0000 L CNN
 F 1 "C104,0603" H 2900 3450 50  0000 L CNN
 F 2 "Capacitor_SMD:C_0603_1608Metric_Pad1.05x0.95mm_HandSolder" H 2800 3450 50  0001 C CNN
@@
 $EndComp
 $Comp
-L taobao-c:C104,0603 C?
-U 1 1 5CED7298
+L taobao-c:C104,0603 C23
+U 1 1 5D32A3BF
 P 2800 2950
-AR Path="/5CF34744/5CED7298" Ref="C?"  Part="1"
-AR Path="/5CFF7883/5CED7298" Ref="C?"  Part="1"
-F 0 "C?" H 2900 3000 50  0000 L CNN
+AR Path="/5CF34744/5D32A3BF" Ref="C23"  Part="1"
+AR Path="/5CFF7883/5D32A3BF" Ref="C?"  Part="1"
+F 0 "C23" H 2900 3000 50  0000 L CNN
 F 1 "C104,0603" H 2900 2950 50  0000 L CNN
 F 2 "Capacitor_SMD:C_0603_1608Metric_Pad1.05x0.95mm_HandSolder" H 2800 2950 50  0001 C CNN
@@
 $EndComp
 $Comp
-L taobao-c:C104,0603 C?
+L taobao-c:C104,0603 C22
 U 1 1 5CED75A5
 P 2800 2500
-AR Path="/5CF34744/5CED75A5" Ref="C?"  Part="1"
+AR Path="/5CF34744/5CED75A5" Ref="C22"  Part="1"
 AR Path="/5CFF7883/5CED75A5" Ref="C?"  Part="1"
-F 0 "C?" H 2900 2550 50  0000 L CNN
+F 0 "C22" H 2900 2550 50  0000 L CNN
 F 1 "C104,0603" H 2900 2500 50  0000 L CNN
 F 2 "Capacitor_SMD:C_0603_1608Metric_Pad1.05x0.95mm_HandSolder" H 2800 2500 50  0001 C CNN
@@
 	2800 3250 2800 3350
 $Comp
-L power:GND #PWR?
+L power:GND #PWR042
 U 1 1 5CED86F3
 P 2800 2650
-AR Path="/5CF34744/5CED86F3" Ref="#PWR?"  Part="1"
+AR Path="/5CF34744/5CED86F3" Ref="#PWR042"  Part="1"
 AR Path="/5CFF7883/5CED86F3" Ref="#PWR?"  Part="1"
-F 0 "#PWR?" H 2800 2400 50  0001 C CNN
+F 0 "#PWR042" H 2800 2400 50  0001 C CNN
 F 1 "GND" H 2850 2450 50  0000 C CNN
 F 2 "" H 2800 2650 50  0001 C CNN
@@
 	2800 2650 2800 2600
 $Comp
-L power:GND #PWR?
-U 1 1 5CED8B04
+L power:GND #PWR044
+U 1 1 5D32A3C2
 P 2800 3100
-AR Path="/5CF34744/5CED8B04" Ref="#PWR?"  Part="1"
-AR Path="/5CFF7883/5CED8B04" Ref="#PWR?"  Part="1"
-F 0 "#PWR?" H 2800 2850 50  0001 C CNN
+AR Path="/5CF34744/5D32A3C2" Ref="#PWR044"  Part="1"
+AR Path="/5CFF7883/5D32A3C2" Ref="#PWR?"  Part="1"
+F 0 "#PWR044" H 2800 2850 50  0001 C CNN
 F 1 "GND" H 2850 2900 50  0000 C CNN
 F 2 "" H 2800 3100 50  0001 C CNN
@@
 	2800 3100 2800 3050
 $Comp
-L power:GND #PWR?
+L power:GND #PWR045
 U 1 1 5CED8F95
 P 2800 3600
-AR Path="/5CF34744/5CED8F95" Ref="#PWR?"  Part="1"
+AR Path="/5CF34744/5CED8F95" Ref="#PWR045"  Part="1"
 AR Path="/5CFF7883/5CED8F95" Ref="#PWR?"  Part="1"
-F 0 "#PWR?" H 2800 3350 50  0001 C CNN
+F 0 "#PWR045" H 2800 3350 50  0001 C CNN
 F 1 "GND" H 2850 3400 50  0000 C CNN
 F 2 "" H 2800 3600 50  0001 C CNN
@@
 	2800 3600 2800 3550
 $Comp
-L power:GND #PWR?
+L power:GND #PWR041
 U 1 1 5CED947F
 P 3350 2600
-AR Path="/5CF34744/5CED947F" Ref="#PWR?"  Part="1"
+AR Path="/5CF34744/5CED947F" Ref="#PWR041"  Part="1"
 AR Path="/5CFF7883/5CED947F" Ref="#PWR?"  Part="1"
-F 0 "#PWR?" H 3350 2350 50  0001 C CNN
+F 0 "#PWR041" H 3350 2350 50  0001 C CNN
 F 1 "GND" H 3400 2400 50  0000 C CNN
 F 2 "" H 3350 2600 50  0001 C CNN
@@
 $EndComp
 $Comp
-L power:GND #PWR?
-U 1 1 5CED96CA
+L power:GND #PWR043
+U 1 1 5D32A3C5
 P 4400 2900
-AR Path="/5CF34744/5CED96CA" Ref="#PWR?"  Part="1"
-AR Path="/5CFF7883/5CED96CA" Ref="#PWR?"  Part="1"
-F 0 "#PWR?" H 4400 2650 50  0001 C CNN
+AR Path="/5CF34744/5D32A3C5" Ref="#PWR043"  Part="1"
+AR Path="/5CFF7883/5D32A3C5" Ref="#PWR?"  Part="1"
+F 0 "#PWR043" H 4400 2650 50  0001 C CNN
 F 1 "GND" H 4450 2700 50  0000 C CNN
 F 2 "" H 4400 2900 50  0001 C CNN
@@
 ROT_ENC_A
 $Comp
-L Connector:Conn_01x03_Female J?
+L Connector:Conn_01x03_Female J2
 U 1 1 5CF225E9
 P 1100 2200
-AR Path="/5CF34744/5CF225E9" Ref="J?"  Part="1"
+AR Path="/5CF34744/5CF225E9" Ref="J2"  Part="1"
 AR Path="/5CFF7883/5CF225E9" Ref="J?"  Part="1"
-F 0 "J?" H 950 2500 50  0000 C CNN
+F 0 "J2" H 950 2500 50  0000 C CNN
 F 1 "ROT_ENC_HEADER" H 950 2400 50  0000 C CNN
 F 2 "Connector_PinHeader_1.27mm:PinHeader_1x03_P1.27mm_Vertical" H 1100 2200 50  0001 C CNN
