File: hardware/buzzer.sch (KiCad schematic (older format))
At the start: 5 parts

Commit message: update for power symbol,
Connections:
- net +3V3 renamed Vbuzzer
Changed lines of the file:
@@
 $EndBitmap
-$Comp
-L power:+3V3 #PWR?
-U 1 1 5CEBF99F
-P 3150 1100
-F 0 "#PWR?" H 3150 950 50  0001 C CNN
-F 1 "+3V3" H 3200 1300 50  0000 C CNN
-F 2 "" H 3150 1100 50  0001 C CNN
-F 3 "" H 3150 1100 50  0001 C CNN
-	1    3150 1100
-	1    0    0    -1
-$EndComp
 $Comp
 L taobao-components:BUZZER,MLT-8530 BZ?
@@
 Wire Wire Line
 	1300 1350 1300 1500
+$Comp
+L my_power:Vbuzzer #PWR?
+U 1 1 5D10D638
+P 3150 1100
+F 0 "#PWR?" H 3150 950 50  0001 C CNN
+F 1 "Vbuzzer" H 3155 1273 50  0000 C CNN
+F 2 "" H 3150 1100 50  0001 C CNN
+F 3 "" H 3150 1100 50  0001 C CNN
+	1    3150 1100
+	1    0    0    -1
+$EndComp
 $EndSCHEMATC

Commit message: update,
Parts:
- gave numbers to parts that had none: 5
Changed lines of the file:
@@
 $EndBitmap
 $Comp
-L taobao-components:BUZZER,MLT-8530 BZ?
+L taobao-components:BUZZER,MLT-8530 BZ1
 U 1 1 5CEC8447
 P 3300 1450
-F 0 "BZ?" H 3500 1500 50  0000 L CNN
+F 0 "BZ1" H 3500 1500 50  0000 L CNN
 F 1 "BUZZER,MLT-8530" H 3500 1400 50  0000 L CNN
 F 2 "footprint-lib:MLT-8530" V 3275 1550 50  0001 C CNN
@@
 $EndComp
 $Comp
-L taobao-transistor:SS9013_J3 Q?
+L taobao-transistor:SS9013_J3 Q1
 U 1 1 5CEC8A45
 P 3050 2000
-F 0 "Q?" H 3250 2050 50  0000 L CNN
+F 0 "Q1" H 3250 2050 50  0000 L CNN
 F 1 "SS9013_J3" H 3250 2000 50  0000 L CNN
 F 2 "footprint-lib:9013,J3,SOT23" H 3250 1925 50  0001 L CIN
@@
 $EndComp
 $Comp
-L taobao-r:R471,0603 R?
+L taobao-r:R471,0603 R27
 U 1 1 5CEC945D
 P 2400 2000
-F 0 "R?" V 2150 2000 50  0000 C CNN
+F 0 "R27" V 2150 2000 50  0000 C CNN
 F 1 "R471,0603" V 2250 2000 50  0000 C CNN
 F 2 "Resistor_SMD:R_0603_1608Metric_Pad1.05x0.95mm_HandSolder" H 2400 2000 50  0001 C CNN
@@
 	3150 1650 3150 1800
 $Comp
-L taobao-d:D_1N4148_T4 D?
+L taobao-d:D_1N4148_T4 D37
 U 1 1 5CECC56E
 P 3000 1450
-F 0 "D?" V 2950 1350 50  0000 R CNN
+F 0 "D37" V 2950 1350 50  0000 R CNN
 F 1 "D_1N4148_T4" V 3000 1350 50  0000 R CNN
 F 2 "Diode_SMD:D_SOD-123" V 3000 1450 50  0001 C CNN
@@
 $EndComp
 $Comp
-L power:GND #PWR?
+L power:GND #PWR0121
 U 1 1 5CECCC65
 P 3150 2500
-F 0 "#PWR?" H 3150 2250 50  0001 C CNN
+F 0 "#PWR0121" H 3150 2250 50  0001 C CNN
 F 1 "GND" H 3200 2300 50  0000 C CNN
 F 2 "" H 3150 2500 50  0001 C CNN
@@
 	1450 2000 2300 2000
 $Comp
-L Connector:Conn_01x02_Female J?
+L Connector:Conn_01x02_Female J4
 U 1 1 5CF28177
 P 900 1250
-F 0 "J?" H 750 1450 50  0000 C CNN
+F 0 "J4" H 750 1450 50  0000 C CNN
 F 1 "BUZZER_HEADER" H 750 1350 50  0000 C CNN
 F 2 "Connector_PinHeader_1.27mm:PinHeader_1x02_P1.27mm_Vertical" H 900 1250 50  0001 C CNN
@@
 	1950 1250 1100 1250
 $Comp
-L power:GND #PWR?
+L power:GND #PWR0120
 U 1 1 5CF28714
 P 1300 1500
-F 0 "#PWR?" H 1300 1250 50  0001 C CNN
+F 0 "#PWR0120" H 1300 1250 50  0001 C CNN
 F 1 "GND" H 1350 1300 50  0000 C CNN
 F 2 "" H 1300 1500 50  0001 C CNN
@@
 	1300 1350 1300 1500
 $Comp
-L my_power:Vbuzzer #PWR?
+L my_power:Vbuzzer #PWR0119
 U 1 1 5D10D638
 P 3150 1100
-F 0 "#PWR?" H 3150 950 50  0001 C CNN
+F 0 "#PWR0119" H 3150 950 50  0001 C CNN
 F 1 "Vbuzzer" H 3155 1273 50  0000 C CNN
 F 2 "" H 3150 1100 50  0001 C CNN
