File: hardware/buzzer.sch (KiCad schematic (older format))
At the start: 5 parts, among them J4 BUZZER_HEADER, Q1 SS9013_J3

Commit message: update,
Parts:
- added C58: C106,0603, Capacitor_SMD:C_0603_1608Metric_Pad1.05x0.95mm_HandSolder, symbol taobao-c:C106,0603
Connections:
- net GND: now also C58.2
- net Vbuzzer: now also C58.1
Changed lines of the file:
@@
 	1    0    0    -1
 $EndComp
+$Comp
+L my_power:Vbuzzer #PWR0164
+U 1 1 5D5FC0D3
+P 4250 1100
+F 0 "#PWR0164" H 4250 950 50  0001 C CNN
+F 1 "Vbuzzer" H 4255 1273 50  0000 C CNN
+F 2 "" H 4250 1100 50  0001 C CNN
+F 3 "" H 4250 1100 50  0001 C CNN
+	1    4250 1100
+	1    0    0    -1
+$EndComp
+$Comp
+L taobao-c:C106,0603 C58
+U 1 1 5D5FC465
+P 4250 1350
+F 0 "C58" H 4342 1396 50  0000 L CNN
+F 1 "C106,0603" H 4342 1305 50  0000 L CNN
+F 2 "Capacitor_SMD:C_0603_1608Metric_Pad1.05x0.95mm_HandSolder" H 4250 1350 50  0001 C CNN
+F 3 "~" H 4250 1350 50  0001 C CNN
+	1    4250 1350
+	1    0    0    -1
+$EndComp
+$Comp
+L power:GND #PWR0165
+U 1 1 5D5FC7FA
+P 4250 1650
+F 0 "#PWR0165" H 4250 1400 50  0001 C CNN
+F 1 "GND" H 4255 1477 50  0000 C CNN
+F 2 "" H 4250 1650 50  0001 C CNN
+F 3 "" H 4250 1650 50  0001 C CNN
+	1    4250 1650
+	1    0    0    -1
+$EndComp
+Wire Wire Line
+	4250 1100 4250 1250
+Wire Wire Line
+	4250 1450 4250 1650
 $EndSCHEMATC

Commit message: update,
Parts:
- renumbered C58 to C25, D37 to D24, J4 to J3, R27 to R15
Changed lines of the file:
@@
 $EndComp
 $Comp
-L taobao-r:R471,0603 R27
+L taobao-r:R471,0603 R15
 U 1 1 5CEC945D
 P 2400 2000
-F 0 "R27" V 2150 2000 50  0000 C CNN
+F 0 "R15" V 2150 2000 50  0000 C CNN
 F 1 "R471,0603" V 2250 2000 50  0000 C CNN
 F 2 "Resistor_SMD:R_0603_1608Metric_Pad1.05x0.95mm_HandSolder" H 2400 2000 50  0001 C CNN
@@
 	3150 1650 3150 1800
 $Comp
-L taobao-d:D_1N4148_T4 D37
+L taobao-d:D_1N4148_T4 D24
 U 1 1 5CECC56E
 P 3000 1450
-F 0 "D37" V 2950 1350 50  0000 R CNN
+F 0 "D24" V 2950 1350 50  0000 R CNN
 F 1 "D_1N4148_T4" V 3000 1350 50  0000 R CNN
 F 2 "Diode_SMD:D_SOD-123" V 3000 1450 50  0001 C CNN
@@
 $EndComp
 $Comp
-L power:GND #PWR0121
+L power:GND #PWR0108
 U 1 1 5CECCC65
 P 3150 2500
-F 0 "#PWR0121" H 3150 2250 50  0001 C CNN
+F 0 "#PWR0108" H 3150 2250 50  0001 C CNN
 F 1 "GND" H 3200 2300 50  0000 C CNN
 F 2 "" H 3150 2500 50  0001 C CNN
@@
 	1450 2000 2300 2000
 $Comp
-L Connector:Conn_01x02_Female J4
+L Connector:Conn_01x02_Female J3
 U 1 1 5CF28177
 P 900 1250
-F 0 "J4" H 750 1450 50  0000 C CNN
+F 0 "J3" H 750 1450 50  0000 C CNN
 F 1 "BUZZER_HEADER" H 750 1350 50  0000 C CNN
 F 2 "Connector_PinHeader_1.27mm:PinHeader_1x02_P1.27mm_Vertical" H 900 1250 50  0001 C CNN
@@
 	1950 1250 1100 1250
 $Comp
-L power:GND #PWR0120
+L power:GND #PWR0106
 U 1 1 5CF28714
 P 1300 1500
-F 0 "#PWR0120" H 1300 1250 50  0001 C CNN
+F 0 "#PWR0106" H 1300 1250 50  0001 C CNN
 F 1 "GND" H 1350 1300 50  0000 C CNN
 F 2 "" H 1300 1500 50  0001 C CNN
@@
 	1300 1350 1300 1500
 $Comp
-L my_power:Vbuzzer #PWR0119
+L my_power:Vbuzzer #PWR0104
 U 1 1 5D10D638
 P 3150 1100
-F 0 "#PWR0119" H 3150 950 50  0001 C CNN
+F 0 "#PWR0104" H 3150 950 50  0001 C CNN
 F 1 "Vbuzzer" H 3155 1273 50  0000 C CNN
 F 2 "" H 3150 1100 50  0001 C CNN
@@
 $EndComp
 $Comp
-L my_power:Vbuzzer #PWR0164
+L my_power:Vbuzzer #PWR0105
 U 1 1 5D5FC0D3
 P 4250 1100
-F 0 "#PWR0164" H 4250 950 50  0001 C CNN
+F 0 "#PWR0105" H 4250 950 50  0001 C CNN
 F 1 "Vbuzzer" H 4255 1273 50  0000 C CNN
 F 2 "" H 4250 1100 50  0001 C CNN
@@
 $EndComp
 $Comp
-L taobao-c:C106,0603 C58
+L taobao-c:C106,0603 C25
 U 1 1 5D5FC465
 P 4250 1350
-F 0 "C58" H 4342 1396 50  0000 L CNN
+F 0 "C25" H 4342 1396 50  0000 L CNN
 F 1 "C106,0603" H 4342 1305 50  0000 L CNN
 F 2 "Capacitor_SMD:C_0603_1608Metric_Pad1.05x0.95mm_HandSolder" H 4250 1350 50  0001 C CNN
@@
 $EndComp
 $Comp
-L power:GND #PWR0165
+L power:GND #PWR0107
 U 1 1 5D5FC7FA
 P 4250 1650
-F 0 "#PWR0165" H 4250 1400 50  0001 C CNN
+F 0 "#PWR0107" H 4250 1400 50  0001 C CNN
 F 1 "GND" H 4255 1477 50  0000 C CNN
 F 2 "" H 4250 1650 50  0001 C CNN
