File: hardware/push_buttton.sch (KiCad schematic (older format))
At the start: 8 parts

Commit message: update,
Parts:
- gave numbers to parts that had none: 8
Changed lines of the file:
@@
 $EndDescr
 $Comp
-L power:+3V3 #PWR?
+L power:+3V3 #PWR0107
 U 1 1 5D0C3DDE
 P 1700 1450
-F 0 "#PWR?" H 1700 1300 50  0001 C CNN
+F 0 "#PWR0107" H 1700 1300 50  0001 C CNN
 F 1 "+3V3" H 1715 1623 50  0000 C CNN
 F 2 "" H 1700 1450 50  0001 C CNN
@@
 $EndComp
 $Comp
-L taobao-r:R103,0603 R?
+L taobao-r:R103,0603 R23
 U 1 1 5D0C4235
 P 1700 1700
-F 0 "R?" H 1759 1746 50  0000 L CNN
+F 0 "R23" H 1759 1746 50  0000 L CNN
 F 1 "R103,0603" H 1759 1655 50  0000 L CNN
 F 2 "Resistor_SMD:R_0603_1608Metric_Pad1.05x0.95mm_HandSolder" H 1700 1700 50  0001 C CNN
@@
 $EndComp
 $Comp
-L taobao-button:SW_RESET,2_leg,SMD SW?
+L taobao-button:SW_RESET,2_leg,SMD SW15
 U 1 1 5D0C44DF
 P 1700 2150
-F 0 "SW?" V 1654 2298 50  0000 L CNN
+F 0 "SW15" V 1654 2298 50  0000 L CNN
 F 1 "USR_BTN_1" V 1745 2298 50  0000 L CNN
 F 2 "footprint-lib:SW_SPST_CK_RS282G05A3" H 1700 2350 50  0001 C CNN
@@
 $EndComp
 $Comp
-L power:GND #PWR?
+L power:GND #PWR0111
 U 1 1 5D0C49CE
 P 1700 2500
-F 0 "#PWR?" H 1700 2250 50  0001 C CNN
+F 0 "#PWR0111" H 1700 2250 50  0001 C CNN
 F 1 "GND" H 1705 2327 50  0000 C CNN
 F 2 "" H 1700 2500 50  0001 C CNN
@@
 	1700 1450 1700 1600
 $Comp
-L power:+3V3 #PWR?
+L power:+3V3 #PWR0108
 U 1 1 5D0C524F
 P 2400 1450
-F 0 "#PWR?" H 2400 1300 50  0001 C CNN
+F 0 "#PWR0108" H 2400 1300 50  0001 C CNN
 F 1 "+3V3" H 2415 1623 50  0000 C CNN
 F 2 "" H 2400 1450 50  0001 C CNN
@@
 $EndComp
 $Comp
-L taobao-r:R103,0603 R?
+L taobao-r:R103,0603 R24
 U 1 1 5D0C5259
 P 2400 1700
-F 0 "R?" H 2459 1746 50  0000 L CNN
+F 0 "R24" H 2459 1746 50  0000 L CNN
 F 1 "R103,0603" H 2459 1655 50  0000 L CNN
 F 2 "Resistor_SMD:R_0603_1608Metric_Pad1.05x0.95mm_HandSolder" H 2400 1700 50  0001 C CNN
@@
 $EndComp
 $Comp
-L taobao-button:SW_RESET,2_leg,SMD SW?
+L taobao-button:SW_RESET,2_leg,SMD SW16
 U 1 1 5D0C5263
 P 2400 2150
-F 0 "SW?" V 2354 2298 50  0000 L CNN
+F 0 "SW16" V 2354 2298 50  0000 L CNN
 F 1 "USR_BTN_2" V 2445 2298 50  0000 L CNN
 F 2 "footprint-lib:SW_SPST_CK_RS282G05A3" H 2400 2350 50  0001 C CNN
@@
 $EndComp
 $Comp
-L power:GND #PWR?
+L power:GND #PWR0112
 U 1 1 5D0C526D
 P 2400 2500
-F 0 "#PWR?" H 2400 2250 50  0001 C CNN
+F 0 "#PWR0112" H 2400 2250 50  0001 C CNN
 F 1 "GND" H 2405 2327 50  0000 C CNN
 F 2 "" H 2400 2500 50  0001 C CNN
@@
 	2400 1450 2400 1600
 $Comp
-L power:+3V3 #PWR?
+L power:+3V3 #PWR0109
 U 1 1 5D0C5F20
 P 3100 1450
-F 0 "#PWR?" H 3100 1300 50  0001 C CNN
+F 0 "#PWR0109" H 3100 1300 50  0001 C CNN
 F 1 "+3V3" H 3115 1623 50  0000 C CNN
 F 2 "" H 3100 1450 50  0001 C CNN
@@
 $EndComp
 $Comp
-L taobao-r:R103,0603 R?
+L taobao-r:R103,0603 R25
 U 1 1 5D0C5F2A
 P 3100 1700
-F 0 "R?" H 3159 1746 50  0000 L CNN
+F 0 "R25" H 3159 1746 50  0000 L CNN
 F 1 "R103,0603" H 3159 1655 50  0000 L CNN
 F 2 "Resistor_SMD:R_0603_1608Metric_Pad1.05x0.95mm_HandSolder" H 3100 1700 50  0001 C CNN
@@
 $EndComp
 $Comp
-L taobao-button:SW_RESET,2_leg,SMD SW?
+L taobao-button:SW_RESET,2_leg,SMD SW17
 U 1 1 5D0C5F34
 P 3100 2150
-F 0 "SW?" V 3054 2298 50  0000 L CNN
+F 0 "SW17" V 3054 2298 50  0000 L CNN
 F 1 "USR_BTN_3" V 3145 2298 50  0000 L CNN
 F 2 "footprint-lib:SW_SPST_CK_RS282G05A3" H 3100 2350 50  0001 C CNN
@@
 $EndComp
 $Comp
-L power:GND #PWR?
+L power:GND #PWR0113
 U 1 1 5D0C5F3E
 P 3100 2500
-F 0 "#PWR?" H 3100 2250 50  0001 C CNN
+F 0 "#PWR0113" H 3100 2250 50  0001 C CNN
 F 1 "GND" H 3105 2327 50  0000 C CNN
 F 2 "" H 3100 2500 50  0001 C CNN
@@
 	3100 1450 3100 1600
 $Comp
-L power:+3V3 #PWR?
+L power:+3V3 #PWR0110
 U 1 1 5D0C5F4B
 P 3800 1450
-F 0 "#PWR?" H 3800 1300 50  0001 C CNN
+F 0 "#PWR0110" H 3800 1300 50  0001 C CNN
 F 1 "+3V3" H 3815 1623 50  0000 C CNN
 F 2 "" H 3800 1450 50  0001 C CNN
@@
 $EndComp
 $Comp
-L taobao-r:R103,0603 R?
+L taobao-r:R103,0603 R26
 U 1 1 5D0C5F55
 P 3800 1700
-F 0 "R?" H 3859 1746 50  0000 L CNN
+F 0 "R26" H 3859 1746 50  0000 L CNN
 F 1 "R103,0603" H 3859 1655 50  0000 L CNN
 F 2 "Resistor_SMD:R_0603_1608Metric_Pad1.05x0.95mm_HandSolder" H 3800 1700 50  0001 C CNN
@@
 $EndComp
 $Comp
-L taobao-button:SW_RESET,2_leg,SMD SW?
+L taobao-button:SW_RESET,2_leg,SMD SW18
 U 1 1 5D0C5F5F
 P 3800 2150
-F 0 "SW?" V 3754 2298 50  0000 L CNN
+F 0 "SW18" V 3754 2298 50  0000 L CNN
 F 1 "USR_BTN_4" V 3845 2298 50  0000 L CNN
 F 2 "footprint-lib:SW_SPST_CK_RS282G05A3" H 3800 2350 50  0001 C CNN
@@
 $EndComp
 $Comp
-L power:GND #PWR?
+L power:GND #PWR0114
 U 1 1 5D0C5F69
 P 3800 2500
-F 0 "#PWR?" H 3800 2250 50  0001 C CNN
+F 0 "#PWR0114" H 3800 2250 50  0001 C CNN
 F 1 "GND" H 3805 2327 50  0000 C CNN
 F 2 "" H 3800 2500 50  0001 C CNN

Commit message: update,
Connections:
- net USR_BTN_1: now reaches R23.2, SW15.1
- net USR_BTN_2: now reaches R24.2, SW16.1
- net USR_BTN_3: now reaches R25.2, SW17.1
- net USR_BTN_4: now reaches R26.2, SW18.1
Other:
- moved on the sheet: R23, R24, R25, R26, SW16, SW17, SW18
Changed lines of the file:
@@
 $Descr User 8500 5500
 encoding utf-8
-Sheet 9 13
+Sheet 7 13
 Title ""
 Date ""
@@
 L taobao-r:R103,0603 R23
 U 1 1 5D0C4235
-P 1700 1700
-F 0 "R23" H 1759 1746 50  0000 L CNN
-F 1 "R103,0603" H 1759 1655 50  0000 L CNN
-F 2 "Resistor_SMD:R_0603_1608Metric_Pad1.05x0.95mm_HandSolder" H 1700 1700 50  0001 C CNN
-F 3 "~" H 1700 1700 50  0001 C CNN
-	1    1700 1700
+P 1700 1600
+F 0 "R23" H 1759 1646 50  0000 L CNN
+F 1 "R103,0603" H 1759 1555 50  0000 L CNN
+F 2 "Resistor_SMD:R_0603_1608Metric_Pad1.05x0.95mm_HandSolder" H 1700 1600 50  0001 C CNN
+F 3 "~" H 1700 1600 50  0001 C CNN
+	1    1700 1600
 	1    0    0    -1
 $EndComp
@@
 	1700 2350 1700 2500
 Wire Wire Line
-	1700 1800 1700 1950
-Wire Wire Line
-	1700 1450 1700 1600
+	1700 1700 1700 1800
+Wire Wire Line
+	1700 1450 1700 1500
 $Comp
 L power:+3V3 #PWR0108
 U 1 1 5D0C524F
-P 2400 1450
-F 0 "#PWR0108" H 2400 1300 50  0001 C CNN
-F 1 "+3V3" H 2415 1623 50  0000 C CNN
-F 2 "" H 2400 1450 50  0001 C CNN
-F 3 "" H 2400 1450 50  0001 C CNN
-	1    2400 1450
+P 2950 1450
+F 0 "#PWR0108" H 2950 1300 50  0001 C CNN
+F 1 "+3V3" H 2965 1623 50  0000 C CNN
+F 2 "" H 2950 1450 50  0001 C CNN
+F 3 "" H 2950 1450 50  0001 C CNN
+	1    2950 1450
 	1    0    0    -1
 $EndComp
@@
 L taobao-r:R103,0603 R24
 U 1 1 5D0C5259
-P 2400 1700
-F 0 "R24" H 2459 1746 50  0000 L CNN
-F 1 "R103,0603" H 2459 1655 50  0000 L CNN
-F 2 "Resistor_SMD:R_0603_1608Metric_Pad1.05x0.95mm_HandSolder" H 2400 1700 50  0001 C CNN
-F 3 "~" H 2400 1700 50  0001 C CNN
-	1    2400 1700
+P 2950 1600
+F 0 "R24" H 3009 1646 50  0000 L CNN
+F 1 "R103,0603" H 3009 1555 50  0000 L CNN
+F 2 "Resistor_SMD:R_0603_1608Metric_Pad1.05x0.95mm_HandSolder" H 2950 1600 50  0001 C CNN
+F 3 "~" H 2950 1600 50  0001 C CNN
+	1    2950 1600
 	1    0    0    -1
 $EndComp
@@
 L taobao-button:SW_RESET,2_leg,SMD SW16
 U 1 1 5D0C5263
-P 2400 2150
-F 0 "SW16" V 2354 2298 50  0000 L CNN
-F 1 "USR_BTN_2" V 2445 2298 50  0000 L CNN
-F 2 "footprint-lib:SW_SPST_CK_RS282G05A3" H 2400 2350 50  0001 C CNN
-F 3 "~" H 2400 2350 50  0001 C CNN
-	1    2400 2150
+P 2950 2150
+F 0 "SW16" V 2904 2298 50  0000 L CNN
+F 1 "USR_BTN_2" V 2995 2298 50  0000 L CNN
+F 2 "footprint-lib:SW_SPST_CK_RS282G05A3" H 2950 2350 50  0001 C CNN
+F 3 "~" H 2950 2350 50  0001 C CNN
+	1    2950 2150
 	0    1    1    0
 $EndComp
@@
 L power:GND #PWR0112
 U 1 1 5D0C526D
-P 2400 2500
-F 0 "#PWR0112" H 2400 2250 50  0001 C CNN
-F 1 "GND" H 2405 2327 50  0000 C CNN
-F 2 "" H 2400 2500 50  0001 C CNN
-F 3 "" H 2400 2500 50  0001 C CNN
-	1    2400 2500
-	1    0    0    -1
-$EndComp
-Wire Wire Line
-	2400 2350 2400 2500
-Wire Wire Line
-	2400 1800 2400 1950
-Wire Wire Line
-	2400 1450 2400 1600
+P 2950 2500
+F 0 "#PWR0112" H 2950 2250 50  0001 C CNN
+F 1 "GND" H 2955 2327 50  0000 C CNN
+F 2 "" H 2950 2500 50  0001 C CNN
+F 3 "" H 2950 2500 50  0001 C CNN
+	1    2950 2500
+	1    0    0    -1
+$EndComp
+Wire Wire Line
+	2950 2350 2950 2500
+Wire Wire Line
+	2950 1700 2950 1800
+Wire Wire Line
+	2950 1450 2950 1500
 $Comp
 L power:+3V3 #PWR0109
 U 1 1 5D0C5F20
-P 3100 1450
-F 0 "#PWR0109" H 3100 1300 50  0001 C CNN
-F 1 "+3V3" H 3115 1623 50  0000 C CNN
-F 2 "" H 3100 1450 50  0001 C CNN
-F 3 "" H 3100 1450 50  0001 C CNN
-	1    3100 1450
+P 4100 1450
+F 0 "#PWR0109" H 4100 1300 50  0001 C CNN
+F 1 "+3V3" H 4115 1623 50  0000 C CNN
+F 2 "" H 4100 1450 50  0001 C CNN
+F 3 "" H 4100 1450 50  0001 C CNN
+	1    4100 1450
 	1    0    0    -1
 $EndComp
@@
 L taobao-r:R103,0603 R25
 U 1 1 5D0C5F2A
-P 3100 1700
-F 0 "R25" H 3159 1746 50  0000 L CNN
-F 1 "R103,0603" H 3159 1655 50  0000 L CNN
-F 2 "Resistor_SMD:R_0603_1608Metric_Pad1.05x0.95mm_HandSolder" H 3100 1700 50  0001 C CNN
-F 3 "~" H 3100 1700 50  0001 C CNN
-	1    3100 1700
+P 4100 1600
+F 0 "R25" H 4159 1646 50  0000 L CNN
+F 1 "R103,0603" H 4159 1555 50  0000 L CNN
+F 2 "Resistor_SMD:R_0603_1608Metric_Pad1.05x0.95mm_HandSolder" H 4100 1600 50  0001 C CNN
+F 3 "~" H 4100 1600 50  0001 C CNN
+	1    4100 1600
 	1    0    0    -1
 $EndComp
@@
 L taobao-button:SW_RESET,2_leg,SMD SW17
 U 1 1 5D0C5F34
-P 3100 2150
-F 0 "SW17" V 3054 2298 50  0000 L CNN
-F 1 "USR_BTN_3" V 3145 2298 50  0000 L CNN
-F 2 "footprint-lib:SW_SPST_CK_RS282G05A3" H 3100 2350 50  0001 C CNN
-F 3 "~" H 3100 2350 50  0001 C CNN
-	1    3100 2150
+P 4100 2150
+F 0 "SW17" V 4054 2298 50  0000 L CNN
+F 1 "USR_BTN_3" V 4145 2298 50  0000 L CNN
+F 2 "footprint-lib:SW_SPST_CK_RS282G05A3" H 4100 2350 50  0001 C CNN
+F 3 "~" H 4100 2350 50  0001 C CNN
+	1    4100 2150
 	0    1    1    0
 $EndComp
@@
 L power:GND #PWR0113
 U 1 1 5D0C5F3E
-P 3100 2500
-F 0 "#PWR0113" H 3100 2250 50  0001 C CNN
-F 1 "GND" H 3105 2327 50  0000 C CNN
-F 2 "" H 3100 2500 50  0001 C CNN
-F 3 "" H 3100 2500 50  0001 C CNN
-	1    3100 2500
-	1    0    0    -1
-$EndComp
-Wire Wire Line
-	3100 2350 3100 2500
-Wire Wire Line
-	3100 1800 3100 1950
-Wire Wire Line
-	3100 1450 3100 1600
+P 4100 2500
+F 0 "#PWR0113" H 4100 2250 50  0001 C CNN
+F 1 "GND" H 4105 2327 50  0000 C CNN
+F 2 "" H 4100 2500 50  0001 C CNN
+F 3 "" H 4100 2500 50  0001 C CNN
+	1    4100 2500
+	1    0    0    -1
+$EndComp
+Wire Wire Line
+	4100 2350 4100 2500
+Wire Wire Line
+	4100 1700 4100 1800
+Wire Wire Line
+	4100 1450 4100 1500
 $Comp
 L power:+3V3 #PWR0110
 U 1 1 5D0C5F4B
-P 3800 1450
-F 0 "#PWR0110" H 3800 1300 50  0001 C CNN
-F 1 "+3V3" H 3815 1623 50  0000 C CNN
-F 2 "" H 3800 1450 50  0001 C CNN
-F 3 "" H 3800 1450 50  0001 C CNN
-	1    3800 1450
+P 5150 1450
+F 0 "#PWR0110" H 5150 1300 50  0001 C CNN
+F 1 "+3V3" H 5165 1623 50  0000 C CNN
+F 2 "" H 5150 1450 50  0001 C CNN
+F 3 "" H 5150 1450 50  0001 C CNN
+	1    5150 1450
 	1    0    0    -1
 $EndComp
@@
 L taobao-r:R103,0603 R26
 U 1 1 5D0C5F55
-P 3800 1700
-F 0 "R26" H 3859 1746 50  0000 L CNN
-F 1 "R103,0603" H 3859 1655 50  0000 L CNN
-F 2 "Resistor_SMD:R_0603_1608Metric_Pad1.05x0.95mm_HandSolder" H 3800 1700 50  0001 C CNN
-F 3 "~" H 3800 1700 50  0001 C CNN
-	1    3800 1700
+P 5150 1600
+F 0 "R26" H 5209 1646 50  0000 L CNN
+F 1 "R103,0603" H 5209 1555 50  0000 L CNN
+F 2 "Resistor_SMD:R_0603_1608Metric_Pad1.05x0.95mm_HandSolder" H 5150 1600 50  0001 C CNN
+F 3 "~" H 5150 1600 50  0001 C CNN
+	1    5150 1600
 	1    0    0    -1
 $EndComp
@@
 L taobao-button:SW_RESET,2_leg,SMD SW18
 U 1 1 5D0C5F5F
-P 3800 2150
-F 0 "SW18" V 3754 2298 50  0000 L CNN
-F 1 "USR_BTN_4" V 3845 2298 50  0000 L CNN
-F 2 "footprint-lib:SW_SPST_CK_RS282G05A3" H 3800 2350 50  0001 C CNN
-F 3 "~" H 3800 2350 50  0001 C CNN
-	1    3800 2150
+P 5150 2150
+F 0 "SW18" V 5104 2298 50  0000 L CNN
+F 1 "USR_BTN_4" V 5195 2298 50  0000 L CNN
+F 2 "footprint-lib:SW_SPST_CK_RS282G05A3" H 5150 2350 50  0001 C CNN
+F 3 "~" H 5150 2350 50  0001 C CNN
+	1    5150 2150
 	0    1    1    0
 $EndComp
@@
 L power:GND #PWR0114
 U 1 1 5D0C5F69
-P 3800 2500
-F 0 "#PWR0114" H 3800 2250 50  0001 C CNN
-F 1 "GND" H 3805 2327 50  0000 C CNN
-F 2 "" H 3800 2500 50  0001 C CNN
-F 3 "" H 3800 2500 50  0001 C CNN
-	1    3800 2500
-	1    0    0    -1
-$EndComp
-Wire Wire Line
-	3800 2350 3800 2500
-Wire Wire Line
-	3800 1800 3800 1950
-Wire Wire Line
-	3800 1450 3800 1600
+P 5150 2500
+F 0 "#PWR0114" H 5150 2250 50  0001 C CNN
+F 1 "GND" H 5155 2327 50  0000 C CNN
+F 2 "" H 5150 2500 50  0001 C CNN
+F 3 "" H 5150 2500 50  0001 C CNN
+	1    5150 2500
+	1    0    0    -1
+$EndComp
+Wire Wire Line
+	5150 2350 5150 2500
+Wire Wire Line
+	5150 1700 5150 1800
+Wire Wire Line
+	5150 1450 5150 1500
+Text HLabel 1000 650  0    50   Input ~ 0
+USR_BTN_1
+Text HLabel 1000 750  0    50   Input ~ 0
+USR_BTN_2
+Text HLabel 1000 850  0    50   Input ~ 0
+USR_BTN_3
+Text HLabel 1000 950  0    50   Input ~ 0
+USR_BTN_4
+Text Label 1550 650  2    50   ~ 0
+USR_BTN_1
+Text Label 1550 750  2    50   ~ 0
+USR_BTN_2
+Text Label 1550 850  2    50   ~ 0
+USR_BTN_3
+Text Label 1550 950  2    50   ~ 0
+USR_BTN_4
+Wire Wire Line
+	1000 650  1550 650
+Wire Wire Line
+	1000 750  1550 750
+Wire Wire Line
+	1000 850  1550 850
+Wire Wire Line
+	1000 950  1550 950
+Text Label 2300 1800 2    50   ~ 0
+USR_BTN_1
+Wire Wire Line
+	2300 1800 1700 1800
+Connection ~ 1700 1800
+Wire Wire Line
+	1700 1800 1700 1950
+Text Label 3500 1800 2    50   ~ 0
+USR_BTN_2
+Wire Wire Line
+	3500 1800 2950 1800
+Connection ~ 2950 1800
+Wire Wire Line
+	2950 1800 2950 1950
+Text Label 4650 1800 2    50   ~ 0
+USR_BTN_3
+Wire Wire Line
+	4650 1800 4100 1800
+Connection ~ 4100 1800
+Wire Wire Line
+	4100 1800 4100 1950
+Text Label 5650 1800 2    50   ~ 0
+USR_BTN_4
+Wire Wire Line
+	5650 1800 5150 1800
+Connection ~ 5150 1800
+Wire Wire Line
+	5150 1800 5150 1950
 $EndSCHEMATC
