File: hardware/push_buttton.sch (KiCad schematic (older format))
At the start: 8 parts, among them SW15 USR_BTN_1, SW16 USR_BTN_2, SW17 USR_BTN_3, SW18 USR_BTN_4

Commit message: update,
Parts:
- renumbered R23 to R10, R24 to R11, R25 to R12, R26 to R13, SW15 to SW1, SW16 to SW2, SW17 to SW3, SW18 to SW4
Changed lines of the file:
@@
 $EndDescr
 $Comp
-L power:+3V3 #PWR0107
+L power:+3V3 #PWR091
 U 1 1 5D0C3DDE
 P 1700 1450
-F 0 "#PWR0107" H 1700 1300 50  0001 C CNN
+F 0 "#PWR091" H 1700 1300 50  0001 C CNN
 F 1 "+3V3" H 1715 1623 50  0000 C CNN
 F 2 "" H 1700 1450 50  0001 C CNN
@@
 $EndComp
 $Comp
-L taobao-r:R103,0603 R23
+L taobao-r:R103,0603 R10
 U 1 1 5D0C4235
 P 1700 1600
-F 0 "R23" H 1759 1646 50  0000 L CNN
+F 0 "R10" H 1759 1646 50  0000 L CNN
 F 1 "R103,0603" H 1759 1555 50  0000 L CNN
 F 2 "Resistor_SMD:R_0603_1608Metric_Pad1.05x0.95mm_HandSolder" H 1700 1600 50  0001 C CNN
@@
 $EndComp
 $Comp
-L taobao-button:SW_RESET,2_leg,SMD SW15
+L taobao-button:SW_RESET,2_leg,SMD SW1
 U 1 1 5D0C44DF
 P 1700 2150
-F 0 "SW15" V 1654 2298 50  0000 L CNN
+F 0 "SW1" V 1654 2298 50  0000 L CNN
 F 1 "USR_BTN_1" V 1745 2298 50  0000 L CNN
 F 2 "footprint-lib:SW_SPST_CK_RS282G05A3" H 1700 2350 50  0001 C CNN
@@
 $EndComp
 $Comp
-L power:GND #PWR0111
+L power:GND #PWR095
 U 1 1 5D0C49CE
 P 1700 2500
-F 0 "#PWR0111" H 1700 2250 50  0001 C CNN
+F 0 "#PWR095" H 1700 2250 50  0001 C CNN
 F 1 "GND" H 1705 2327 50  0000 C CNN
 F 2 "" H 1700 2500 50  0001 C CNN
@@
 	1700 1450 1700 1500
 $Comp
-L power:+3V3 #PWR0108
+L power:+3V3 #PWR092
 U 1 1 5D0C524F
 P 2950 1450
-F 0 "#PWR0108" H 2950 1300 50  0001 C CNN
+F 0 "#PWR092" H 2950 1300 50  0001 C CNN
 F 1 "+3V3" H 2965 1623 50  0000 C CNN
 F 2 "" H 2950 1450 50  0001 C CNN
@@
 $EndComp
 $Comp
-L taobao-r:R103,0603 R24
+L taobao-r:R103,0603 R11
 U 1 1 5D0C5259
 P 2950 1600
-F 0 "R24" H 3009 1646 50  0000 L CNN
+F 0 "R11" H 3009 1646 50  0000 L CNN
 F 1 "R103,0603" H 3009 1555 50  0000 L CNN
 F 2 "Resistor_SMD:R_0603_1608Metric_Pad1.05x0.95mm_HandSolder" H 2950 1600 50  0001 C CNN
@@
 $EndComp
 $Comp
-L taobao-button:SW_RESET,2_leg,SMD SW16
+L taobao-button:SW_RESET,2_leg,SMD SW2
 U 1 1 5D0C5263
 P 2950 2150
-F 0 "SW16" V 2904 2298 50  0000 L CNN
+F 0 "SW2" V 2904 2298 50  0000 L CNN
 F 1 "USR_BTN_2" V 2995 2298 50  0000 L CNN
 F 2 "footprint-lib:SW_SPST_CK_RS282G05A3" H 2950 2350 50  0001 C CNN
@@
 $EndComp
 $Comp
-L power:GND #PWR0112
+L power:GND #PWR096
 U 1 1 5D0C526D
 P 2950 2500
-F 0 "#PWR0112" H 2950 2250 50  0001 C CNN
+F 0 "#PWR096" H 2950 2250 50  0001 C CNN
 F 1 "GND" H 2955 2327 50  0000 C CNN
 F 2 "" H 2950 2500 50  0001 C CNN
@@
 	2950 1450 2950 1500
 $Comp
-L power:+3V3 #PWR0109
+L power:+3V3 #PWR093
 U 1 1 5D0C5F20
 P 4100 1450
-F 0 "#PWR0109" H 4100 1300 50  0001 C CNN
+F 0 "#PWR093" H 4100 1300 50  0001 C CNN
 F 1 "+3V3" H 4115 1623 50  0000 C CNN
 F 2 "" H 4100 1450 50  0001 C CNN
@@
 $EndComp
 $Comp
-L taobao-r:R103,0603 R25
+L taobao-r:R103,0603 R12
 U 1 1 5D0C5F2A
 P 4100 1600
-F 0 "R25" H 4159 1646 50  0000 L CNN
+F 0 "R12" H 4159 1646 50  0000 L CNN
 F 1 "R103,0603" H 4159 1555 50  0000 L CNN
 F 2 "Resistor_SMD:R_0603_1608Metric_Pad1.05x0.95mm_HandSolder" H 4100 1600 50  0001 C CNN
@@
 $EndComp
 $Comp
-L taobao-button:SW_RESET,2_leg,SMD SW17
+L taobao-button:SW_RESET,2_leg,SMD SW3
 U 1 1 5D0C5F34
 P 4100 2150
-F 0 "SW17" V 4054 2298 50  0000 L CNN
+F 0 "SW3" V 4054 2298 50  0000 L CNN
 F 1 "USR_BTN_3" V 4145 2298 50  0000 L CNN
 F 2 "footprint-lib:SW_SPST_CK_RS282G05A3" H 4100 2350 50  0001 C CNN
@@
 $EndComp
 $Comp
-L power:GND #PWR0113
+L power:GND #PWR097
 U 1 1 5D0C5F3E
 P 4100 2500
-F 0 "#PWR0113" H 4100 2250 50  0001 C CNN
+F 0 "#PWR097" H 4100 2250 50  0001 C CNN
 F 1 "GND" H 4105 2327 50  0000 C CNN
 F 2 "" H 4100 2500 50  0001 C CNN
@@
 	4100 1450 4100 1500
 $Comp
-L power:+3V3 #PWR0110
+L power:+3V3 #PWR094
 U 1 1 5D0C5F4B
 P 5150 1450
-F 0 "#PWR0110" H 5150 1300 50  0001 C CNN
+F 0 "#PWR094" H 5150 1300 50  0001 C CNN
 F 1 "+3V3" H 5165 1623 50  0000 C CNN
 F 2 "" H 5150 1450 50  0001 C CNN
@@
 $EndComp
 $Comp
-L taobao-r:R103,0603 R26
+L taobao-r:R103,0603 R13
 U 1 1 5D0C5F55
 P 5150 1600
-F 0 "R26" H 5209 1646 50  0000 L CNN
+F 0 "R13" H 5209 1646 50  0000 L CNN
 F 1 "R103,0603" H 5209 1555 50  0000 L CNN
 F 2 "Resistor_SMD:R_0603_1608Metric_Pad1.05x0.95mm_HandSolder" H 5150 1600 50  0001 C CNN
@@
 $EndComp
 $Comp
-L taobao-button:SW_RESET,2_leg,SMD SW18
+L taobao-button:SW_RESET,2_leg,SMD SW4
 U 1 1 5D0C5F5F
 P 5150 2150
-F 0 "SW18" V 5104 2298 50  0000 L CNN
+F 0 "SW4" V 5104 2298 50  0000 L CNN
 F 1 "USR_BTN_4" V 5195 2298 50  0000 L CNN
 F 2 "footprint-lib:SW_SPST_CK_RS282G05A3" H 5150 2350 50  0001 C CNN
@@
 $EndComp
 $Comp
-L power:GND #PWR0114
+L power:GND #PWR098
 U 1 1 5D0C5F69
 P 5150 2500
-F 0 "#PWR0114" H 5150 2250 50  0001 C CNN
+F 0 "#PWR098" H 5150 2250 50  0001 C CNN
 F 1 "GND" H 5155 2327 50  0000 C CNN
 F 2 "" H 5150 2500 50  0001 C CNN

Commit message: update remote btn4 and all capacitor in place,
Parts:
- removed R13: R103,0603, Resistor_SMD:R_0603_1608Metric_Pad1.05x0.95mm_HandSolder, symbol taobao-r:R103,0603
- removed SW4: USR_BTN_4, footprint-lib:SW_SPST_CK_RS282G05A3, symbol taobao-button:SW_RESET,2_leg,SMD
Changed lines of the file:
@@
 Wire Wire Line
 	4100 1450 4100 1500
-$Comp
-L power:+3V3 #PWR094
-U 1 1 5D0C5F4B
-P 5150 1450
-F 0 "#PWR094" H 5150 1300 50  0001 C CNN
-F 1 "+3V3" H 5165 1623 50  0000 C CNN
-F 2 "" H 5150 1450 50  0001 C CNN
-F 3 "" H 5150 1450 50  0001 C CNN
-	1    5150 1450
-	1    0    0    -1
-$EndComp
-$Comp
-L taobao-r:R103,0603 R13
-U 1 1 5D0C5F55
-P 5150 1600
-F 0 "R13" H 5209 1646 50  0000 L CNN
-F 1 "R103,0603" H 5209 1555 50  0000 L CNN
-F 2 "Resistor_SMD:R_0603_1608Metric_Pad1.05x0.95mm_HandSolder" H 5150 1600 50  0001 C CNN
-F 3 "~" H 5150 1600 50  0001 C CNN
-	1    5150 1600
-	1    0    0    -1
-$EndComp
-$Comp
-L taobao-button:SW_RESET,2_leg,SMD SW4
-U 1 1 5D0C5F5F
-P 5150 2150
-F 0 "SW4" V 5104 2298 50  0000 L CNN
-F 1 "USR_BTN_4" V 5195 2298 50  0000 L CNN
-F 2 "footprint-lib:SW_SPST_CK_RS282G05A3" H 5150 2350 50  0001 C CNN
-F 3 "~" H 5150 2350 50  0001 C CNN
-	1    5150 2150
-	0    1    1    0
-$EndComp
-$Comp
-L power:GND #PWR098
-U 1 1 5D0C5F69
-P 5150 2500
-F 0 "#PWR098" H 5150 2250 50  0001 C CNN
-F 1 "GND" H 5155 2327 50  0000 C CNN
-F 2 "" H 5150 2500 50  0001 C CNN
-F 3 "" H 5150 2500 50  0001 C CNN
-	1    5150 2500
-	1    0    0    -1
-$EndComp
-Wire Wire Line
-	5150 2350 5150 2500
-Wire Wire Line
-	5150 1700 5150 1800
-Wire Wire Line
-	5150 1450 5150 1500
 Text HLabel 1000 650  0    50   Input ~ 0
 USR_BTN_1
@@
 Wire Wire Line
 	4100 1800 4100 1950
-Text Label 5650 1800 2    50   ~ 0
-USR_BTN_4
-Wire Wire Line
-	5650 1800 5150 1800
-Connection ~ 5150 1800
-Wire Wire Line
-	5150 1800 5150 1950
 $EndSCHEMATC
