File: hardware/rot_enc2.sch (KiCad schematic (older format))
At the start: 8 parts

Commit message: update for cherry key,wd
Parts:
- SW?: value EC11_VERTICAL -> ROT2
Changed lines of the file:
@@
 AR Path="/5CFF7883/5D0A34E5" Ref="SW?"  Part="1"
 F 0 "SW?" H 3900 2300 50  0000 C CNN
-F 1 "EC11_VERTICAL" H 3900 2400 50  0000 C CNN
+F 1 "ROT2" H 3900 2400 50  0000 C CNN
 F 2 "footprint-lib:RotaryEncoder_Alps_EC11E_Vertical_H20mm" H 3900 2350 50  0001 C CNN
 F 3 "https://item.taobao.com/item.htm?spm=a1z09.2.0.0.61152e8dxnonTp&id=532637189592&_u=rot8j1n8a4b" H 3900 2960 50  0001 C CNN

Commit message: update,
Parts:
- removed C?: C104,0603, Capacitor_SMD:C_0603_1608Metric_Pad1.05x0.95mm_HandSolder, symbol taobao-c:C104,0603
- removed J?: ROT_ENC_HEADER, Connector_PinHeader_1.27mm:PinHeader_1x03_P1.27mm_Vertical, symbol Connector:Conn_01x03_Female
- removed R?: R273,0603, Resistor_SMD:R_0603_1608Metric_Pad1.05x0.95mm_HandSolder, symbol taobao-r:R273,0603
- removed SW?: ROT2, footprint-lib:RotaryEncoder_Alps_EC11E_Vertical_H20mm, symbol taobao-components:EC11_VERTICAL
- added C43: C104,0603, Capacitor_SMD:C_0603_1608Metric_Pad1.05x0.95mm_HandSolder, symbol taobao-c:C104,0603
- added J5: ROT_ENC_HEADER, Connector_PinHeader_1.27mm:PinHeader_1x03_P1.27mm_Vertical, symbol Connector:Conn_01x03_Female
- added R28: R273,0603, Resistor_SMD:R_0603_1608Metric_Pad1.05x0.95mm_HandSolder, symbol taobao-r:R273,0603
- added SW19: ROT2, footprint-lib:RotaryEncoder_Alps_EC11E_Vertical_H20mm, symbol taobao-components:EC11_VERTICAL
- gave numbers to parts that had none: 4
Connections:
- net A: now also C43.1, J5.1 (Pin_1), R28.2
- net B: now also J5.2 (Pin_2)
- net GND: now also C43.2, SW19.C, SW19.E
- net SW_OUT: now also J5.3 (Pin_3)
- net at R29.1: now also SW19.A
- net at R30.1: now also SW19.D
- new net: R28.1, SW19.B
Changed lines of the file:
@@
 $Comp
 L taobao-components:EC11_VERTICAL SW?
-U 1 1 5D0A34E5
+U 1 1 5D32A3C7
 P 3900 2700
-AR Path="/5CF34744/5D0A34E5" Ref="SW?"  Part="1"
-AR Path="/5CFF7883/5D0A34E5" Ref="SW?"  Part="1"
-F 0 "SW?" H 3900 2300 50  0000 C CNN
+AR Path="/5CF34744/5D32A3C7" Ref="SW?"  Part="1"
+AR Path="/5CFF7883/5D32A3C7" Ref="SW19"  Part="1"
+F 0 "SW19" H 3900 2300 50  0000 C CNN
 F 1 "ROT2" H 3900 2400 50  0000 C CNN
 F 2 "footprint-lib:RotaryEncoder_Alps_EC11E_Vertical_H20mm" H 3900 2350 50  0001 C CNN
@@
 $Comp
 L taobao-r:R273,0603 R?
-U 1 1 5CED60AF
+U 1 1 5D32A3BB
 P 3150 2300
-AR Path="/5CF34744/5CED60AF" Ref="R?"  Part="1"
-AR Path="/5CFF7883/5CED60AF" Ref="R?"  Part="1"
-F 0 "R?" V 2900 2300 50  0000 C CNN
+AR Path="/5CF34744/5D32A3BB" Ref="R?"  Part="1"
+AR Path="/5CFF7883/5D32A3BB" Ref="R28"  Part="1"
+F 0 "R28" V 2900 2300 50  0000 C CNN
 F 1 "R273,0603" V 3000 2300 50  0000 C CNN
 F 2 "Resistor_SMD:R_0603_1608Metric_Pad1.05x0.95mm_HandSolder" H 3150 2300 50  0001 C CNN
@@
 P 3150 2800
 AR Path="/5CF34744/5CED6622" Ref="R?"  Part="1"
-AR Path="/5CFF7883/5CED6622" Ref="R?"  Part="1"
-F 0 "R?" V 2900 2800 50  0000 C CNN
+AR Path="/5CFF7883/5CED6622" Ref="R29"  Part="1"
+F 0 "R29" V 2900 2800 50  0000 C CNN
 F 1 "R273,0603" V 3000 2800 50  0000 C CNN
 F 2 "Resistor_SMD:R_0603_1608Metric_Pad1.05x0.95mm_HandSolder" H 3150 2800 50  0001 C CNN
@@
 P 3150 3250
 AR Path="/5CF34744/5CED67EF" Ref="R?"  Part="1"
-AR Path="/5CFF7883/5CED67EF" Ref="R?"  Part="1"
-F 0 "R?" V 2900 3250 50  0000 C CNN
+AR Path="/5CFF7883/5CED67EF" Ref="R30"  Part="1"
+F 0 "R30" V 2900 3250 50  0000 C CNN
 F 1 "R273,0603" V 3000 3250 50  0000 C CNN
 F 2 "Resistor_SMD:R_0603_1608Metric_Pad1.05x0.95mm_HandSolder" H 3150 3250 50  0001 C CNN
@@
 P 2800 3450
 AR Path="/5CF34744/5CED6CD1" Ref="C?"  Part="1"
-AR Path="/5CFF7883/5CED6CD1" Ref="C?"  Part="1"
-F 0 "C?" H 2900 3500 50  0000 L CNN
+AR Path="/5CFF7883/5CED6CD1" Ref="C45"  Part="1"
+F 0 "C45" H 2900 3500 50  0000 L CNN
 F 1 "C104,0603" H 2900 3450 50  0000 L CNN
 F 2 "Capacitor_SMD:C_0603_1608Metric_Pad1.05x0.95mm_HandSolder" H 2800 3450 50  0001 C CNN
@@
 P 2800 2950
 AR Path="/5CF34744/5CED7298" Ref="C?"  Part="1"
-AR Path="/5CFF7883/5CED7298" Ref="C?"  Part="1"
-F 0 "C?" H 2900 3000 50  0000 L CNN
+AR Path="/5CFF7883/5CED7298" Ref="C44"  Part="1"
+F 0 "C44" H 2900 3000 50  0000 L CNN
 F 1 "C104,0603" H 2900 2950 50  0000 L CNN
 F 2 "Capacitor_SMD:C_0603_1608Metric_Pad1.05x0.95mm_HandSolder" H 2800 2950 50  0001 C CNN
@@
 $Comp
 L taobao-c:C104,0603 C?
-U 1 1 5CED75A5
+U 1 1 5D32A3C0
 P 2800 2500
-AR Path="/5CF34744/5CED75A5" Ref="C?"  Part="1"
-AR Path="/5CFF7883/5CED75A5" Ref="C?"  Part="1"
-F 0 "C?" H 2900 2550 50  0000 L CNN
+AR Path="/5CF34744/5D32A3C0" Ref="C?"  Part="1"
+AR Path="/5CFF7883/5D32A3C0" Ref="C43"  Part="1"
+F 0 "C43" H 2900 2550 50  0000 L CNN
 F 1 "C104,0603" H 2900 2500 50  0000 L CNN
 F 2 "Capacitor_SMD:C_0603_1608Metric_Pad1.05x0.95mm_HandSolder" H 2800 2500 50  0001 C CNN
@@
 $Comp
 L power:GND #PWR?
-U 1 1 5CED86F3
+U 1 1 5D32A3C1
 P 2800 2650
-AR Path="/5CF34744/5CED86F3" Ref="#PWR?"  Part="1"
-AR Path="/5CFF7883/5CED86F3" Ref="#PWR?"  Part="1"
-F 0 "#PWR?" H 2800 2400 50  0001 C CNN
+AR Path="/5CF34744/5D32A3C1" Ref="#PWR?"  Part="1"
+AR Path="/5CFF7883/5D32A3C1" Ref="#PWR0123"  Part="1"
+F 0 "#PWR0123" H 2800 2400 50  0001 C CNN
 F 1 "GND" H 2850 2450 50  0000 C CNN
 F 2 "" H 2800 2650 50  0001 C CNN
@@
 P 2800 3100
 AR Path="/5CF34744/5CED8B04" Ref="#PWR?"  Part="1"
-AR Path="/5CFF7883/5CED8B04" Ref="#PWR?"  Part="1"
-F 0 "#PWR?" H 2800 2850 50  0001 C CNN
+AR Path="/5CFF7883/5CED8B04" Ref="#PWR0125"  Part="1"
+F 0 "#PWR0125" H 2800 2850 50  0001 C CNN
 F 1 "GND" H 2850 2900 50  0000 C CNN
 F 2 "" H 2800 3100 50  0001 C CNN
@@
 $Comp
 L power:GND #PWR?
-U 1 1 5CED8F95
+U 1 1 5D32A3C3
 P 2800 3600
-AR Path="/5CF34744/5CED8F95" Ref="#PWR?"  Part="1"
-AR Path="/5CFF7883/5CED8F95" Ref="#PWR?"  Part="1"
-F 0 "#PWR?" H 2800 3350 50  0001 C CNN
+AR Path="/5CF34744/5D32A3C3" Ref="#PWR?"  Part="1"
+AR Path="/5CFF7883/5D32A3C3" Ref="#PWR0126"  Part="1"
+F 0 "#PWR0126" H 2800 3350 50  0001 C CNN
 F 1 "GND" H 2850 3400 50  0000 C CNN
 F 2 "" H 2800 3600 50  0001 C CNN
@@
 $Comp
 L power:GND #PWR?
-U 1 1 5CED947F
+U 1 1 5D32A3C4
 P 3350 2600
-AR Path="/5CF34744/5CED947F" Ref="#PWR?"  Part="1"
-AR Path="/5CFF7883/5CED947F" Ref="#PWR?"  Part="1"
-F 0 "#PWR?" H 3350 2350 50  0001 C CNN
+AR Path="/5CF34744/5D32A3C4" Ref="#PWR?"  Part="1"
+AR Path="/5CFF7883/5D32A3C4" Ref="#PWR0122"  Part="1"
+F 0 "#PWR0122" H 3350 2350 50  0001 C CNN
 F 1 "GND" H 3400 2400 50  0000 C CNN
 F 2 "" H 3350 2600 50  0001 C CNN
@@
 P 4400 2900
 AR Path="/5CF34744/5CED96CA" Ref="#PWR?"  Part="1"
-AR Path="/5CFF7883/5CED96CA" Ref="#PWR?"  Part="1"
-F 0 "#PWR?" H 4400 2650 50  0001 C CNN
+AR Path="/5CFF7883/5CED96CA" Ref="#PWR0124"  Part="1"
+F 0 "#PWR0124" H 4400 2650 50  0001 C CNN
 F 1 "GND" H 4450 2700 50  0000 C CNN
 F 2 "" H 4400 2900 50  0001 C CNN
@@
 $Comp
 L Connector:Conn_01x03_Female J?
-U 1 1 5CF225E9
+U 1 1 5D32A3C6
 P 1100 2200
-AR Path="/5CF34744/5CF225E9" Ref="J?"  Part="1"
-AR Path="/5CFF7883/5CF225E9" Ref="J?"  Part="1"
-F 0 "J?" H 950 2500 50  0000 C CNN
+AR Path="/5CF34744/5D32A3C6" Ref="J?"  Part="1"
+AR Path="/5CFF7883/5D32A3C6" Ref="J5"  Part="1"
+F 0 "J5" H 950 2500 50  0000 C CNN
 F 1 "ROT_ENC_HEADER" H 950 2400 50  0000 C CNN
 F 2 "Connector_PinHeader_1.27mm:PinHeader_1x03_P1.27mm_Vertical" H 1100 2200 50  0001 C CNN
