File: hardware/rot_enc2.sch (KiCad schematic (older format))
At the start: 8 parts, among them J5 ROT_ENC_HEADER, SW19 ROT2

Commit message: update,
Parts:
- renumbered C43 to C26, C44 to C27, C45 to C28, J5 to J4, R28 to R16, R29 to R17, R30 to R18, SW19 to SW5
Changed lines of the file:
@@
 P 3900 2700
 AR Path="/5CF34744/5D32A3C7" Ref="SW?"  Part="1"
-AR Path="/5CFF7883/5D32A3C7" Ref="SW19"  Part="1"
-F 0 "SW19" H 3900 2300 50  0000 C CNN
+AR Path="/5CFF7883/5D32A3C7" Ref="SW5"  Part="1"
+F 0 "SW5" H 3900 2300 50  0000 C CNN
 F 1 "ROT2" H 3900 2400 50  0000 C CNN
 F 2 "footprint-lib:RotaryEncoder_Alps_EC11E_Vertical_H20mm" H 3900 2350 50  0001 C CNN
@@
 P 3150 2300
 AR Path="/5CF34744/5D32A3BB" Ref="R?"  Part="1"
-AR Path="/5CFF7883/5D32A3BB" Ref="R28"  Part="1"
-F 0 "R28" V 2900 2300 50  0000 C CNN
+AR Path="/5CFF7883/5D32A3BB" Ref="R16"  Part="1"
+F 0 "R16" V 2900 2300 50  0000 C CNN
 F 1 "R273,0603" V 3000 2300 50  0000 C CNN
 F 2 "Resistor_SMD:R_0603_1608Metric_Pad1.05x0.95mm_HandSolder" H 3150 2300 50  0001 C CNN
@@
 P 3150 2800
 AR Path="/5CF34744/5CED6622" Ref="R?"  Part="1"
-AR Path="/5CFF7883/5CED6622" Ref="R29"  Part="1"
-F 0 "R29" V 2900 2800 50  0000 C CNN
+AR Path="/5CFF7883/5CED6622" Ref="R17"  Part="1"
+F 0 "R17" V 2900 2800 50  0000 C CNN
 F 1 "R273,0603" V 3000 2800 50  0000 C CNN
 F 2 "Resistor_SMD:R_0603_1608Metric_Pad1.05x0.95mm_HandSolder" H 3150 2800 50  0001 C CNN
@@
 P 3150 3250
 AR Path="/5CF34744/5CED67EF" Ref="R?"  Part="1"
-AR Path="/5CFF7883/5CED67EF" Ref="R30"  Part="1"
-F 0 "R30" V 2900 3250 50  0000 C CNN
+AR Path="/5CFF7883/5CED67EF" Ref="R18"  Part="1"
+F 0 "R18" V 2900 3250 50  0000 C CNN
 F 1 "R273,0603" V 3000 3250 50  0000 C CNN
 F 2 "Resistor_SMD:R_0603_1608Metric_Pad1.05x0.95mm_HandSolder" H 3150 3250 50  0001 C CNN
@@
 P 2800 3450
 AR Path="/5CF34744/5CED6CD1" Ref="C?"  Part="1"
-AR Path="/5CFF7883/5CED6CD1" Ref="C45"  Part="1"
-F 0 "C45" H 2900 3500 50  0000 L CNN
+AR Path="/5CFF7883/5CED6CD1" Ref="C28"  Part="1"
+F 0 "C28" H 2900 3500 50  0000 L CNN
 F 1 "C104,0603" H 2900 3450 50  0000 L CNN
 F 2 "Capacitor_SMD:C_0603_1608Metric_Pad1.05x0.95mm_HandSolder" H 2800 3450 50  0001 C CNN
@@
 P 2800 2950
 AR Path="/5CF34744/5CED7298" Ref="C?"  Part="1"
-AR Path="/5CFF7883/5CED7298" Ref="C44"  Part="1"
-F 0 "C44" H 2900 3000 50  0000 L CNN
+AR Path="/5CFF7883/5CED7298" Ref="C27"  Part="1"
+F 0 "C27" H 2900 3000 50  0000 L CNN
 F 1 "C104,0603" H 2900 2950 50  0000 L CNN
 F 2 "Capacitor_SMD:C_0603_1608Metric_Pad1.05x0.95mm_HandSolder" H 2800 2950 50  0001 C CNN
@@
 P 2800 2500
 AR Path="/5CF34744/5D32A3C0" Ref="C?"  Part="1"
-AR Path="/5CFF7883/5D32A3C0" Ref="C43"  Part="1"
-F 0 "C43" H 2900 2550 50  0000 L CNN
+AR Path="/5CFF7883/5D32A3C0" Ref="C26"  Part="1"
+F 0 "C26" H 2900 2550 50  0000 L CNN
 F 1 "C104,0603" H 2900 2500 50  0000 L CNN
 F 2 "Capacitor_SMD:C_0603_1608Metric_Pad1.05x0.95mm_HandSolder" H 2800 2500 50  0001 C CNN
@@
 P 2800 2650
 AR Path="/5CF34744/5D32A3C1" Ref="#PWR?"  Part="1"
-AR Path="/5CFF7883/5D32A3C1" Ref="#PWR0123"  Part="1"
-F 0 "#PWR0123" H 2800 2400 50  0001 C CNN
+AR Path="/5CFF7883/5D32A3C1" Ref="#PWR0110"  Part="1"
+F 0 "#PWR0110" H 2800 2400 50  0001 C CNN
 F 1 "GND" H 2850 2450 50  0000 C CNN
 F 2 "" H 2800 2650 50  0001 C CNN
@@
 P 2800 3100
 AR Path="/5CF34744/5CED8B04" Ref="#PWR?"  Part="1"
-AR Path="/5CFF7883/5CED8B04" Ref="#PWR0125"  Part="1"
-F 0 "#PWR0125" H 2800 2850 50  0001 C CNN
+AR Path="/5CFF7883/5CED8B04" Ref="#PWR0112"  Part="1"
+F 0 "#PWR0112" H 2800 2850 50  0001 C CNN
 F 1 "GND" H 2850 2900 50  0000 C CNN
 F 2 "" H 2800 3100 50  0001 C CNN
@@
 P 2800 3600
 AR Path="/5CF34744/5D32A3C3" Ref="#PWR?"  Part="1"
-AR Path="/5CFF7883/5D32A3C3" Ref="#PWR0126"  Part="1"
-F 0 "#PWR0126" H 2800 3350 50  0001 C CNN
+AR Path="/5CFF7883/5D32A3C3" Ref="#PWR0113"  Part="1"
+F 0 "#PWR0113" H 2800 3350 50  0001 C CNN
 F 1 "GND" H 2850 3400 50  0000 C CNN
 F 2 "" H 2800 3600 50  0001 C CNN
@@
 P 3350 2600
 AR Path="/5CF34744/5D32A3C4" Ref="#PWR?"  Part="1"
-AR Path="/5CFF7883/5D32A3C4" Ref="#PWR0122"  Part="1"
-F 0 "#PWR0122" H 3350 2350 50  0001 C CNN
+AR Path="/5CFF7883/5D32A3C4" Ref="#PWR0109"  Part="1"
+F 0 "#PWR0109" H 3350 2350 50  0001 C CNN
 F 1 "GND" H 3400 2400 50  0000 C CNN
 F 2 "" H 3350 2600 50  0001 C CNN
@@
 P 4400 2900
 AR Path="/5CF34744/5CED96CA" Ref="#PWR?"  Part="1"
-AR Path="/5CFF7883/5CED96CA" Ref="#PWR0124"  Part="1"
-F 0 "#PWR0124" H 4400 2650 50  0001 C CNN
+AR Path="/5CFF7883/5CED96CA" Ref="#PWR0111"  Part="1"
+F 0 "#PWR0111" H 4400 2650 50  0001 C CNN
 F 1 "GND" H 4450 2700 50  0000 C CNN
 F 2 "" H 4400 2900 50  0001 C CNN
@@
 P 1100 2200
 AR Path="/5CF34744/5D32A3C6" Ref="J?"  Part="1"
-AR Path="/5CFF7883/5D32A3C6" Ref="J5"  Part="1"
-F 0 "J5" H 950 2500 50  0000 C CNN
+AR Path="/5CFF7883/5D32A3C6" Ref="J4"  Part="1"
+F 0 "J4" H 950 2500 50  0000 C CNN
 F 1 "ROT_ENC_HEADER" H 950 2400 50  0000 C CNN
 F 2 "Connector_PinHeader_1.27mm:PinHeader_1x03_P1.27mm_Vertical" H 1100 2200 50  0001 C CNN

Commit message: update for tidy tracks,
Connections:
- net A: now also C27.1, R17.2; no longer C26.1, R16.2
- net B: now also C26.1, R16.2; no longer C27.1, R17.2
Changed lines of the file:
@@
 Wire Wire Line
 	4300 3250 3250 3250
+Text Label 2000 2800 0    50   ~ 0
+ROT_ENC_A
 Text Label 2000 2300 0    50   ~ 0
-ROT_ENC_A
-Text Label 2000 2800 0    50   ~ 0
 ROT_ENC_B
 Text Label 2000 3250 0    50   ~ 0
