File: hardware/status_display.sch (KiCad schematic (older format))
At the start: 6 parts

Commit message: update,
Parts:
- gave numbers to parts that had none: 6
Changed lines of the file:
@@
 $EndDescr
 $Comp
-L power:+3V3 #PWR?
+L power:+3V3 #PWR046
 U 1 1 5D0EA4C1
 P 2050 1600
-F 0 "#PWR?" H 2050 1450 50  0001 C CNN
+F 0 "#PWR046" H 2050 1450 50  0001 C CNN
 F 1 "+3V3" H 2065 1773 50  0000 C CNN
 F 2 "" H 2050 1600 50  0001 C CNN
@@
 $EndComp
 $Comp
-L taobao-led:LED_GREEN,0603 D?
+L taobao-led:LED_GREEN,0603 D16
 U 1 1 5D0EAAE1
 P 2050 2150
-F 0 "D?" V 2096 2082 50  0000 R CNN
+F 0 "D16" V 2096 2082 50  0000 R CNN
 F 1 "USR_LED_1" V 2005 2082 50  0000 R CNN
 F 2 "footprint-lib:LED_0603_1608Metric" V 2050 2150 50  0001 C CNN
@@
 $EndComp
 $Comp
-L taobao-r:R103,0603 R?
+L taobao-r:R103,0603 R20
 U 1 1 5D0EB0E2
 P 2050 1850
-F 0 "R?" H 2109 1896 50  0000 L CNN
+F 0 "R20" H 2109 1896 50  0000 L CNN
 F 1 "R103,0603" H 2109 1805 50  0000 L CNN
 F 2 "Resistor_SMD:R_0603_1608Metric_Pad1.05x0.95mm_HandSolder" H 2050 1850 50  0001 C CNN
@@
 	2050 1600 2050 1750
 $Comp
-L power:+3V3 #PWR?
+L power:+3V3 #PWR047
 U 1 1 5D0EC06B
 P 3200 1600
-F 0 "#PWR?" H 3200 1450 50  0001 C CNN
+F 0 "#PWR047" H 3200 1450 50  0001 C CNN
 F 1 "+3V3" H 3215 1773 50  0000 C CNN
 F 2 "" H 3200 1600 50  0001 C CNN
@@
 $EndComp
 $Comp
-L taobao-led:LED_GREEN,0603 D?
+L taobao-led:LED_GREEN,0603 D17
 U 1 1 5D0EC075
 P 3200 2150
-F 0 "D?" V 3246 2082 50  0000 R CNN
+F 0 "D17" V 3246 2082 50  0000 R CNN
 F 1 "USR_LED_2" V 3155 2082 50  0000 R CNN
 F 2 "footprint-lib:LED_0603_1608Metric" V 3200 2150 50  0001 C CNN
@@
 $EndComp
 $Comp
-L taobao-r:R103,0603 R?
+L taobao-r:R103,0603 R21
 U 1 1 5D0EC07F
 P 3200 1850
-F 0 "R?" H 3259 1896 50  0000 L CNN
+F 0 "R21" H 3259 1896 50  0000 L CNN
 F 1 "R103,0603" H 3259 1805 50  0000 L CNN
 F 2 "Resistor_SMD:R_0603_1608Metric_Pad1.05x0.95mm_HandSolder" H 3200 1850 50  0001 C CNN
@@
 	3200 1600 3200 1750
 $Comp
-L power:+3V3 #PWR?
+L power:+3V3 #PWR048
 U 1 1 5D0EC76C
 P 4300 1600
-F 0 "#PWR?" H 4300 1450 50  0001 C CNN
+F 0 "#PWR048" H 4300 1450 50  0001 C CNN
 F 1 "+3V3" H 4315 1773 50  0000 C CNN
 F 2 "" H 4300 1600 50  0001 C CNN
@@
 $EndComp
 $Comp
-L taobao-led:LED_GREEN,0603 D?
+L taobao-led:LED_GREEN,0603 D18
 U 1 1 5D0EC776
 P 4300 2150
-F 0 "D?" V 4346 2082 50  0000 R CNN
+F 0 "D18" V 4346 2082 50  0000 R CNN
 F 1 "USR_LED_3" V 4255 2082 50  0000 R CNN
 F 2 "footprint-lib:LED_0603_1608Metric" V 4300 2150 50  0001 C CNN
@@
 $EndComp
 $Comp
-L taobao-r:R103,0603 R?
+L taobao-r:R103,0603 R22
 U 1 1 5D0EC780
 P 4300 1850
-F 0 "R?" H 4359 1896 50  0000 L CNN
+F 0 "R22" H 4359 1896 50  0000 L CNN
 F 1 "R103,0603" H 4359 1805 50  0000 L CNN
 F 2 "Resistor_SMD:R_0603_1608Metric_Pad1.05x0.95mm_HandSolder" H 4300 1850 50  0001 C CNN
