File: hardware/status_display.sch (KiCad schematic (older format))
At the start: 6 parts

Commit message: update,
Parts:
- added C56: C106,0603, Capacitor_SMD:C_0603_1608Metric_Pad1.05x0.95mm_HandSolder, symbol taobao-c:C106,0603
Connections:
- net +3V3: now also C56.1
- new net GND: C56.2
Changed lines of the file:
@@
 Text HLabel 1000 900  0    50   Input ~ 0
 USR_LED_3
+$Comp
+L power:+3V3 #PWR0160
+U 1 1 5D5FA30F
+P 5450 1600
+F 0 "#PWR0160" H 5450 1450 50  0001 C CNN
+F 1 "+3V3" H 5465 1773 50  0000 C CNN
+F 2 "" H 5450 1600 50  0001 C CNN
+F 3 "" H 5450 1600 50  0001 C CNN
+	1    5450 1600
+	1    0    0    -1
+$EndComp
+$Comp
+L taobao-c:C106,0603 C56
+U 1 1 5D5FA71C
+P 5450 1800
+F 0 "C56" H 5542 1846 50  0000 L CNN
+F 1 "C106,0603" H 5542 1755 50  0000 L CNN
+F 2 "Capacitor_SMD:C_0603_1608Metric_Pad1.05x0.95mm_HandSolder" H 5450 1800 50  0001 C CNN
+F 3 "~" H 5450 1800 50  0001 C CNN
+	1    5450 1800
+	1    0    0    -1
+$EndComp
+$Comp
+L power:GND #PWR0161
+U 1 1 5D5FAE0A
+P 5450 2050
+F 0 "#PWR0161" H 5450 1800 50  0001 C CNN
+F 1 "GND" H 5455 1877 50  0000 C CNN
+F 2 "" H 5450 2050 50  0001 C CNN
+F 3 "" H 5450 2050 50  0001 C CNN
+	1    5450 2050
+	1    0    0    -1
+$EndComp
+Wire Wire Line
+	5450 1900 5450 2050
+Wire Wire Line
+	5450 1600 5450 1700
 $EndSCHEMATC

Commit message: update,
Other:
- moved on the sheet: C56
Changed lines of the file:
@@
 L power:+3V3 #PWR0160
 U 1 1 5D5FA30F
-P 5450 1600
-F 0 "#PWR0160" H 5450 1450 50  0001 C CNN
-F 1 "+3V3" H 5465 1773 50  0000 C CNN
-F 2 "" H 5450 1600 50  0001 C CNN
-F 3 "" H 5450 1600 50  0001 C CNN
-	1    5450 1600
+P 5200 1750
+F 0 "#PWR0160" H 5200 1600 50  0001 C CNN
+F 1 "+3V3" H 5215 1923 50  0000 C CNN
+F 2 "" H 5200 1750 50  0001 C CNN
+F 3 "" H 5200 1750 50  0001 C CNN
+	1    5200 1750
 	1    0    0    -1
 $EndComp
@@
 L taobao-c:C106,0603 C56
 U 1 1 5D5FA71C
-P 5450 1800
-F 0 "C56" H 5542 1846 50  0000 L CNN
-F 1 "C106,0603" H 5542 1755 50  0000 L CNN
-F 2 "Capacitor_SMD:C_0603_1608Metric_Pad1.05x0.95mm_HandSolder" H 5450 1800 50  0001 C CNN
-F 3 "~" H 5450 1800 50  0001 C CNN
-	1    5450 1800
+P 5200 1950
+F 0 "C56" H 5292 1996 50  0000 L CNN
+F 1 "C106,0603" H 5292 1905 50  0000 L CNN
+F 2 "Capacitor_SMD:C_0603_1608Metric_Pad1.05x0.95mm_HandSolder" H 5200 1950 50  0001 C CNN
+F 3 "~" H 5200 1950 50  0001 C CNN
+	1    5200 1950
 	1    0    0    -1
 $EndComp
@@
 L power:GND #PWR0161
 U 1 1 5D5FAE0A
-P 5450 2050
-F 0 "#PWR0161" H 5450 1800 50  0001 C CNN
-F 1 "GND" H 5455 1877 50  0000 C CNN
-F 2 "" H 5450 2050 50  0001 C CNN
-F 3 "" H 5450 2050 50  0001 C CNN
-	1    5450 2050
+P 5200 2200
+F 0 "#PWR0161" H 5200 1950 50  0001 C CNN
+F 1 "GND" H 5205 2027 50  0000 C CNN
+F 2 "" H 5200 2200 50  0001 C CNN
+F 3 "" H 5200 2200 50  0001 C CNN
+	1    5200 2200
 	1    0    0    -1
 $EndComp
 Wire Wire Line
-	5450 1900 5450 2050
+	5200 2050 5200 2200
 Wire Wire Line
-	5450 1600 5450 1700
+	5200 1750 5200 1850
 $EndSCHEMATC

Commit message: update,
Parts:
- renumbered C56 to C5, D16 to D3, D17 to D4, D18 to D5, R20 to R7, R21 to R8, R22 to R9
Changed lines of the file:
@@
 $EndDescr
 $Comp
-L power:+3V3 #PWR046
+L power:+3V3 #PWR026
 U 1 1 5D0EA4C1
 P 2050 1600
-F 0 "#PWR046" H 2050 1450 50  0001 C CNN
+F 0 "#PWR026" H 2050 1450 50  0001 C CNN
 F 1 "+3V3" H 2065 1773 50  0000 C CNN
 F 2 "" H 2050 1600 50  0001 C CNN
@@
 $EndComp
 $Comp
-L taobao-led:LED_GREEN,0603 D16
+L taobao-led:LED_GREEN,0603 D3
 U 1 1 5D0EAAE1
 P 2050 2150
-F 0 "D16" V 2096 2082 50  0000 R CNN
+F 0 "D3" V 2096 2082 50  0000 R CNN
 F 1 "USR_LED_1" V 2005 2082 50  0000 R CNN
 F 2 "footprint-lib:LED_0603_1608Metric" V 2050 2150 50  0001 C CNN
@@
 $EndComp
 $Comp
-L taobao-r:R103,0603 R20
+L taobao-r:R103,0603 R7
 U 1 1 5D0EB0E2
 P 2050 1850
-F 0 "R20" H 2109 1896 50  0000 L CNN
+F 0 "R7" H 2109 1896 50  0000 L CNN
 F 1 "R103,0603" H 2109 1805 50  0000 L CNN
 F 2 "Resistor_SMD:R_0603_1608Metric_Pad1.05x0.95mm_HandSolder" H 2050 1850 50  0001 C CNN
@@
 	2050 1600 2050 1750
 $Comp
-L power:+3V3 #PWR047
+L power:+3V3 #PWR027
 U 1 1 5D0EC06B
 P 3200 1600
-F 0 "#PWR047" H 3200 1450 50  0001 C CNN
+F 0 "#PWR027" H 3200 1450 50  0001 C CNN
 F 1 "+3V3" H 3215 1773 50  0000 C CNN
 F 2 "" H 3200 1600 50  0001 C CNN
@@
 $EndComp
 $Comp
-L taobao-led:LED_GREEN,0603 D17
+L taobao-led:LED_GREEN,0603 D4
 U 1 1 5D0EC075
 P 3200 2150
-F 0 "D17" V 3246 2082 50  0000 R CNN
+F 0 "D4" V 3246 2082 50  0000 R CNN
 F 1 "USR_LED_2" V 3155 2082 50  0000 R CNN
 F 2 "footprint-lib:LED_0603_1608Metric" V 3200 2150 50  0001 C CNN
@@
 $EndComp
 $Comp
-L taobao-r:R103,0603 R21
+L taobao-r:R103,0603 R8
 U 1 1 5D0EC07F
 P 3200 1850
-F 0 "R21" H 3259 1896 50  0000 L CNN
+F 0 "R8" H 3259 1896 50  0000 L CNN
 F 1 "R103,0603" H 3259 1805 50  0000 L CNN
 F 2 "Resistor_SMD:R_0603_1608Metric_Pad1.05x0.95mm_HandSolder" H 3200 1850 50  0001 C CNN
@@
 	3200 1600 3200 1750
 $Comp
-L power:+3V3 #PWR048
+L power:+3V3 #PWR028
 U 1 1 5D0EC76C
 P 4300 1600
-F 0 "#PWR048" H 4300 1450 50  0001 C CNN
+F 0 "#PWR028" H 4300 1450 50  0001 C CNN
 F 1 "+3V3" H 4315 1773 50  0000 C CNN
 F 2 "" H 4300 1600 50  0001 C CNN
@@
 $EndComp
 $Comp
-L taobao-led:LED_GREEN,0603 D18
+L taobao-led:LED_GREEN,0603 D5
 U 1 1 5D0EC776
 P 4300 2150
-F 0 "D18" V 4346 2082 50  0000 R CNN
+F 0 "D5" V 4346 2082 50  0000 R CNN
 F 1 "USR_LED_3" V 4255 2082 50  0000 R CNN
 F 2 "footprint-lib:LED_0603_1608Metric" V 4300 2150 50  0001 C CNN
@@
 $EndComp
 $Comp
-L taobao-r:R103,0603 R22
+L taobao-r:R103,0603 R9
 U 1 1 5D0EC780
 P 4300 1850
-F 0 "R22" H 4359 1896 50  0000 L CNN
+F 0 "R9" H 4359 1896 50  0000 L CNN
 F 1 "R103,0603" H 4359 1805 50  0000 L CNN
 F 2 "Resistor_SMD:R_0603_1608Metric_Pad1.05x0.95mm_HandSolder" H 4300 1850 50  0001 C CNN
@@
 USR_LED_3
 $Comp
-L power:+3V3 #PWR0160
+L power:+3V3 #PWR029
 U 1 1 5D5FA30F
 P 5200 1750
-F 0 "#PWR0160" H 5200 1600 50  0001 C CNN
+F 0 "#PWR029" H 5200 1600 50  0001 C CNN
 F 1 "+3V3" H 5215 1923 50  0000 C CNN
 F 2 "" H 5200 1750 50  0001 C CNN
@@
 $EndComp
 $Comp
-L taobao-c:C106,0603 C56
+L taobao-c:C106,0603 C5
 U 1 1 5D5FA71C
 P 5200 1950
-F 0 "C56" H 5292 1996 50  0000 L CNN
+F 0 "C5" H 5292 1996 50  0000 L CNN
 F 1 "C106,0603" H 5292 1905 50  0000 L CNN
 F 2 "Capacitor_SMD:C_0603_1608Metric_Pad1.05x0.95mm_HandSolder" H 5200 1950 50  0001 C CNN
@@
 $EndComp
 $Comp
-L power:GND #PWR0161
+L power:GND #PWR030
 U 1 1 5D5FAE0A
 P 5200 2200
-F 0 "#PWR0161" H 5200 1950 50  0001 C CNN
+F 0 "#PWR030" H 5200 1950 50  0001 C CNN
 F 1 "GND" H 5205 2027 50  0000 C CNN
 F 2 "" H 5200 2200 50  0001 C CNN
