File: hardware/stm32_swd.sch (KiCad schematic (older format))
At the start: 2 parts

Commit message: update,
Parts:
- removed U?: USB_Micro, footprint-lib:USB_Micro-B_Molex-105017-0001, symbol taobao-components:USB_Micro
- removed U?: TPD4S012, footprints-lib:TPD4S012, symbol taobao-components:TPD4S012
- added C?: C105, Capacitor_SMD:C_0603_1608Metric_Pad1.05x0.95mm_HandSolder, symbol taobao-c:C105
- added C? (x2): CP100uf,16V, Capacitor_SMD:CP_Elec_6.3x5.3, symbol taobao-cp:CP100uf,16V
- added C? (x2): C20pf,0603, Capacitor_SMD:C_0603_1608Metric_Pad1.05x0.95mm_HandSolder, symbol taobao-c:C20pf,0603
- added C? (x5): C104,0603, Capacitor_SMD:C_0603_1608Metric_Pad1.05x0.95mm_HandSolder, symbol taobao-c:C104,0603
- added J?: SWD_HEADER, footprint-lib:BLUEPILL_SWD, symbol taobao-components:BLUEPILL_SWD
- added R? (x2): R221,0603, Resistor_SMD:R_0603_1608Metric_Pad1.05x0.95mm_HandSolder, symbol taobao-r:R221,0603
- added R? (x3): R104,0603, Resistor_SMD:R_0603_1608Metric_Pad1.05x0.95mm_HandSolder, symbol taobao-r:R104,0603
- added R?: R101,0603, Resistor_SMD:R_0603_1608Metric_Pad1.05x0.95mm_HandSolder, symbol taobao-r:R101,0603
- added RN?: RN_221,0603, Resistor_SMD:R_Array_Concave_4x0603, symbol taobao-rpack:RN_221,0603
- added RN?: RN_4R7,0603, Resistor_SMD:R_Array_Concave_4x0603, symbol taobao-rpack:RN_4R7,0603
- added TP?: TP_VUSB1, TestPoint:TestPoint_THTPad_D2.0mm_Drill1.0mm, symbol my_testpoint:TestPoint_2mm
- added U?: AMS1117-3.3, Package_TO_SOT_SMD:SOT-223-3_TabPin2, symbol Regulator_Linear:AMS1117-3.3
- added U?: STM32F103C8T6_rect, footprint-lib:STM32F103C8T6, symbol taobao-components:STM32F103C8T6_rect
- added U?: USB_Micro, footprint-lib:USB_Micro-B_Molex-105017-0001, symbol taobao-components:USB_Micro
- added U?: USBLC6-2SC6_SOT23-6, footprints-lib:USBLC6-2, symbol taobao-components:USBLC6-2SC6_SOT23-6
- added VUSB1_HEALTHY, VUSB1_HEALTHY?: LED_GREEN,0603, footprint-lib:LED_0603_1608Metric, symbol taobao-led:LED_GREEN,0603
- added Y?: O_8M, Crystal:Crystal_HC49-4H_Vertical, symbol taobao-osc:O_8M
Connections:
- net GND: now also C?.1, C?.1, C?.1, C?.1, C?.2, C?.2, C?.2, C?.2, C?.2, C?.2, J?.1 (Pin_1), R?.1, R?.1, RN?.2 (R2.1), U?.1 (GND), U?.2 (GND), U?.20 (PB2/BOOT1), U?.23 (VSS_1), U?.35 (VSS_2), U?.47 (VSS_3), U?.5 (GND), U?.6 (MH1), U?.7 (MH2), U?.8 (MH3), U?.8 (VSSA), U?.9 (MH4), VUSB1_HEALTHY.1 (K), VUSB1_HEALTHY?.1 (K)
- net USB_N: now also RN?.8 (R1.2)
- net USB_P: now also RN?.7 (R2.2)
- new net: RN?.7 (R2.2), RN?.8 (R1.2), U?.10 (PA0-ADC0/WKUP/USART2CTS/TIM2CH1ETR)
- new net: R?.2, U?.2 (PC13-TAMPER-RTC)
- new net: R?.2, U?.25 (PB12-SPI2NSS)
- new net: R?.2, U?.44 (BOOT0)
- new net: C?.2, U?.5 (PD0-OSCIN), Y?.2
- new net: C?.2, U?.6 (PD1-OSCOUT), Y?.1
- new net: C?.1, R?.2, U?.7 (NRST)
- new net: U?.1 (I/O1), U?.2 (D-)
- new net: U?.3 (D+), U?.3 (I/O2)
- new net: RN?.1 (R1.1), U?.4 (I/O2)
- new net: RN?.2 (R2.1), U?.6 (I/O1)
- new net: R?.1, VUSB1_HEALTHY.2 (A)
- new net: R?.1, VUSB1_HEALTHY?.2 (A)
- new net LED_STLINK: U?.30 (PA9-TIM1CH2/USART1TX)
- new net SWCLK: J?.2 (Pin_2), U?.37 (PA14-JTCK/SWCLK)
- new net SWDIO: J?.3 (Pin_3), U?.34 (PA13-JTMS/SWDIO)
- new net T_JTCK: U?.26 (PB13-SPI2SCK)
- new net T_JTMS: R?.1, U?.27 (PB14-SPI2MISO)
- new net USB_DM: U?.32 (PA11-USART1CTS/TIM1CH4/USBDM)
- new net USB_DP: U?.33 (PA12-USART1RTS/USBDP)
- new net Vstm32_stlink: C?.1, C?.1, C?.1, C?.1, C?.2, C?.2, J?.4 (Pin_4), R?.1, R?.2, RN?.1 (R1.1), U?.1 (VBAT), U?.2 (VO), U?.24 (VDD_1), U?.36 (VDD_2), U?.48 (VDD_3), U?.9 (VDDA)
- new net Vusb_1: C?.1, R?.2, TP?.1, U?.1 (VCC), U?.3 (VI), U?.5 (Vbus)

Commit message: update,
Parts:
- added D?: LED_GREEN,0603, footprint-lib:LED_0603_1608Metric, symbol taobao-led:LED_GREEN,0603
- added D?: LED_RED,0603, footprint-lib:LED_0603_1608Metric, symbol taobao-led:LED_GREEN,0603
- added J?: SWD_SWD, footprint-lib:BLUEPILL_SWD, symbol taobao-components:BLUEPILL_SWD
- added JP? (x2): SolderJumper_2_Open_round, Jumper:SolderJumper-2_P1.3mm_Open_RoundedPad1.0x1.5mm, symbol my_solder_jumper:SolderJumper_2_Open_round
- added R? (x2): R221,0603, Resistor_SMD:R_0603_1608Metric_Pad1.05x0.95mm_HandSolder, symbol taobao-r:R221,0603
- added RN?: RN_221,0603, Resistor_SMD:R_Array_Concave_4x0603, symbol taobao-rpack:RN_221,0603
- J?: value SWD_HEADER -> SWD_SWD
Connections:
- net GND: now also D?.1 (K), J?.1 (Pin_1)
- net LED_STLINK: now also RN?.1 (R1.1), RN?.2 (R2.1)
- net T_JTCK: now also R?.2
- net T_JTMS: now also R?.2
- net Vstm32_stlink: now also D?.2 (A), JP?.1 (A), JP?.1 (A); no longer J?.4 (Pin_4)
- new net: J?.4 (Pin_4), JP?.2 (B) (x2)
- new net: D?.2 (A), RN?.7 (R2.2)
- new net: D?.1 (K), RN?.8 (R1.2)
- new net: J?.2 (Pin_2), R?.1
- new net: J?.3 (Pin_3), R?.1
Other:
- moved on the sheet: C?, J?, R?, RN?, TP?, U?, VUSB1_HEALTHY, VUSB1_HEALTHY?

Commit message: update,
Parts:
- removed R?: R221,0603, Resistor_SMD:R_0603_1608Metric_Pad1.05x0.95mm_HandSolder, symbol taobao-r:R221,0603
- removed RN?: RN_4R7,0603, Resistor_SMD:R_Array_Concave_4x0603, symbol taobao-rpack:RN_4R7,0603
- removed VUSB1_HEALTHY: LED_GREEN,0603, footprint-lib:LED_0603_1608Metric, symbol taobao-led:LED_GREEN,0603
- added R?: R152,0603, Resistor_SMD:R_0603_1608Metric_Pad1.05x0.95mm_HandSolder, symbol taobao-r:R152,0603
- added RN?: RN_472,0603, Resistor_SMD:R_Array_Concave_4x0603, symbol taobao-rpack:RN_472,0603
- JP?: value SolderJumper_2_Open_round -> SWD_SWD_EN
- JP?: value SolderJumper_2_Open_round -> SWD_3V3_EN
- R? (x2): value R221,0603 -> R220,0603
Connections:
- net USB_DM is gone; now on net USB_N: U?.32 (PA11-USART1CTS/TIM1CH4/USBDM)
- net USB_DP is gone; now on net USB_P: U?.33 (PA12-USART1RTS/USBDP)
- net GND: now also RN?.2 (R2.1)
- net Vstm32_stlink: now also R?.1, RN?.1 (R1.1)
- net at U?.10 (PA0-ADC0/WKUP/USART2CTS/TIM2CH1ETR): now also RN?.7 (R2.2), RN?.8 (R1.2)
- net at RN?.2 (R2.1), U?.6 (I/O1): now also R?.2
Other:
- note added: "for programming the child stm32"
- note added: "for programming the st-link itself"
- moved on the sheet: C?, D?, J?, JP?, R?, RN?, TP?, U?, VUSB1_HEALTHY?, Y?

Commit message: update,
Parts:
- gave numbers to parts that had none: 34

Commit message: update,
Connections:
- net SWCLK is gone; now on net D_SWCLK: J6.2 (Pin_2), U7.37 (PA14-JTCK/SWCLK)
- net SWDIO is gone; now on net D_SWDIO: J6.3 (Pin_3), U7.34 (PA13-JTMS/SWDIO)
- net D_SWCLK: now reaches J7.2 (Pin_2), R34.1
- net D_SWDIO: now reaches J7.3 (Pin_3), R35.1
Other:
- moved on the sheet: J7
Changed lines of the file:
@@
 $Descr A3 16535 11693
 encoding utf-8
-Sheet 13 13
+Sheet 10 13
 Title ""
 Date ""
@@
 Wire Wire Line
 	12800 4800 12800 4900
-$Comp
-L taobao-components:BLUEPILL_SWD J7
-U 1 1 5D156281
-P 13200 5000
-F 0 "J7" H 13580 4992 50  0000 L CNN
-F 1 "SWD_SWD" H 13580 4901 50  0000 L CNN
-F 2 "footprint-lib:BLUEPILL_SWD" H 13250 4600 50  0001 C CNN
-F 3 "" H 13200 5000 50  0001 C CNN
-	1    13200 5000
-	1    0    0    -1
-$EndComp
 Text Label 12000 5100 0    50   ~ 0
 T_JTMS
@@
 Wire Wire Line
 	12000 5100 12450 5100
-Wire Wire Line
-	12650 5000 13000 5000
-Wire Wire Line
-	12650 5100 13000 5100
-Wire Wire Line
-	12800 4900 13000 4900
 $Comp
 L my_power:Vstm32_stlink #PWR0129
@@
 	11900 3450 12950 3450
 Wire Wire Line
-	11800 5200 13000 5200
-Wire Wire Line
 	11800 5100 11800 5200
 Wire Wire Line
@@
 	1    0    0    -1
 $EndComp
+Wire Wire Line
+	11800 5200 13650 5200
+Wire Wire Line
+	12650 5100 13650 5100
+Wire Wire Line
+	12650 5000 13650 5000
+Wire Wire Line
+	12800 4900 13650 4900
+$Comp
+L taobao-components:BLUEPILL_SWD J7
+U 1 1 5D156281
+P 13850 5000
+F 0 "J7" H 14230 4992 50  0000 L CNN
+F 1 "SWD_SWD" H 14230 4901 50  0000 L CNN
+F 2 "footprint-lib:BLUEPILL_SWD" H 13900 4600 50  0001 C CNN
+F 3 "" H 13850 5000 50  0001 C CNN
+	1    13850 5000
+	1    0    0    -1
+$EndComp
+Text Label 13450 5100 2    50   ~ 0
+D_SWDIO
+Text Label 13450 5000 2    50   ~ 0
+D_SWCLK
+Text Label 1600 800  2    50   ~ 0
+SWCLK
+Text Label 1600 900  2    50   ~ 0
+SWDIO
+Text HLabel 1150 800  0    50   Input ~ 0
+D_SWCLK
+Text HLabel 1150 900  0    50   Input ~ 0
+D_SWDIO
+Wire Wire Line
+	1150 800  1600 800
+Wire Wire Line
+	1150 900  1600 900
 $EndSCHEMATC
