File: hardware/stm32_swd.sch (KiCad schematic (older format))
At the start: 34 parts, among them J6 SWD_SWD, J7 SWD_SWD, U10 USBLC6-2SC6_SOT23-6, U7 STM32F103C8T6_rect, U8 USB_Micro, U9 AMS1117-3.3, Y3 O_8M

Commit message: update,
Parts:
- added R40: R104,0603, Resistor_SMD:R_0603_1608Metric_Pad1.05x0.95mm_HandSolder, symbol taobao-r:R104,0603
Connections:
- net GND: now also R40.2
- net at U8.4 (ID): now also R40.1
- no-connect marks 0 -> 36
Changed lines of the file:
@@
 Wire Wire Line
 	1150 900  1600 900
+NoConn ~ 6500 8750
+NoConn ~ 6500 8850
+NoConn ~ 6900 8750
+NoConn ~ 6900 8850
+NoConn ~ 8000 5400
+NoConn ~ 8000 5600
+NoConn ~ 8000 5700
+NoConn ~ 4100 3400
+NoConn ~ 4100 3500
+NoConn ~ 1200 4550
+NoConn ~ 1200 4650
+NoConn ~ 1600 4650
+NoConn ~ 1600 4550
+NoConn ~ 4100 4900
+NoConn ~ 4100 5000
+NoConn ~ 4100 5100
+NoConn ~ 4100 5200
+NoConn ~ 4100 5300
+NoConn ~ 4100 5400
+NoConn ~ 4100 5500
+NoConn ~ 4100 5700
+NoConn ~ 4100 5800
+NoConn ~ 4100 4200
+NoConn ~ 4100 4300
+$Comp
+L taobao-r:R104,0603 R40
+U 1 1 5D70A604
+P 4650 8300
+F 0 "R40" H 4709 8346 50  0000 L CNN
+F 1 "R104,0603" H 4709 8255 50  0000 L CNN
+F 2 "Resistor_SMD:R_0603_1608Metric_Pad1.05x0.95mm_HandSolder" H 4650 8300 50  0001 C CNN
+F 3 "~" H 4650 8300 50  0001 C CNN
+	1    4650 8300
+	1    0    0    -1
+$EndComp
+$Comp
+L power:GND #PWR?
+U 1 1 5D70A8BF
+P 4650 8500
+AR Path="/5D0A467E/5D70A8BF" Ref="#PWR?"  Part="1"
+AR Path="/5CF48B33/5D70A8BF" Ref="#PWR011"  Part="1"
+F 0 "#PWR011" H 4650 8250 50  0001 C CNN
+F 1 "GND" H 4655 8327 50  0000 C CNN
+F 2 "" H 4650 8500 50  0001 C CNN
+F 3 "" H 4650 8500 50  0001 C CNN
+	1    4650 8500
+	-1   0    0    -1
+$EndComp
+Wire Wire Line
+	4650 8500 4650 8400
+Wire Wire Line
+	4350 8100 4650 8100
+Wire Wire Line
+	4650 8100 4650 8200
+NoConn ~ 8000 3400
+NoConn ~ 8000 3500
+NoConn ~ 8000 3700
+NoConn ~ 8000 3800
+NoConn ~ 8000 3900
+NoConn ~ 8000 4000
+NoConn ~ 8000 4100
+NoConn ~ 8000 4200
+NoConn ~ 13950 8400
+NoConn ~ 13950 8500
+NoConn ~ 14350 8400
+NoConn ~ 14350 8500
 $EndSCHEMATC

Commit message: update,
Parts:
- renumbered C46 to C29, C47 to C30, C48 to C31, C49 to C32, C50 to C33, C51 to C34, C52 to C35, C53 to C36, C54 to C37, C55 to C38, D38 to D25, D39 to D26, J6 to J5, J7 to J6, JP8 to JP?, JP7 to JP?, R31 to R19, R32 to R20, R33 to R21, R34 to R22, R35 to R23, R36 to R24, R37 to R25, R40 to R26, R38 to R27, RN4 to RN?, RN3 to RN?, RN2 to RN?, TP4 to TP?, U7 to U6, U8 to U7, U9 to U8, U10 to U9, Y3 to Y1

Commit message: update footprint,
Parts:
- gave numbers to parts that had none: 6
Changed lines of the file:
@@
 $EndComp
 $Comp
-L my_testpoint:TestPoint_2mm TP?
+L my_testpoint:TestPoint_2mm TP8
 U 1 1 5CF8BD26
 P 4600 7200
-F 0 "TP?" V 4554 7388 50  0000 L CNN
+F 0 "TP8" V 4554 7388 50  0000 L CNN
 F 1 "TP_VUSB1" V 4645 7388 50  0000 L CNN
 F 2 "TestPoint:TestPoint_THTPad_D2.0mm_Drill1.0mm" H 4800 7200 50  0001 C CNN
@@
 	4450 7800 6350 7800
 $Comp
-L taobao-rpack:RN_221,0603 RN?
+L taobao-rpack:RN_221,0603 RN4
 U 1 1 5CF99338
 P 6700 8750
-F 0 "RN?" V 6283 8750 50  0000 C CNN
+F 0 "RN4" V 6283 8750 50  0000 C CNN
 F 1 "RN_221,0603" V 6374 8750 50  0000 C CNN
 F 2 "Resistor_SMD:R_Array_Concave_4x0603" V 6975 8750 50  0001 C CNN
@@
 $EndComp
 $Comp
-L taobao-rpack:RN_221,0603 RN?
+L taobao-rpack:RN_221,0603 RN3
 U 1 1 5D0FD752
 P 14150 8400
-F 0 "RN?" V 13733 8400 50  0000 C CNN
+F 0 "RN3" V 13733 8400 50  0000 C CNN
 F 1 "RN_221,0603" V 13824 8400 50  0000 C CNN
 F 2 "Resistor_SMD:R_Array_Concave_4x0603" V 14425 8400 50  0001 C CNN
@@
 T_JTCK
 $Comp
-L my_solder_jumper:SolderJumper_2_Open_round JP?
+L my_solder_jumper:SolderJumper_2_Open_round JP6
 U 1 1 5D166FFC
 P 11800 4950
-F 0 "JP?" V 11754 4863 50  0000 R CNN
+F 0 "JP6" V 11754 4863 50  0000 R CNN
 F 1 "SWD_SWD_EN" V 11845 4863 50  0000 R CNN
 F 2 "Jumper:SolderJumper-2_P1.3mm_Open_RoundedPad1.0x1.5mm" H 11800 4950 50  0001 C CNN
@@
 $EndComp
 $Comp
-L my_solder_jumper:SolderJumper_2_Open_round JP?
+L my_solder_jumper:SolderJumper_2_Open_round JP5
 U 1 1 5D196ACA
 P 11900 3250
-F 0 "JP?" V 11854 3163 50  0000 R CNN
+F 0 "JP5" V 11854 3163 50  0000 R CNN
 F 1 "SWD_3V3_EN" V 11945 3163 50  0000 R CNN
 F 2 "Jumper:SolderJumper-2_P1.3mm_Open_RoundedPad1.0x1.5mm" H 11900 3250 50  0001 C CNN
@@
 	3450 3300 4100 3300
 $Comp
-L taobao-rpack:RN_472,0603 RN?
+L taobao-rpack:RN_472,0603 RN2
 U 1 1 5D1C71FE
 P 1400 4550
-F 0 "RN?" V 983 4550 50  0000 C CNN
+F 0 "RN2" V 983 4550 50  0000 C CNN
 F 1 "RN_472,0603" V 1074 4550 50  0000 C CNN
 F 2 "Resistor_SMD:R_Array_Concave_4x0603" V 1675 4550 50  0001 C CNN

Commit message: update footprint,
Parts:
- U7: value USB_Micro -> SWD
- U9: footprint footprints-lib:USBLC6-2 -> footprint-lib:USBLC6-2SC6_SOT23-6
Changed lines of the file:
@@
 AR Path="/5CF48B33/5CF71140" Ref="U7"  Part="1"
 F 0 "U7" H 3950 8465 50  0000 C CNN
-F 1 "USB_Micro" H 3950 8374 50  0000 C CNN
+F 1 "SWD" H 3950 8374 50  0000 C CNN
 F 2 "footprint-lib:USB_Micro-B_Molex-105017-0001" H 3950 7500 50  0001 C CNN
 F 3 "" H 3950 7500 50  0001 C CNN
@@
 F 0 "U9" H 5750 8285 50  0000 C CNN
 F 1 "USBLC6-2SC6_SOT23-6" H 5750 8376 50  0000 C CNN
-F 2 "footprints-lib:USBLC6-2" H 5750 8150 50  0001 C CNN
+F 2 "footprint-lib:USBLC6-2SC6_SOT23-6" H 5750 8150 50  0001 C CNN
 F 3 "" H 5750 8600 50  0001 C CNN
 	1    5750 8650

Commit message: update footprint,
Parts:
- U8: footprint Package_TO_SOT_SMD:SOT-223-3_TabPin2 -> footprint-lib:AMS1117_SOT-223
Changed lines of the file:
@@
 EESchema Schematic File Version 4
-LIBS:stm32_aux_keyboard-cache
 EELAYER 29 0
 EELAYER END
 $Descr A3 16535 11693
 encoding utf-8
-Sheet 10 13
+Sheet 1 1
 Title ""
 Date ""
@@
 AR Path="/5D0A467E/5CF71140" Ref="U?"  Part="1"
 AR Path="/5CF48B33/5CF71140" Ref="U7"  Part="1"
+AR Path="/5CF71140" Ref="U7"  Part="1"
 F 0 "U7" H 3950 8465 50  0000 C CNN
 F 1 "SWD" H 3950 8374 50  0000 C CNN
@@
 AR Path="/5D0A467E/5CF71146" Ref="#PWR?"  Part="1"
 AR Path="/5CF48B33/5CF71146" Ref="#PWR0139"  Part="1"
+AR Path="/5CF71146" Ref="#PWR0139"  Part="1"
 F 0 "#PWR0139" H 3350 8250 50  0001 C CNN
 F 1 "GND" H 3355 8327 50  0000 C CNN
@@
 AR Path="/5D0A467E/5CF71157" Ref="#PWR?"  Part="1"
 AR Path="/5CF48B33/5CF71157" Ref="#PWR0140"  Part="1"
+AR Path="/5CF71157" Ref="#PWR0140"  Part="1"
 F 0 "#PWR0140" H 4450 8250 50  0001 C CNN
 F 1 "GND" H 4455 8327 50  0000 C CNN
@@
 AR Path="/5CF34646/5CF5CD4C" Ref="C?"  Part="1"
 AR Path="/5CF48B33/5CF5CD4C" Ref="C37"  Part="1"
+AR Path="/5CF5CD4C" Ref="C37"  Part="1"
 F 0 "C37" H 11288 8296 50  0000 L CNN
 F 1 "CP100uf,16V" H 11288 8205 50  0000 L CNN
@@
 AR Path="/5CF34646/5CF5CD46" Ref="C?"  Part="1"
 AR Path="/5CF48B33/5CF5CD46" Ref="C36"  Part="1"
+AR Path="/5CF5CD46" Ref="C36"  Part="1"
 F 0 "C36" H 10163 8296 50  0000 R CNN
 F 1 "CP100uf,16V" H 10163 8205 50  0000 R CNN
@@
 AR Path="/5CF34646/5CF5CD2B" Ref="#PWR?"  Part="1"
 AR Path="/5CF48B33/5CF5CD2B" Ref="#PWR0144"  Part="1"
+AR Path="/5CF5CD2B" Ref="#PWR0144"  Part="1"
 F 0 "#PWR0144" H 11400 8300 50  0001 C CNN
 F 1 "GND" H 11405 8377 50  0000 C CNN
@@
 AR Path="/5CF34646/5CF5CD1F" Ref="#PWR?"  Part="1"
 AR Path="/5CF48B33/5CF5CD1F" Ref="#PWR0143"  Part="1"
+AR Path="/5CF5CD1F" Ref="#PWR0143"  Part="1"
 F 0 "#PWR0143" H 10750 8300 50  0001 C CNN
 F 1 "GND" H 10755 8377 50  0000 C CNN
@@
 AR Path="/5CF34646/5CF5CD18" Ref="#PWR?"  Part="1"
 AR Path="/5CF48B33/5CF5CD18" Ref="#PWR0142"  Part="1"
+AR Path="/5CF5CD18" Ref="#PWR0142"  Part="1"
 F 0 "#PWR0142" H 10250 8300 50  0001 C CNN
 F 1 "GND" H 10255 8377 50  0000 C CNN
@@
 AR Path="/5CF34646/5CF5CD0D" Ref="C?"  Part="1"
 AR Path="/5CF48B33/5CF5CD0D" Ref="C38"  Part="1"
+AR Path="/5CF5CD0D" Ref="C38"  Part="1"
 F 0 "C38" H 11692 8296 50  0000 L CNN
 F 1 "C105" H 11692 8205 50  0000 L CNN
@@
 AR Path="/5CF34646/5CF5CD07" Ref="U?"  Part="1"
 AR Path="/5CF48B33/5CF5CD07" Ref="U8"  Part="1"
+AR Path="/5CF5CD07" Ref="U8"  Part="1"
 F 0 "U8" H 10750 8242 50  0000 C CNN
 F 1 "AMS1117-3.3" H 10750 8151 50  0000 C CNN
-F 2 "Package_TO_SOT_SMD:SOT-223-3_TabPin2" H 10750 8200 50  0001 C CNN
+F 2 "footprint-lib:AMS1117_SOT-223" H 10750 8200 50  0001 C CNN
 F 3 "http://www.advanced-monolithic.com/pdf/ds1117.pdf" H 10850 7750 50  0001 C CNN
 	1    10750 8000
@@
 AR Path="/5D0A467E/5D70A8BF" Ref="#PWR?"  Part="1"
 AR Path="/5CF48B33/5D70A8BF" Ref="#PWR0141"  Part="1"
+AR Path="/5D70A8BF" Ref="#PWR0141"  Part="1"
 F 0 "#PWR0141" H 4650 8250 50  0001 C CNN
 F 1 "GND" H 4655 8327 50  0000 C CNN

Commit message: update,
Connections:
- net USB_N: now also RN4.7 (R2.2); no longer RN4.8 (R1.2)
- net USB_P: now also RN4.8 (R1.2); no longer RN4.7 (R2.2)
- net at U9.4 (I/O2): now also RN4.2 (R2.1); no longer RN4.1 (R1.1)
- net at R27.2, U9.6 (I/O1): now also RN4.1 (R1.1); no longer RN4.2 (R2.1)
Other:
- moved on the sheet: RN4
Changed lines of the file:
@@
 $Descr A3 16535 11693
 encoding utf-8
-Sheet 1 13
+Sheet 10 13
 Title ""
 Date ""
@@
 L taobao-rpack:RN_221,0603 RN4
 U 1 1 5CF99338
-P 6700 8750
-F 0 "RN4" V 6283 8750 50  0000 C CNN
-F 1 "RN_221,0603" V 6374 8750 50  0000 C CNN
-F 2 "Resistor_SMD:R_Array_Concave_4x0603" V 6975 8750 50  0001 C CNN
-F 3 "~" H 6700 8750 50  0001 C CNN
-	1    6700 8750
-	0    1    1    0
+P 6700 8450
+F 0 "RN4" V 6283 8450 50  0000 C CNN
+F 1 "RN_221,0603" V 6374 8450 50  0000 C CNN
+F 2 "Resistor_SMD:R_Array_Concave_4x0603" V 6975 8450 50  0001 C CNN
+F 3 "~" H 6700 8450 50  0001 C CNN
+	1    6700 8450
+	0    1    -1   0
 $EndComp
 Wire Wire Line
@@
 Wire Wire Line
 	1150 900  1600 900
-NoConn ~ 6500 8750
-NoConn ~ 6500 8850
-NoConn ~ 6900 8750
-NoConn ~ 6900 8850
+NoConn ~ 6500 8450
+NoConn ~ 6500 8350
+NoConn ~ 6900 8450
+NoConn ~ 6900 8350
 NoConn ~ 8000 5400
 NoConn ~ 8000 5600
