File: hardware/usb.sch (KiCad schematic (older format))
At the start: 3 parts, among them U5 USB_Micro, U6 USBLC6-2SC6_SOT23-6

Commit message: update,
Parts:
- added R39: R104,0603, Resistor_SMD:R_0603_1608Metric_Pad1.05x0.95mm_HandSolder, symbol taobao-r:R104,0603
Connections:
- net GND: now also R39.2
- net at U5.4 (ID): now also R39.1
- no-connect marks 0 -> 4
Changed lines of the file:
@@
 	-1   0    0    -1
 $EndComp
+NoConn ~ 3600 2400
+NoConn ~ 3600 2500
+NoConn ~ 4000 2500
+NoConn ~ 4000 2400
+$Comp
+L taobao-r:R104,0603 R39
+U 1 1 5D660AA1
+P 1900 2000
+F 0 "R39" H 1959 2046 50  0000 L CNN
+F 1 "R104,0603" H 1959 1955 50  0000 L CNN
+F 2 "Resistor_SMD:R_0603_1608Metric_Pad1.05x0.95mm_HandSolder" H 1900 2000 50  0001 C CNN
+F 3 "~" H 1900 2000 50  0001 C CNN
+	1    1900 2000
+	1    0    0    -1
+$EndComp
+$Comp
+L power:GND #PWR010
+U 1 1 5D66101C
+P 1900 2200
+F 0 "#PWR010" H 1900 1950 50  0001 C CNN
+F 1 "GND" H 1905 2027 50  0000 C CNN
+F 2 "" H 1900 2200 50  0001 C CNN
+F 3 "" H 1900 2200 50  0001 C CNN
+	1    1900 2200
+	-1   0    0    -1
+$EndComp
+Wire Wire Line
+	1900 2200 1900 2100
+Wire Wire Line
+	1700 1800 1900 1800
+Wire Wire Line
+	1900 1800 1900 1900
 $EndSCHEMATC

Commit message: update,
Parts:
- renumbered R39 to R14, RN1 to RN?, U5 to U4, U6 to U5
Changed lines of the file:
@@
 	2300 2300 2300 1900
 $Comp
-L power:GND #PWR0118
+L power:GND #PWR0103
 U 1 1 5D3240FA
 P 2300 2300
-F 0 "#PWR0118" H 2300 2050 50  0001 C CNN
+F 0 "#PWR0103" H 2300 2050 50  0001 C CNN
 F 1 "GND" H 2305 2127 50  0000 C CNN
 F 2 "" H 2300 2300 50  0001 C CNN
@@
 	3250 1800 3450 1800
 $Comp
-L taobao-rpack:RN_220,0603 RN1
+L taobao-rpack:RN_220,0603 RN?
 U 1 1 5D31870E
 P 3800 2400
-F 0 "RN1" V 3383 2400 50  0000 C CNN
+F 0 "RN?" V 3383 2400 50  0000 C CNN
 F 1 "RN_220,0603" V 3474 2400 50  0000 C CNN
 F 2 "Resistor_SMD:R_Array_Concave_4x0603" V 4075 2400 50  0001 C CNN
@@
 	2350 2000 2050 2000
 $Comp
-L taobao-components:USBLC6-2SC6_SOT23-6 U6
+L taobao-components:USBLC6-2SC6_SOT23-6 U5
 U 1 1 5D3156EE
 P 2800 1900
-F 0 "U6" H 2800 2265 50  0000 C CNN
+F 0 "U5" H 2800 2265 50  0000 C CNN
 F 1 "USBLC6-2SC6_SOT23-6" H 2800 2174 50  0000 C CNN
 F 2 "footprints-lib:USBLC6-2" H 2800 1400 50  0001 C CNN
@@
 	1700 1600 2050 1600
 $Comp
-L my_power:Vusb #PWR0115
+L my_power:Vusb #PWR099
 U 1 1 5D0A9977
 P 1800 1150
-F 0 "#PWR0115" H 1800 1000 50  0001 C CNN
+F 0 "#PWR099" H 1800 1000 50  0001 C CNN
 F 1 "Vusb" H 1815 1323 50  0000 C CNN
 F 2 "" H 1800 1150 50  0001 C CNN
@@
 	1800 2200 1800 1900
 $Comp
-L power:GND #PWR0117
+L power:GND #PWR0101
 U 1 1 5D0A5204
 P 1800 2200
-F 0 "#PWR0117" H 1800 1950 50  0001 C CNN
+F 0 "#PWR0101" H 1800 1950 50  0001 C CNN
 F 1 "GND" H 1805 2027 50  0000 C CNN
 F 2 "" H 1800 2200 50  0001 C CNN
@@
 	900  1500 700  1500
 $Comp
-L power:GND #PWR0116
+L power:GND #PWR0100
 U 1 1 5D0A4EF1
 P 700 2200
-F 0 "#PWR0116" H 700 1950 50  0001 C CNN
+F 0 "#PWR0100" H 700 1950 50  0001 C CNN
 F 1 "GND" H 705 2027 50  0000 C CNN
 F 2 "" H 700 2200 50  0001 C CNN
@@
 $EndComp
 $Comp
-L taobao-components:USB_Micro U5
+L taobao-components:USB_Micro U4
 U 1 1 5D0A4A6D
 P 1300 1700
-F 0 "U5" H 1300 2165 50  0000 C CNN
+F 0 "U4" H 1300 2165 50  0000 C CNN
 F 1 "USB_Micro" H 1300 2074 50  0000 C CNN
 F 2 "footprint-lib:USB_Micro-B_Molex-105017-0001" H 1300 1200 50  0001 C CNN
@@
 NoConn ~ 4000 2400
 $Comp
-L taobao-r:R104,0603 R39
+L taobao-r:R104,0603 R14
 U 1 1 5D660AA1
 P 1900 2000
-F 0 "R39" H 1959 2046 50  0000 L CNN
+F 0 "R14" H 1959 2046 50  0000 L CNN
 F 1 "R104,0603" H 1959 1955 50  0000 L CNN
 F 2 "Resistor_SMD:R_0603_1608Metric_Pad1.05x0.95mm_HandSolder" H 1900 2000 50  0001 C CNN
@@
 $EndComp
 $Comp
-L power:GND #PWR010
+L power:GND #PWR0102
 U 1 1 5D66101C
 P 1900 2200
-F 0 "#PWR010" H 1900 1950 50  0001 C CNN
+F 0 "#PWR0102" H 1900 1950 50  0001 C CNN
 F 1 "GND" H 1905 2027 50  0000 C CNN
 F 2 "" H 1900 2200 50  0001 C CNN

Commit message: update footprint,
Parts:
- gave numbers to parts that had none: 1
Changed lines of the file:
@@
 	3250 1800 3450 1800
 $Comp
-L taobao-rpack:RN_220,0603 RN?
+L taobao-rpack:RN_220,0603 RN1
 U 1 1 5D31870E
 P 3800 2400
-F 0 "RN?" V 3383 2400 50  0000 C CNN
+F 0 "RN1" V 3383 2400 50  0000 C CNN
 F 1 "RN_220,0603" V 3474 2400 50  0000 C CNN
 F 2 "Resistor_SMD:R_Array_Concave_4x0603" V 4075 2400 50  0001 C CNN

Commit message: update footprint,
Parts:
- U4: value USB_Micro -> USB
- U5: footprint footprints-lib:USBLC6-2 -> footprint-lib:USBLC6-2SC6_SOT23-6
Changed lines of the file:
@@
 F 0 "U5" H 2800 2265 50  0000 C CNN
 F 1 "USBLC6-2SC6_SOT23-6" H 2800 2174 50  0000 C CNN
-F 2 "footprints-lib:USBLC6-2" H 2800 1400 50  0001 C CNN
+F 2 "footprint-lib:USBLC6-2SC6_SOT23-6" H 2800 1400 50  0001 C CNN
 F 3 "" H 2800 1850 50  0001 C CNN
 	1    2800 1900
@@
 P 1300 1700
 F 0 "U4" H 1300 2165 50  0000 C CNN
-F 1 "USB_Micro" H 1300 2074 50  0000 C CNN
+F 1 "USB" H 1300 2074 50  0000 C CNN
 F 2 "footprint-lib:USB_Micro-B_Molex-105017-0001" H 1300 1200 50  0001 C CNN
 F 3 "" H 1300 1200 50  0001 C CNN
