File: hardware/WS2812.sch (KiCad schematic (older format))
At the start: 12 parts

Commit message: update for cherry key,
Parts:
- added C? (x13): C106,0805, Capacitor_SMD:C_0805_2012Metric_Pad1.15x1.40mm_HandSolder, symbol taobao-c:C106,0805
- added D? (x13): WS2812B, LED_SMD:LED_WS2812B_PLCC4_5.0x5.0mm_P3.2mm, symbol LED:WS2812B
Connections:
- net +5V: now also C?.2, C?.2, C?.2, C?.2, C?.2, C?.2, C?.2, C?.2, C?.2, C?.2, C?.2, C?.2, C?.2, D?.1 (VDD), D?.1 (VDD), D?.1 (VDD), D?.1 (VDD), D?.1 (VDD), D?.1 (VDD), D?.1 (VDD), D?.1 (VDD), D?.1 (VDD), D?.1 (VDD), D?.1 (VDD), D?.1 (VDD), D?.1 (VDD)
- net GND: now also C?.1, C?.1, C?.1, C?.1, C?.1, C?.1, C?.1, C?.1, C?.1, C?.1, C?.1, C?.1, C?.1, D?.3 (VSS), D?.3 (VSS), D?.3 (VSS), D?.3 (VSS), D?.3 (VSS), D?.3 (VSS), D?.3 (VSS), D?.3 (VSS), D?.3 (VSS), D?.3 (VSS), D?.3 (VSS), D?.3 (VSS), D?.3 (VSS)
- net at D?.2 (DOUT): now also D?.4 (DIN)
- new net: D?.2 (DOUT), D?.4 (DIN) (x12)
Other:
- moved on the sheet: C?, D?, J?

Commit message: update for cherry key,
Parts:
- removed C? (x4): C106,0805, Capacitor_SMD:C_0805_2012Metric_Pad1.15x1.40mm_HandSolder, symbol taobao-c:C106,0805
- removed D? (x4): WS2812B, LED_SMD:LED_WS2812B_PLCC4_5.0x5.0mm_P3.2mm, symbol LED:WS2812B

Commit message: update for power symbol,
Parts:
- removed C? (x13): C106,0805, Capacitor_SMD:C_0805_2012Metric_Pad1.15x1.40mm_HandSolder, symbol taobao-c:C106,0805
- removed D? (x13): WS2812B, LED_SMD:LED_WS2812B_PLCC4_5.0x5.0mm_P3.2mm, symbol LED:WS2812B
- added C? (x17): C106,0805, Capacitor_SMD:C_0805_2012Metric_Pad1.15x1.40mm_HandSolder, symbol taobao-c:C106,0805
- added D? (x17): WS2812B, LED_SMD:LED_WS2812B_PLCC4_5.0x5.0mm_P3.2mm, symbol LED:WS2812B
Connections:
- net GND: now also C?.1, C?.1, C?.1, C?.1, C?.1, C?.1, C?.1, C?.1, C?.1, C?.1, C?.1, C?.1, C?.1, C?.1, C?.1, C?.1, C?.1, D?.3 (VSS), D?.3 (VSS), D?.3 (VSS), D?.3 (VSS), D?.3 (VSS), D?.3 (VSS), D?.3 (VSS), D?.3 (VSS), D?.3 (VSS), D?.3 (VSS), D?.3 (VSS), D?.3 (VSS), D?.3 (VSS), D?.3 (VSS), D?.3 (VSS), D?.3 (VSS), D?.3 (VSS)
- net at D?.2 (DOUT): now also D?.4 (DIN)
- net +5V renamed VCC
- net VCC: now also C?.2, C?.2, C?.2, C?.2, C?.2, C?.2, C?.2, C?.2, C?.2, C?.2, C?.2, C?.2, C?.2, C?.2, C?.2, C?.2, C?.2, D?.1 (VDD), D?.1 (VDD), D?.1 (VDD), D?.1 (VDD), D?.1 (VDD), D?.1 (VDD), D?.1 (VDD), D?.1 (VDD), D?.1 (VDD), D?.1 (VDD), D?.1 (VDD), D?.1 (VDD), D?.1 (VDD), D?.1 (VDD), D?.1 (VDD), D?.1 (VDD), D?.1 (VDD)
- new net: D?.2 (DOUT), D?.4 (DIN) (x16)
- no-connect marks 1 -> 0

Commit message: update,
Parts:
- gave numbers to parts that had none: 38

Commit message: update,
Connections:
- no-connect marks 0 -> 1
Changed lines of the file:
@@
 $Descr A4 11693 8268
 encoding utf-8
-Sheet 6 13
+Sheet 5 13
 Title ""
 Date ""
@@
 Wire Wire Line
 	8000 3550 7800 3550
+NoConn ~ 7800 5050
 $EndSCHEMATC
