File: hardware/stm32_aux_keyboard.sch (KiCad schematic (older format))
At the start: 0 parts

Commit message: update for cherry key,
Changed lines of the file:
@@
 $Descr User 8500 5500
 encoding utf-8
-Sheet 1 11
+Sheet 1 12
 Title ""
 Date ""
@@
 $EndSheet
 $Sheet
-S 1900 750  950  600
+S 1950 750  950  600
 U 5CF34713
 F0 "keyboard_key" 50
@@
 $EndSheet
 $Sheet
-S 1900 1650 950  600
+S 1950 2400 950  600
 U 5CF34744
 F0 "rot_enc" 50
@@
 $EndSheet
 $Sheet
-S 1900 2550 950  600
+S 1950 3350 950  600
 U 5CF34798
 F0 "status_display" 50
@@
 $EndSheet
 $Sheet
-S 3600 3350 950  600
+S 3650 4150 950  600
 U 5CF369D9
 F0 "push_buttton" 50
@@
 $EndSheet
 $Sheet
-S 1900 3350 950  600
+S 1950 4150 950  600
 U 5D0AD7CC
 F0 "buzzer" 50
 F1 "buzzer.sch" 50
 $EndSheet
+$Sheet
+S 1950 1550 950  600
+U 5CFF7883
+F0 "rot_enc2" 50
+F1 "rot_enc2.sch" 50
+$EndSheet
 $EndSCHEMATC

Commit message: update,
Changed lines of the file:
@@
 $Descr User 8500 5500
 encoding utf-8
-Sheet 1 12
+Sheet 1 13
 Title ""
 Date ""
@@
 F1 "rot_enc2.sch" 50
 $EndSheet
+$Sheet
+S 3550 100  650  300
+U 5CF48B33
+F0 "stm32_swd" 50
+F1 "stm32_swd.sch" 50
+$EndSheet
 $EndSCHEMATC

Commit message: update,
Changed lines of the file:
@@
 EELAYER 29 0
 EELAYER END
-$Descr User 8500 5500
+$Descr A4 11693 8268
 encoding utf-8
 Sheet 1 13
@@
 $EndDescr
 $Sheet
-S 3550 750  950  600
+S 8300 1800 950  600
+U 5CF34615
+F0 "oled" 50
+F1 "oled.sch" 50
+F2 "SDA" I L 8300 2050 50
+F3 "SCL" I L 8300 2150 50
+$EndSheet
+$Sheet
+S 750  6900 950  600
+U 5CF34646
+F0 "power" 50
+F1 "power.sch" 50
+$EndSheet
+$Sheet
+S 3600 3750 950  600
+U 5CF34798
+F0 "status_display" 50
+F1 "status_display.sch" 50
+F2 "USR_LED_1" I R 4550 3950 50
+F3 "USR_LED_2" I R 4550 4050 50
+F4 "USR_LED_3" I R 4550 4150 50
+$EndSheet
+$Sheet
+S 8300 2750 950  600
+U 5CF35582
+F0 "WS2812" 50
+F1 "WS2812.sch" 50
+F2 "WS2812_IN" I L 8300 3050 50
+$EndSheet
+$Sheet
+S 3600 5350 950  600
+U 5CF369D9
+F0 "push_buttton" 50
+F1 "push_buttton.sch" 50
+F2 "USR_BTN_1" I R 4550 5500 50
+F3 "USR_BTN_2" I R 4550 5600 50
+F4 "USR_BTN_3" I R 4550 5700 50
+F5 "USR_BTN_4" I R 4550 5800 50
+$EndSheet
+$Sheet
+S 8300 3800 750  400
+U 5D0A467E
+F0 "usb" 50
+F1 "usb.sch" 50
+F2 "USB_P" I L 8300 3900 50
+F3 "USB_N" I L 8300 4000 50
+$EndSheet
+$Sheet
+S 3600 4550 950  600
+U 5D0AD7CC
+F0 "buzzer" 50
+F1 "buzzer.sch" 50
+F2 "BUZZER_IN" I R 4550 4850 50
+$EndSheet
+$Sheet
+S 3600 1950 950  600
+U 5CFF7883
+F0 "rot_enc2" 50
+F1 "rot_enc2.sch" 50
+F2 "SW_OUT" I R 4550 2150 50
+F3 "B" I R 4550 2250 50
+F4 "A" I R 4550 2350 50
+$EndSheet
+$Sheet
+S 8300 1250 650  300
+U 5CF48B33
+F0 "stm32_swd" 50
+F1 "stm32_swd.sch" 50
+F2 "D_SWCLK" I L 8300 1350 50
+F3 "D_SWDIO" I L 8300 1450 50
+$EndSheet
+$Sheet
+S 3600 850  950  950
+U 5CF34713
+F0 "keyboard_key" 50
+F1 "keyboard_key.sch" 50
+F2 "ROW1" I R 4550 950 50
+F3 "ROW2" I R 4550 1050 50
+F4 "ROW3" I R 4550 1150 50
+F5 "ROW4" I R 4550 1250 50
+F6 "COL1" I R 4550 1500 50
+F7 "COL2" I R 4550 1600 50
+F8 "COL3" I R 4550 1700 50
+$EndSheet
+$Sheet
+S 3600 2800 950  600
+U 5CF34744
+F0 "rot_enc" 50
+F1 "rot_enc.sch" 50
+F2 "SW_OUT" I R 4550 2950 50
+F3 "B" I R 4550 3050 50
+F4 "A" I R 4550 3150 50
+$EndSheet
+$Sheet
+S 5700 850  2100 5050
 U 5CF345FD
 F0 "stm32_core" 50
 F1 "stm32_core.sch" 50
-$EndSheet
-$Sheet
-S 5100 750  950  600
-U 5CF34615
-F0 "oled" 50
-F1 "oled.sch" 50
-$EndSheet
-$Sheet
-S 650  4200 950  600
-U 5CF34646
-F0 "power" 50
-F1 "power.sch" 50
-$EndSheet
-$Sheet
-S 1950 750  950  600
-U 5CF34713
-F0 "keyboard_key" 50
-F1 "keyboard_key.sch" 50
-$EndSheet
-$Sheet
-S 1950 2400 950  600
-U 5CF34744
-F0 "rot_enc" 50
-F1 "rot_enc.sch" 50
-$EndSheet
-$Sheet
-S 1950 3350 950  600
-U 5CF34798
-F0 "status_display" 50
-F1 "status_display.sch" 50
-$EndSheet
-$Sheet
-S 5100 1700 950  600
-U 5CF35582
-F0 "WS2812" 50
-F1 "WS2812.sch" 50
-$EndSheet
-$Sheet
-S 3650 4150 950  600
-U 5CF369D9
-F0 "push_buttton" 50
-F1 "push_buttton.sch" 50
-$EndSheet
-$Sheet
-S 5100 2750 750  400
-U 5D0A467E
-F0 "usb" 50
-F1 "usb.sch" 50
-$EndSheet
-$Sheet
-S 1950 4150 950  600
-U 5D0AD7CC
-F0 "buzzer" 50
-F1 "buzzer.sch" 50
-$EndSheet
-$Sheet
-S 1950 1550 950  600
-U 5CFF7883
-F0 "rot_enc2" 50
-F1 "rot_enc2.sch" 50
-$EndSheet
-$Sheet
-S 3550 100  650  300
-U 5CF48B33
-F0 "stm32_swd" 50
-F1 "stm32_swd.sch" 50
-$EndSheet
+F2 "SDA" I R 7800 2050 50
+F3 "SCL" I R 7800 2150 50
+F4 "ROW1" I L 5700 950 50
+F5 "ROW2" I L 5700 1050 50
+F6 "ROW3" I L 5700 1150 50
+F7 "ROW4" I L 5700 1250 50
+F8 "COL1" I L 5700 1500 50
+F9 "COL2" I L 5700 1600 50
+F10 "COL3" I L 5700 1700 50
+F11 "ROT_ENC_A1" I L 5700 2350 50
+F12 "ROT_ENC_A2" I L 5700 3150 50
+F13 "ROT_ENC_B1" I L 5700 2250 50
+F14 "ROT_ENC_B2" I L 5700 3050 50
+F15 "ROT_ENC_SW1" I L 5700 2150 50
+F16 "ROT_ENC_SW2" I L 5700 2950 50
+F17 "WS2812_OUT" I R 7800 3050 50
+F18 "TTL_TX" I R 7800 5050 50
+F19 "TTL_RX" I R 7800 5150 50
+F20 "USR_BTN1" I L 5700 5500 50
+F21 "USR_BTN2" I L 5700 5600 50
+F22 "USR_BTN3" I L 5700 5700 50
+F23 "USR_BTN4" I L 5700 5800 50
+F24 "USR_STA1" I L 5700 3950 50
+F25 "USR_STA2" I L 5700 4050 50
+F26 "USR_STA3" I L 5700 4150 50
+F27 "BUZZER" I L 5700 4850 50
+F28 "SWCLK" I R 7800 1350 50
+F29 "SWDIO" I R 7800 1450 50
+F30 "USB_P" I R 7800 3900 50
+F31 "USB_N" I R 7800 4000 50
+$EndSheet
+Wire Wire Line
+	4550 950  5700 950
+Wire Wire Line
+	4550 1050 5700 1050
+Wire Wire Line
+	4550 1150 5700 1150
+Wire Wire Line
+	4550 1250 5700 1250
+Wire Wire Line
+	4550 1500 5700 1500
+Wire Wire Line
+	4550 1600 5700 1600
+Wire Wire Line
+	4550 1700 5700 1700
+Wire Wire Line
+	4550 2150 5700 2150
+Wire Wire Line
+	4550 2250 5700 2250
+Wire Wire Line
+	4550 2350 5700 2350
+Wire Wire Line
+	4550 2950 5700 2950
+Wire Wire Line
+	4550 3050 5700 3050
+Wire Wire Line
+	4550 3150 5700 3150
+Wire Wire Line
+	4550 3950 5700 3950
+Wire Wire Line
+	4550 4050 5700 4050
+Wire Wire Line
+	4550 4150 5700 4150
+Wire Wire Line
+	4550 4850 5700 4850
+Wire Wire Line
+	4550 5500 5700 5500
+Wire Wire Line
+	4550 5600 5700 5600
+Wire Wire Line
+	4550 5700 5700 5700
+Wire Wire Line
+	4550 5800 5700 5800
+Wire Wire Line
+	7800 3050 8300 3050
+Wire Wire Line
+	7800 2050 8300 2050
+Wire Wire Line
+	7800 2150 8300 2150
+Wire Wire Line
+	7800 1350 8300 1350
+Wire Wire Line
+	7800 1450 8300 1450
+Wire Wire Line
+	7800 3900 8300 3900
+Wire Wire Line
+	7800 4000 8300 4000
 $EndSCHEMATC

Commit message: update,
Connections:
- no-connect marks 0 -> 2
Other:
- note added: "DRC ok, 8 error accepted"
Changed lines of the file:
@@
 Wire Wire Line
 	7800 4000 8300 4000
+NoConn ~ 7800 5050
+NoConn ~ 7800 5150
+Text Notes 7000 6750 0    100  ~ 0
+DRC ok, 8 error accepted
 $EndSCHEMATC
