File: hardware/stm32_aux_keyboard.sch (KiCad schematic (older format))
At the start: 0 parts

Commit message: update footprint,
Parts:
- added H1, H2, H3, H4, H5, H6: MOUNT_M2, footprint-lib:MountingHole_2.7mm_M2.5,rpi_like, symbol taobao-mounting-hole:MOUNT_M2
Changed lines of the file:
@@
 Text Notes 7150 6750 0    100  ~ 0
 DRC ok, 8 error accepted
+$Comp
+L taobao-mounting-hole:MOUNT_M2 H1
+U 1 1 5CF47DFC
+P 5900 6600
+F 0 "H1" H 6000 6650 50  0000 L CNN
+F 1 "MOUNT_M2" H 6000 6600 50  0000 L CNN
+F 2 "footprint-lib:MountingHole_2.7mm_M2.5,rpi_like" H 5900 6600 50  0001 C CNN
+F 3 "~" H 5900 6600 50  0001 C CNN
+	1    5900 6600
+	1    0    0    -1
+$EndComp
+$Comp
+L taobao-mounting-hole:MOUNT_M2 H2
+U 1 1 5CF481A7
+P 5900 6800
+F 0 "H2" H 6000 6850 50  0000 L CNN
+F 1 "MOUNT_M2" H 6000 6800 50  0000 L CNN
+F 2 "footprint-lib:MountingHole_2.7mm_M2.5,rpi_like" H 5900 6800 50  0001 C CNN
+F 3 "~" H 5900 6800 50  0001 C CNN
+	1    5900 6800
+	1    0    0    -1
+$EndComp
+$Comp
+L taobao-mounting-hole:MOUNT_M2 H3
+U 1 1 5CF484A8
+P 5900 7000
+F 0 "H3" H 6000 7050 50  0000 L CNN
+F 1 "MOUNT_M2" H 6000 7000 50  0000 L CNN
+F 2 "footprint-lib:MountingHole_2.7mm_M2.5,rpi_like" H 5900 7000 50  0001 C CNN
+F 3 "~" H 5900 7000 50  0001 C CNN
+	1    5900 7000
+	1    0    0    -1
+$EndComp
+$Comp
+L taobao-mounting-hole:MOUNT_M2 H4
+U 1 1 5CF484B2
+P 5900 7200
+F 0 "H4" H 6000 7250 50  0000 L CNN
+F 1 "MOUNT_M2" H 6000 7200 50  0000 L CNN
+F 2 "footprint-lib:MountingHole_2.7mm_M2.5,rpi_like" H 5900 7200 50  0001 C CNN
+F 3 "~" H 5900 7200 50  0001 C CNN
+	1    5900 7200
+	1    0    0    -1
+$EndComp
+$Comp
+L taobao-mounting-hole:MOUNT_M2 H5
+U 1 1 5CF532EE
+P 5900 7400
+F 0 "H5" H 6000 7450 50  0000 L CNN
+F 1 "MOUNT_M2" H 6000 7400 50  0000 L CNN
+F 2 "footprint-lib:MountingHole_2.7mm_M2.5,rpi_like" H 5900 7400 50  0001 C CNN
+F 3 "~" H 5900 7400 50  0001 C CNN
+	1    5900 7400
+	1    0    0    -1
+$EndComp
+$Comp
+L taobao-mounting-hole:MOUNT_M2 H6
+U 1 1 5CF532F8
+P 5900 7600
+F 0 "H6" H 6000 7650 50  0000 L CNN
+F 1 "MOUNT_M2" H 6000 7600 50  0000 L CNN
+F 2 "footprint-lib:MountingHole_2.7mm_M2.5,rpi_like" H 5900 7600 50  0001 C CNN
+F 3 "~" H 5900 7600 50  0001 C CNN
+	1    5900 7600
+	1    0    0    -1
+$EndComp
 $EndSCHEMATC

Commit message: update for add supporting hold,
Parts:
- added H7, H8: MOUNT_M2, footprint-lib:MountingHole_2.7mm_M2.5,rpi_like, symbol taobao-mounting-hole:MOUNT_M2
Changed lines of the file:
@@
+	1    0    0    -1
+$EndComp
+$Comp
+L taobao-mounting-hole:MOUNT_M2 H7
+U 1 1 5D7BA4AD
+P 5600 7600
+F 0 "H7" H 5700 7650 50  0000 L CNN
+F 1 "MOUNT_M2" H 5700 7600 50  0000 L CNN
+F 2 "footprint-lib:MountingHole_2.7mm_M2.5,rpi_like" H 5600 7600 50  0001 C CNN
+F 3 "~" H 5600 7600 50  0001 C CNN
+	1    5600 7600
+	1    0    0    -1
+$EndComp
+$Comp
+L taobao-mounting-hole:MOUNT_M2 H8
+U 1 1 5D7BC5AB
+P 5600 7400
+F 0 "H8" H 5700 7450 50  0000 L CNN
+F 1 "MOUNT_M2" H 5700 7400 50  0000 L CNN
+F 2 "footprint-lib:MountingHole_2.7mm_M2.5,rpi_like" H 5600 7400 50  0001 C CNN
+F 3 "~" H 5600 7400 50  0001 C CNN
+	1    5600 7400
 	1    0    0    -1
 $EndComp

Commit message: prepare to fab,
Changed lines of the file:
@@
 EESchema Schematic File Version 4
 LIBS:stm32_aux_keyboard-cache
+LIBS:LM75-tryout-cache
 EELAYER 29 0
 EELAYER END
 $Descr A4 11693 8268
 encoding utf-8
-Sheet 1 13
+Sheet 1 15
 Title ""
 Date ""
@@
 $EndSheet
 $Sheet
-S 8300 2750 950  600
+S 8300 4150 950  600
 U 5CF35582
 F0 "WS2812" 50
 F1 "WS2812.sch" 50
-F2 "WS2812_IN" I L 8300 3050 50
+F2 "WS2812_IN" I L 8300 4450 50
 $EndSheet
 $Sheet
@@
 $EndSheet
 $Sheet
-S 8300 3800 750  400
+S 8250 5050 750  400
 U 5D0A467E
 F0 "usb" 50
 F1 "usb.sch" 50
-F2 "USB_P" I L 8300 3900 50
-F3 "USB_N" I L 8300 4000 50
+F2 "USB_P" I L 8250 5150 50
+F3 "USB_N" I L 8250 5250 50
 $EndSheet
 $Sheet
@@
 F15 "ROT_ENC_SW1" I L 5700 2150 50
 F16 "ROT_ENC_SW2" I L 5700 2950 50
-F17 "WS2812_OUT" I R 7800 3050 50
-F18 "TTL_TX" I R 7800 5050 50
-F19 "TTL_RX" I R 7800 5150 50
+F17 "WS2812_OUT" I R 7800 4450 50
+F18 "TTL_TX" I R 7800 5600 50
+F19 "TTL_RX" I R 7800 5700 50
 F20 "USR_BTN1" I L 5700 5500 50
 F21 "USR_BTN2" I L 5700 5600 50
@@
 F28 "SWCLK" I R 7800 1350 50
 F29 "SWDIO" I R 7800 1450 50
-F30 "USB_P" I R 7800 3900 50
-F31 "USB_N" I R 7800 4000 50
+F30 "USB_P" I R 7800 5150 50
+F31 "USB_N" I R 7800 5250 50
 $EndSheet
 Wire Wire Line
@@
 	4550 5800 5700 5800
 Wire Wire Line
-	7800 3050 8300 3050
-Wire Wire Line
-	7800 2050 8300 2050
-Wire Wire Line
-	7800 2150 8300 2150
+	7800 4450 8300 4450
+Wire Wire Line
+	7800 2050 8150 2050
+Wire Wire Line
+	7800 2150 8050 2150
 Wire Wire Line
 	7800 1350 8300 1350
@@
 	7800 1450 8300 1450
 Wire Wire Line
-	7800 3900 8300 3900
-Wire Wire Line
-	7800 4000 8300 4000
-NoConn ~ 7800 5050
-NoConn ~ 7800 5150
+	7800 5150 8250 5150
+Wire Wire Line
+	7800 5250 8250 5250
+NoConn ~ 7800 5600
+NoConn ~ 7800 5700
 Text Notes 7150 6750 0    100  ~ 0
 DRC ok, 8 error accepted
@@
 	1    0    0    -1
 $EndComp
+$Sheet
+S 8300 2600 850  450
+U 5CFA91A2
+F0 "i2c" 50
+F1 "i2c.sch" 50
+F2 "SDA" I L 8300 2750 50
+F3 "SCL" I L 8300 2850 50
+$EndSheet
+$Sheet
+S 8300 3250 850  550
+U 5CFABBB6
+F0 "24cxx" 50
+F1 "24cxx.sch" 50
+F2 "SCL" I L 8300 3600 50
+F3 "SDA" I L 8300 3500 50
+$EndSheet
+Wire Wire Line
+	8150 2050 8150 2750
+Wire Wire Line
+	8150 2750 8300 2750
+Connection ~ 8150 2050
+Wire Wire Line
+	8150 2050 8300 2050
+Wire Wire Line
+	8150 2750 8150 3500
+Wire Wire Line
+	8150 3500 8300 3500
+Connection ~ 8150 2750
+Wire Wire Line
+	8300 3600 8050 3600
+Wire Wire Line
+	8050 3600 8050 2850
+Connection ~ 8050 2150
+Wire Wire Line
+	8050 2150 8300 2150
+Wire Wire Line
+	8300 2850 8050 2850
+Connection ~ 8050 2850
+Wire Wire Line
+	8050 2850 8050 2150
 $EndSCHEMATC
