File: hardware/stm32_core.sch (KiCad schematic (older format))
At the start: 36 parts, among them J1 I2C_HEADER,2.54, SW1 RESET, U1 STM32F103C8T6, Y1 O8M, Y2 O32.768K

Commit message: update,
Parts:
- removed SW1: RESET, footprint-lib:SW_SPST_CK_RS282G05A3, symbol taobao-button:SW_RESET,2_leg,SMD
- added SW?: SW_RESET,2_leg,SMD, footprint-lib:SW_SPST_CK_RS282G05A3, symbol taobao-button:SW_RESET,2_leg,SMD
Connections:
- net GND: now also SW?.1
- net RESET: now also SW?.2
Changed lines of the file:
@@
-$EndComp
-$Comp
-L taobao-button:SW_RESET,2_leg,SMD SW1
-U 1 1 5CF92D41
-P 9350 4400
-F 0 "SW1" V 9396 4548 50  0000 L CNN
-F 1 "RESET" V 9305 4548 50  0000 L CNN
-F 2 "footprint-lib:SW_SPST_CK_RS282G05A3" H 9350 4600 50  0001 C CNN
-F 3 "~" H 9350 4600 50  0001 C CNN
-	1    9350 4400
-	0    -1   -1   0
 $EndComp
 $Comp
@@
 Wire Wire Line
 	7700 3650 8050 3650
+$Comp
+L taobao-button:SW_RESET,2_leg,SMD SW?
+U 1 1 5D5B9C66
+P 9350 4400
+F 0 "SW?" V 9250 4650 50  0000 R CNN
+F 1 "SW_RESET,2_leg,SMD" V 9150 5250 50  0000 R CNN
+F 2 "footprint-lib:SW_SPST_CK_RS282G05A3" H 9350 4600 50  0001 C CNN
+F 3 "~" H 9350 4600 50  0001 C CNN
+	1    9350 4400
+	0    -1   -1   0
+$EndComp
 $EndSCHEMATC

Commit message: update,
Parts:
- gave numbers to parts that had none: 1
Changed lines of the file:
@@
 PA11
 $Comp
-L my_power:Vstm32 #PWR?
+L my_power:Vstm32 #PWR0166
 U 1 1 5D45FAEE
 P 9400 5350
-F 0 "#PWR?" H 9400 5200 50  0001 C CNN
+F 0 "#PWR0166" H 9400 5200 50  0001 C CNN
 F 1 "Vstm32" H 9405 5523 50  0000 C CNN
 F 2 "" H 9400 5350 50  0001 C CNN
@@
 	7700 3650 8050 3650
 $Comp
-L taobao-button:SW_RESET,2_leg,SMD SW?
+L taobao-button:SW_RESET,2_leg,SMD SW1
 U 1 1 5D5B9C66
 P 9350 4400
-F 0 "SW?" V 9250 4650 50  0000 R CNN
+F 0 "SW1" V 9250 4650 50  0000 R CNN
 F 1 "SW_RESET,2_leg,SMD" V 9150 5250 50  0000 R CNN
 F 2 "footprint-lib:SW_SPST_CK_RS282G05A3" H 9350 4600 50  0001 C CNN

Commit message: update,
Connections:
- no-connect marks 24 -> 25
Changed lines of the file:
@@
 	0    -1   -1   0
 $EndComp
+Text HLabel 1100 5150 0    50   Input ~ 0
+TTL_TX
+Wire Wire Line
+	1650 5150 1100 5150
+Text Label 1650 5150 2    50   ~ 0
+PA9
+Text HLabel 1100 5250 0    50   Input ~ 0
+TTL_RX
+Wire Wire Line
+	1650 5250 1100 5250
+Text Label 1650 5250 2    50   ~ 0
+PA10
+NoConn ~ 4500 1300
 $EndSCHEMATC

Commit message: update,
Parts:
- renumbered C1 to C42, C2 to C43, C6 to C44, C5 to C45, C4 to C46, C15 to C47, C16 to C48, C17 to C49, C18 to C50, C3 to C51, C7 to C52, C8 to C53, C9 to C54, C10 to C55, C11 to C56, C12 to C57, C13 to C58, C14 to C59, D1 to D39, J1 to J8, JP1 to JP?, JP2 to JP?, R1 to R31, R2 to R32, R3 to R33, R6 to R34, R4 to R35, R5 to R36, R7 to R37, R8 to R38, R9 to R39, R10 to R40, SW1 to SW19, U1 to U10, Y1 to Y2, Y2 to Y3

Commit message: update footprint,
Parts:
- gave numbers to parts that had none: 2
Changed lines of the file:
@@
 $EndComp
 $Comp
-L my_solder_jumper:SolderJumper_3_Bridged12 JP?
+L my_solder_jumper:SolderJumper_3_Bridged12 JP7
 U 1 1 5CF7DD63
 P 9300 1600
-F 0 "JP?" V 9346 1668 50  0000 L CNN
+F 0 "JP7" V 9346 1668 50  0000 L CNN
 F 1 "BOOT0" V 9255 1668 50  0000 L CNN
 F 2 "Jumper:SolderJumper-3_P1.3mm_Bridged2Bar12_Pad1.0x1.5mm" H 9300 1600 50  0001 C CNN
@@
 $EndComp
 $Comp
-L my_solder_jumper:SolderJumper_3_Bridged12 JP?
+L my_solder_jumper:SolderJumper_3_Bridged12 JP8
 U 1 1 5CF7E819
 P 10150 1600
-F 0 "JP?" V 10196 1668 50  0000 L CNN
+F 0 "JP8" V 10196 1668 50  0000 L CNN
 F 1 "BOOT1" V 10105 1668 50  0000 L CNN
 F 2 "Jumper:SolderJumper-3_P1.3mm_Bridged2Bar12_Pad1.0x1.5mm" H 10150 1600 50  0001 C CNN

Commit message: update footprint,
Parts:
- J8: footprint Connector_PinHeader_2.54mm:PinHeader_1x02_P2.54mm_Vertical -> footprint-lib:I2C_DEBUG,2.54
Changed lines of the file:
@@
 F 0 "J8" H 10372 6024 50  0000 R CNN
 F 1 "I2C_HEADER,2.54" H 10372 5933 50  0000 R CNN
-F 2 "Connector_PinHeader_2.54mm:PinHeader_1x02_P2.54mm_Vertical" H 10400 5600 50  0001 C CNN
+F 2 "footprint-lib:I2C_DEBUG,2.54" H 10400 5600 50  0001 C CNN
 F 3 "" H 10400 5950 50  0001 C CNN
 	1    10400 6000

Commit message: update footprint,
Parts:
- D39: footprint LED_SMD:LED_0805_2012Metric_Pad1.15x1.40mm_HandSolder -> footprint-lib:LED_0603_1608Metric
Changed lines of the file:
@@
 EESchema Schematic File Version 4
-LIBS:stm32_aux_keyboard-cache
 EELAYER 29 0
 EELAYER END
 $Descr A4 11693 8268
 encoding utf-8
-Sheet 13 13
+Sheet 1 1
 Title ""
 Date ""
@@
 F 0 "D39" V 8096 3882 50  0000 R CNN
 F 1 "PC13" V 8005 3882 50  0000 R CNN
-F 2 "LED_SMD:LED_0805_2012Metric_Pad1.15x1.40mm_HandSolder" V 8050 3950 50  0001 C CNN
+F 2 "footprint-lib:LED_0603_1608Metric" V 8050 3950 50  0001 C CNN
 F 3 "~" V 8050 3950 50  0001 C CNN
 	1    8050 3950
