File: hardware/stm32_core.sch (KiCad schematic (older format))
At the start: 36 parts, among them J8 I2C_HEADER,2.54, SW19 SW_RESET,2_leg,SMD, U10 STM32F103C8T6, Y2 O8M, Y3 O32.768K

Commit message: update for routing,
Connections:
- net +3V3 is gone; now on net Vstm32: C42.1
Changed lines of the file:
@@
 Text Label 1600 6450 2    50   ~ 0
 VDDA
-$Comp
-L power:+3V3 #PWR0153
-U 1 1 5BCF284B
-P 3750 900
-F 0 "#PWR0153" H 3750 750 50  0001 C CNN
-F 1 "+3V3" H 3800 1100 50  0000 C CNN
-F 2 "" H 3750 900 50  0001 C CNN
-F 3 "" H 3750 900 50  0001 C CNN
-	1    3750 900
-	0    -1   -1   0
-$EndComp
 Wire Wire Line
 	1600 6450 1250 6450
@@
 PA10
 NoConn ~ 4500 1300
+$Comp
+L my_power:Vstm32 #PWR?
+U 1 1 5CF57716
+P 3750 900
+F 0 "#PWR?" H 3750 750 50  0001 C CNN
+F 1 "Vstm32" H 3755 1073 50  0000 C CNN
+F 2 "" H 3750 900 50  0001 C CNN
+F 3 "" H 3750 900 50  0001 C CNN
+	1    3750 900
+	0    -1   -1   0
+$EndComp
 $EndSCHEMATC

Commit message: check footprint,
Parts:
- Y3: value O32.768K -> O_EPSON_32.768K
Changed lines of the file:
@@
-$EndComp
-$Comp
-L taobao-components:O_EPSON_32.768K Y3
-U 1 1 5BCBF11C
-P 8050 5650
-F 0 "Y3" V 8004 5738 50  0000 L CNN
-F 1 "O32.768K" V 8095 5738 50  0000 L CNN
-F 2 "footprint-lib:MC-306" H 8050 5650 50  0001 C CNN
-F 3 "~" H 8050 5650 50  0001 C CNN
-	1    8050 5650
-	1    0    0    -1
 $EndComp
 $Comp
@@
 	0    -1   -1   0
 $EndComp
+$Comp
+L taobao-components:O_EPSON_32.768K Y3
+U 1 1 5CFA3682
+P 8050 5650
+F 0 "Y3" H 8050 5875 50  0000 C CNN
+F 1 "O_EPSON_32.768K" H 8050 5784 50  0000 C CNN
+F 2 "footprint-lib:MC-306" H 8050 5450 50  0001 C CNN
+F 3 "https://support.epson.biz/td/api/doc_check.php?dl=brief_MC-306&lang=en" H 8050 5650 50  0001 C CNN
+	1    8050 5650
+	1    0    0    -1
+$EndComp
 $EndSCHEMATC
