File: hardware/power.kicad_pcb (KiCad board)
At the start: 2 copper layers, 22 parts, among them U2 footprint-lib:AMS1117_SOT-223

Commit message: update footprint,
Parts:
- moved R5 30.5 mm to (40.0, 72.5)
- moved D1 28.8 mm to (35.0, 72.5)
- moved JP3 26.5 mm to (65.0, 85.0)
- moved TP2 25.7 mm to (70.0, 80.0)
- moved D2 23.0 mm to (35.0, 75.0), turned to 0 degrees
- moved TP1 21.3 mm to (70.0, 95.0)
- moved R4 20.7 mm to (30.0, 90.0), turned to 90 degrees
- moved R6 20.0 mm to (40.0, 75.0), turned to 0 degrees
- moved TP6 18.8 mm to (45.0, 90.0)
- moved JP4 17.8 mm to (65.0, 90.0)
- moved F1 17.3 mm to (35.0, 90.0), turned to 90 degrees
- moved R3 16.7 mm to (32.5, 90.0), turned to 270 degrees
- moved TP5 16.5 mm to (50.0, 90.0)
- moved TP3 15.5 mm to (70.0, 85.0)
- moved TP7 11.1 mm to (55.0, 90.0)
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
Commit message: update for routing,
Parts:
- C4, R3, R4: moved to B.Cu
- U2: value footprint-lib:AMS1117_SOT-223 -> AMS1117-3.3; moved to B.Cu
- moved TP1 17.7 mm to (53.5, 88.5)
- moved TP4 17.1 mm to (53.5, 85.5)
- moved TP3 16.7 mm to (53.5, 82.5)
- moved TP2 16.5 mm to (53.5, 79.5)
- moved JP1 16.3 mm to (50.0, 88.5), turned to 180 degrees
- moved JP4 15.7 mm to (50.0, 85.5), turned to 180 degrees
- moved JP3 15.2 mm to (50.0, 82.5), turned to 180 degrees
- moved JP2 15.0 mm to (50.0, 79.5), turned to 180 degrees
- moved TP5 13.5 mm to (36.5, 90.5)
- moved TP7 12.5 mm to (42.5, 90.5)
- moved C4 9.33 mm to (45.0, 83.5)
- moved R4 7.40 mm to (28.5, 82.8)
- moved R3 7.25 mm to (32.8, 82.8)
- moved D1 6.73 mm to (40.0, 77.0), turned to 270 degrees
- moved C3 5.77 mm to (43.5, 83.5)
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Routing:
- net GND: track 0.00 -> 61.7 mm
- net +5V: track 0.00 -> 50.7 mm
- net +3V3: track 0.00 -> 36.6 mm
- net Vusb: track 0.00 -> 5.60 mm, vias 0 -> 1
- net Net-(R3-Pad2): track 0.00 -> 4.28 mm
- net Vws2812: track 0.00 -> 2.85 mm
- net Vstm32: track 0.00 -> 2.85 mm
- net Voled: track 0.00 -> 2.85 mm
- net Vbuzzer: track 0.00 -> 2.85 mm
- net Net-(D2-Pad1): track 0.00 -> 2.04 mm
- net Net-(D1-Pad1): track 0.00 -> 2.04 mm
