File: hardware/keyboard_key.kicad_pcb (KiCad board)
At the start: 2 copper layers, 24 parts, among them SW10 KEY22, SW11 KEY23, SW12 KEY31, SW13 KEY32, SW14 KEY33, SW15 KEY41, SW16 KEY42, SW17 KEY43, SW6 KEY11, SW7 KEY12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

Commit message: update for autoroute complete,
Routing:
- net /COL1: track 103.2 -> 0.00 mm
- net /COL2: track 98.6 -> 0.00 mm
- net /COL3: track 78.7 -> 0.00 mm
- net /ROW2: track 71.9 -> 0.00 mm
- net /ROW4: track 71.4 -> 0.00 mm
- net /ROW3: track 41.2 -> 0.00 mm
- net /ROW1: track 40.0 -> 0.00 mm
- net Net-(D37-Pad2): track 9.45 -> 0.00 mm
- net Net-(D36-Pad2): track 9.45 -> 0.00 mm
- net Net-(D33-Pad2): track 9.45 -> 0.00 mm
- net Net-(D32-Pad2): track 9.45 -> 0.00 mm
- net Net-(D31-Pad2): track 9.45 -> 0.00 mm
- net Net-(D29-Pad2): track 9.45 -> 0.00 mm
- net Net-(D28-Pad2): track 9.45 -> 0.00 mm
- net Net-(D27-Pad2): track 9.45 -> 0.00 mm
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Changed lines of the file:
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@@
     (thickness 1.6)
     (drawings 0)
-    (tracks 97)
+    (tracks 0)
     (zones 0)
     (modules 24)
@@
     )
   )
-  (segment (start 20 21.65) (end 20 22.4253) (width 0.25) (layer B.Cu) (net 1))
-  (segment (start 20 22.4253) (end 22.46 24.8853) (width 0.25) (layer B.Cu) (net 1))
-  (segment (start 22.46 24.8853) (end 22.46 30.08) (width 0.25) (layer B.Cu) (net 1))
-  (segment (start 40 18.35) (end 60 18.35) (width 0.25) (layer B.Cu) (net 2))
-  (segment (start 20 18.35) (end 40 18.35) (width 0.25) (layer B.Cu) (net 2))
-  (segment (start 40 21.65) (end 40 22.4253) (width 0.25) (layer B.Cu) (net 3))
-  (segment (start 40 22.4253) (end 42.46 24.8853) (width 0.25) (layer B.Cu) (net 3))
-  (segment (start 42.46 24.8853) (end 42.46 30.08) (width 0.25) (layer B.Cu) (net 3))
-  (segment (start 60 21.65) (end 60 22.4253) (width 0.25) (layer B.Cu) (net 4))
-  (segment (start 60 22.4253) (end 62.46 24.8853) (width 0.25) (layer B.Cu) (net 4))
-  (segment (start 62.46 24.8853) (end 62.46 30.08) (width 0.25) (layer B.Cu) (net 4))
-  (segment (start 80 21.65) (end 80 22.4253) (width 0.25) (layer B.Cu) (net 5))
-  (segment (start 80 22.4253) (end 82.46 24.8853) (width 0.25) (layer B.Cu) (net 5))
-  (segment (start 82.46 24.8853) (end 82.46 30.08) (width 0.25) (layer B.Cu) (net 5))
-  (segment (start 20 38.35) (end 20.9253 38.35) (width 0.25) (layer B.Cu) (net 6))
-  (segment (start 40 37.9623) (end 21.313 37.9623) (width 0.25) (layer B.Cu) (net 6))
-  (segment (start 21.313 37.9623) (end 20.9253 38.35) (width 0.25) (layer B.Cu) (net 6))
-  (segment (start 40 37.9623) (end 40 37.5747) (width 0.25) (layer B.Cu) (net 6))
-  (segment (start 40 38.35) (end 40 37.9623) (width 0.25) (layer B.Cu) (net 6))
-  (segment (start 80 18.35) (end 80 19.1253) (width 0.25) (layer B.Cu) (net 6))
-  (segment (start 80 19.1253) (end 54.1548 19.1253) (width 0.25) (layer B.Cu) (net 6))
-  (segment (start 54.1548 19.1253) (end 44.813 28.4671) (width 0.25) (layer B.Cu) (net 6))
-  (segment (start 44.813 28.4671) (end 44.813 32.7617) (width 0.25) (layer B.Cu) (net 6))
-  (segment (start 44.813 32.7617) (end 40 37.5747) (width 0.25) (layer B.Cu) (net 6))
-  (segment (start 20 41.65) (end 20 42.4253) (width 0.25) (layer B.Cu) (net 7))
-  (segment (start 20 42.4253) (end 22.46 44.8853) (width 0.25) (layer B.Cu) (net 7))
-  (segment (start 22.46 44.8853) (end 22.46 50.08) (width 0.25) (layer B.Cu) (net 7))
-  (segment (start 40 41.65) (end 40 42.4253) (width 0.25) (layer B.Cu) (net 8))
-  (segment (start 40 42.4253) (end 42.46 44.8853) (width 0.25) (layer B.Cu) (net 8))
-  (segment (start 42.46 44.8853) (end 42.46 50.08) (width 0.25) (layer B.Cu) (net 8))
-  (segment (start 60 41.65) (end 60 42.4253) (width 0.25) (layer B.Cu) (net 9))
-  (segment (start 60 42.4253) (end 62.46 44.8853) (width 0.25) (layer B.Cu) (net 9))
-  (segment (start 62.46 44.8853) (end 62.46 50.08) (width 0.25) (layer B.Cu) (net 9))
-  (segment (start 80 38.35) (end 79.0747 38.35) (width 0.25) (layer B.Cu) (net 10))
-  (segment (start 60 38.7376) (end 78.6871 38.7376) (width 0.25) (layer B.Cu) (net 10))
-  (segment (start 78.6871 38.7376) (end 79.0747 38.35) (width 0.25) (layer B.Cu) (net 10))
-  (segment (start 60 38.7376) (end 60 39.1253) (width 0.25) (layer B.Cu) (net 10))
-  (segment (start 60 38.35) (end 60 38.7376) (width 0.25) (layer B.Cu) (net 10))
-  (segment (start 60 39.1253) (end 58.6861 40.4392) (width 0.25) (layer B.Cu) (net 10))
-  (segment (start 58.6861 40.4392) (end 58.6861 56.2608) (width 0.25) (layer B.Cu) (net 10))
-  (segment (start 58.6861 56.2608) (end 60 57.5747) (width 0.25) (layer B.Cu) (net 10))
-  (segment (start 60 58.35) (end 60 57.5747) (width 0.25) (layer B.Cu) (net 10))
-  (segment (start 80 41.65) (end 80 42.4253) (width 0.25) (layer B.Cu) (net 11))
-  (segment (start 80 42.4253) (end 82.46 44.8853) (width 0.25) (layer B.Cu) (net 11))
-  (segment (start 82.46 44.8853) (end 82.46 50.08) (width 0.25) (layer B.Cu) (net 11))
-  (segment (start 60 62.4253) (end 62.0097 64.435) (width 0.25) (layer B.Cu) (net 12))
-  (segment (start 62.0097 64.435) (end 62.0097 69.6297) (width 0.25) (layer B.Cu) (net 12))
-  (segment (start 62.0097 69.6297) (end 62.46 70.08) (width 0.25) (layer B.Cu) (net 12))
-  (segment (start 60 61.65) (end 60 62.4253) (width 0.25) (layer B.Cu) (net 12))
-  (segment (start 40 62.4253) (end 42.46 64.8853) (width 0.25) (layer B.Cu) (net 13))
-  (segment (start 42.46 64.8853) (end 42.46 70.08) (width 0.25) (layer B.Cu) (net 13))
-  (segment (start 40 61.65) (end 40 62.4253) (width 0.25) (layer B.Cu) (net 13))
-  (segment (start 40 58.5438) (end 42.0263 60.5701) (width 0.25) (layer B.Cu) (net 14))
-  (segment (start 42.0263 60.5701) (end 60.4754 60.5701) (width 0.25) (layer B.Cu) (net 14))
-  (segment (start 60.4754 60.5701) (end 62.46 62.5547) (width 0.25) (layer B.Cu) (net 14))
-  (segment (start 62.46 62.5547) (end 62.46 65.7424) (width 0.25) (layer B.Cu) (net 14))
-  (segment (start 62.46 65.7424) (end 65.745 69.0274) (width 0.25) (layer B.Cu) (net 14))
-  (segment (start 65.745 69.0274) (end 70.0979 69.0274) (width 0.25) (layer B.Cu) (net 14))
-  (segment (start 70.0979 69.0274) (end 80 59.1253) (width 0.25) (layer B.Cu) (net 14))
-  (segment (start 40 58.5438) (end 21.1191 58.5438) (width 0.25) (layer B.Cu) (net 14))
-  (segment (start 21.1191 58.5438) (end 20.9253 58.35) (width 0.25) (layer B.Cu) (net 14))
-  (segment (start 80 58.35) (end 80 59.1253) (width 0.25) (layer B.Cu) (net 14))
-  (segment (start 20 58.35) (end 20.9253 58.35) (width 0.25) (layer B.Cu) (net 14))
-  (segment (start 40 58.35) (end 40 58.5438) (width 0.25) (layer B.Cu) (net 14))
-  (segment (start 20 62.4253) (end 22.0097 64.435) (width 0.25) (layer B.Cu) (net 15))
-  (segment (start 22.0097 64.435) (end 22.0097 69.6297) (width 0.25) (layer B.Cu) (net 15))
-  (segment (start 22.0097 69.6297) (end 22.46 70.08) (width 0.25) (layer B.Cu) (net 15))
-  (segment (start 20 61.65) (end 20 62.4253) (width 0.25) (layer B.Cu) (net 15))
-  (segment (start 80 61.65) (end 80 62.4253) (width 0.25) (layer B.Cu) (net 16))
-  (segment (start 80 62.4253) (end 82.46 64.8853) (width 0.25) (layer B.Cu) (net 16))
-  (segment (start 82.46 64.8853) (end 82.46 70.08) (width 0.25) (layer B.Cu) (net 16))
-  (segment (start 68.81 47.54) (end 72.3579 47.54) (width 0.25) (layer B.Cu) (net 17))
-  (segment (start 72.3579 47.54) (end 88.81 31.0879) (width 0.25) (layer B.Cu) (net 17))
-  (segment (start 88.81 31.0879) (end 88.81 27.54) (width 0.25) (layer B.Cu) (net 17))
-  (segment (start 61.9734 54.3766) (end 61.9734 54.8896) (width 0.25) (layer F.Cu) (net 17))
-  (segment (start 61.9734 54.8896) (end 49.323 67.54) (width 0.25) (layer F.Cu) (net 17))
-  (segment (start 49.323 67.54) (end 48.81 67.54) (width 0.25) (layer F.Cu) (net 17))
-  (segment (start 28.81 27.54) (end 35.1368 27.54) (width 0.25) (layer F.Cu) (net 17))
-  (segment (start 35.1368 27.54) (end 61.9734 54.3766) (width 0.25) (layer F.Cu) (net 17))
-  (segment (start 68.81 47.54) (end 61.9734 54.3766) (width 0.25) (layer F.Cu) (net 17))
-  (segment (start 48.81 27.54) (end 56.1753 27.54) (width 0.25) (layer F.Cu) (net 18))
-  (segment (start 56.1753 27.54) (end 76.1753 47.54) (width 0.25) (layer F.Cu) (net 18))
-  (segment (start 76.1753 47.54) (end 88.81 47.54) (width 0.25) (layer F.Cu) (net 18))
-  (segment (start 48.81 27.54) (end 48.81 31.0522) (width 0.25) (layer B.Cu) (net 18))
-  (segment (start 48.81 31.0522) (end 32.3222 47.54) (width 0.25) (layer B.Cu) (net 18))
-  (segment (start 32.3222 47.54) (end 28.81 47.54) (width 0.25) (layer B.Cu) (net 18))
-  (segment (start 28.81 47.54) (end 28.81 67.54) (width 0.25) (layer F.Cu) (net 18))
-  (segment (start 50.044 47.54) (end 50.044 49.9041) (width 0.25) (layer B.Cu) (net 19))
-  (segment (start 50.044 49.9041) (end 59.6031 59.4632) (width 0.25) (layer B.Cu) (net 19))
-  (segment (start 59.6031 59.4632) (end 62.8103 59.4632) (width 0.25) (layer B.Cu) (net 19))
-  (segment (start 62.8103 59.4632) (end 68.81 65.4629) (width 0.25) (layer B.Cu) (net 19))
-  (segment (start 68.81 65.4629) (end 68.81 67.54) (width 0.25) (layer B.Cu) (net 19))
-  (segment (start 68.81 27.54) (end 68.81 28.004) (width 0.25) (layer B.Cu) (net 19))
-  (segment (start 68.81 28.004) (end 50.044 46.77) (width 0.25) (layer B.Cu) (net 19))
-  (segment (start 50.044 46.77) (end 50.044 47.54) (width 0.25) (layer B.Cu) (net 19))
-  (segment (start 50.044 47.54) (end 48.81 47.54) (width 0.25) (layer B.Cu) (net 19))
-  (segment (start 68.81 67.54) (end 88.81 67.54) (width 0.25) (layer F.Cu) (net 19))
 )
